File: pcb/register/register.kicad_sch (KiCad schematic)
At the start: 58 parts, among them J1 Conn_01x08, J2 Conn_01x08, J3 Conn_01x08, Q1 2N7000, Q10 2N7000, Q11 2N7000, Q2 2N7000, Q3 2N7000, Q4 2N7000, Q5 2N7000, Q6 2N7000, Q7 2N7000, Q8 2N7000, Q9 2N7000, U1 74HC00, U10 74HC00, U11 74HC00, U12 74HC00, U13 74HC00, U14 74HC00, U15 74HC00, U16 74HC00, U17 74HC00, U18 74HC00, U19 74HC00, U2 74HC00, U20 74HC00, U21 74HC00, U22 74HC00, U23 74HC00, U3 74HC00, U4 74HC00, U5 74HC00, U6 74HC00, U7 74HC00, U8 74HC00, U9 74HC00

Commit message: register file
Parts:
- removed Q11, Q9: 2N7000, Package_TO_SOT_THT:TO-92_Inline, symbol Transistor_FET:2N7000
- removed R10, R11, R9: 1K, Resistor_THT:R_Axial_DIN0207_L6.3mm_D2.5mm_P7.62mm_Horizontal, symbol Device:R_Small
- added C1, C10, C11, C12, C13, C14, C15, C16, C17, C18, C19, C2, C20, C21, C22, C23, C24, C3, C4, C5, C6, C7, C8, C9: 100nF, Capacitor_THT:C_Radial_D5.0mm_H11.0mm_P2.00mm, symbol Device:C_Small
- added H4: MountingHole_Pad, MountingHole:MountingHole_3.5mm_Pad, symbol Mechanical:MountingHole_Pad
- added Q9: BS250, Package_TO_SOT_THT:TO-92_Inline, symbol Transistor_FET:BS250
- added R12, R13, R14, R15, R16, R17, R18, R19: 1K, Resistor_THT:R_Axial_DIN0207_L6.3mm_D2.5mm_P7.62mm_Horizontal, symbol Device:R_Small
- added U24: 74HC00, Package_DIP:DIP-14_W7.62mm_LongPads, symbol 74xx:74HC00
Connections:
- net +5V: now also R1.2, R2.2, R3.2, R4.2, R5.2, R6.2, R7.2, R8.2, C1.1, C10.1, C11.1, C12.1, C13.1, C14.1, C15.1, C16.1, C17.1, C18.1, C19.1, C2.1, C20.1, C21.1, C22.1, C23.1, C24.1, C3.1, C4.1, C5.1, C6.1, C7.1, C8.1, C9.1, Q9.3 (S), U24.14 (VCC); no longer Q1.1 (S), Q10.1 (S), Q2.1 (S), Q3.1 (S), Q4.1 (S), Q5.1 (S), Q6.1 (S), Q7.1 (S), Q8.1 (S)
- net GND: now also Q1.1 (S), Q10.1 (S), Q2.1 (S), Q3.1 (S), Q4.1 (S), Q5.1 (S), Q6.1 (S), Q7.1 (S), Q8.1 (S), C1.2, C10.2, C11.2, C12.2, C13.2, C14.2, C15.2, C16.2, C17.2, C18.2, C19.2, C2.2, C20.2, C21.2, C22.2, C23.2, C24.2, C3.2, C4.2, C5.2, C6.2, C7.2, C8.2, C9.2, H4.1, U24.7 (GND); no longer D1.1 (K), D2.1 (K), D3.1 (K), D4.1 (K), D5.1 (K), D6.1 (K), D7.1 (K), D8.1 (K)
- net READ_0: now also R12.2; no longer Q7.2 (G)
- net READ_1: now also R13.2; no longer Q6.2 (G)
- net READ_2: now also R14.2; no longer Q5.2 (G)
- net READ_3: now also R15.2; no longer Q4.2 (G)
- net READ_4: now also R16.2; no longer Q3.2 (G)
- net READ_5: now also R17.2; no longer Q2.2 (G)
- net READ_6: now also R18.2; no longer Q1.2 (G)
- net READ_7: now also R19.2; no longer Q8.2 (G)
- net at U1.13, U1.9, U3.13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: now also U24.3; no longer U13.13, U13.9, U14.13, U14.9, U15.13, U15.9, U16.13, U16.9
- net at Q7.3 (D): now also D7.1 (K); no longer R1.2
- net at Q6.3 (D): now also D6.1 (K); no longer R2.2
- net at U10.10, U10.2, U21.10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: now also Q10.3 (D), Q9.1 (D)
- net at J3.3 (Pin_3), U23.1: now also U23.12, U23.13
- net at Q3.3 (D): now also D3.1 (K); no longer R5.2
- net at Q4.3 (D): now also D4.1 (K); no longer R4.2
- net at Q8.3 (D): now also D8.1 (K); no longer R8.2
- net at Q5.3 (D): now also D5.1 (K); no longer R3.2
- net at Q1.3 (D): now also D1.1 (K); no longer R7.2
- net at Q10.2 (G), U23.11: now also Q9.2 (G)
- net at Q2.3 (D): now also D2.1 (K); no longer R6.2
- new net: Q8.2 (G), R19.1
- new net: U2.1, U2.5, U24.1, U24.11, U24.2, U4.1, U4.5, U8.1, U8.5, U9.1, U9.5
- new net: Q3.2 (G), R14.1
- new net: U17.1, U17.5, U18.1, U18.5, U19.1, U19.5, U20.1, U20.5, U24.10, U24.6, U24.9
- new net: U13.13, U13.9, U14.13, U14.9, U15.13, U15.9, U16.13, U16.9, U24.8
- new net: Q2.2 (G), R13.1
- new net: Q4.2 (G), R15.1
- new net: Q7.2 (G), R18.1
- new net: U23.8, U24.12, U24.13, U24.4, U24.5
- new net: Q1.2 (G), R12.1
- new net: Q5.2 (G), R16.1
- new net: Q6.2 (G), R17.1
Other:
- moved on the sheet: D1, D2, D3, D4, D5, D6, D7, D8, R1, R2, R3, R4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
