File: pcb/register/register.kicad_pcb (KiCad board)
At the start: 2 copper layers, 213.4 x 66 mm, 58 parts, among them J1 Conn_01x08, J2 Conn_01x08, J3 Conn_01x08, Q1 2N7000, Q10 2N7000, Q11 2N7000, Q2 2N7000, Q3 2N7000, Q4 2N7000, Q5 2N7000, Q6 2N7000, Q7 2N7000, Q8 2N7000, Q9 2N7000, U1 74HC00, U10 74HC00, U11 74HC00, U12 74HC00, U13 74HC00, U14 74HC00, U15 74HC00, U16 74HC00, U17 74HC00, U18 74HC00, U19 74HC00, U2 74HC00, U20 74HC00, U21 74HC00, U22 74HC00, U23 74HC00, U3 74HC00, U4 74HC00, U5 74HC00, U6 74HC00, U7 74HC00, U8 74HC00, U9 74HC00

Commit message: register file
Parts:
- removed J1, J2, J3: Conn_01x08, Connector_IDC:IDC-Header_2x04_P2.54mm_Vertical
- removed Q11: 2N7000, Package_TO_SOT_THT:TO-92_Inline
- removed R10, R11, R9: 1K, Resistor_THT:R_Axial_DIN0207_L6.3mm_D2.5mm_P7.62mm_Horizontal
- added C1: 100nF, Capacitor_THT:C_Radial_D5.0mm_H11.0mm_P2.00mm, F.Cu at (110.5, 53.1)
- added C10: 100nF, Capacitor_THT:C_Radial_D5.0mm_H11.0mm_P2.00mm, F.Cu at (121.9, 68.8)
- added C11: 100nF, Capacitor_THT:C_Radial_D5.0mm_H11.0mm_P2.00mm, F.Cu at (133.3, 68.8)
- added C12: 100nF, Capacitor_THT:C_Radial_D5.0mm_H11.0mm_P2.00mm, F.Cu at (144.8, 68.8)
- added C13: 100nF, Capacitor_THT:C_Radial_D5.0mm_H11.0mm_P2.00mm, F.Cu at (156.2, 68.8)
- added C14: 100nF, Capacitor_THT:C_Radial_D5.0mm_H11.0mm_P2.00mm, F.Cu at (167.6, 68.8)
- added C15: 100nF, Capacitor_THT:C_Radial_D5.0mm_H11.0mm_P2.00mm, F.Cu at (179.1, 68.8)
- added C16: 100nF, Capacitor_THT:C_Radial_D5.0mm_H11.0mm_P2.00mm, F.Cu at (190.5, 68.8)
- added C17: 100nF, Capacitor_THT:C_Radial_D5.0mm_H11.0mm_P2.00mm, F.Cu at (116.2, 53.1)
- added C18: 100nF, Capacitor_THT:C_Radial_D5.0mm_H11.0mm_P2.00mm, F.Cu at (139.1, 53.1)
- added C19: 100nF, Capacitor_THT:C_Radial_D5.0mm_H11.0mm_P2.00mm, F.Cu at (161.9, 53.1)
- added C2: 100nF, Capacitor_THT:C_Radial_D5.0mm_H11.0mm_P2.00mm, F.Cu at (121.9, 53.1)
- added C20: 100nF, Capacitor_THT:C_Radial_D5.0mm_H11.0mm_P2.00mm, F.Cu at (184.8, 53.1)
- added C21: 100nF, Capacitor_THT:C_Radial_D5.0mm_H11.0mm_P2.00mm, F.Cu at (87.6, 53.1)
- added C22: 100nF, Capacitor_THT:C_Radial_D5.0mm_H11.0mm_P2.00mm, F.Cu at (99.1, 53.1)
- added C23: 100nF, Capacitor_THT:C_Radial_D5.0mm_H11.0mm_P2.00mm, F.Cu at (87.6, 68.8)
- added C24: 100nF, Capacitor_THT:C_Radial_D5.0mm_H11.0mm_P2.00mm, F.Cu at (99.1, 68.8)
- added C3: 100nF, Capacitor_THT:C_Radial_D5.0mm_H11.0mm_P2.00mm, F.Cu at (133.3, 53.1)
- added C4: 100nF, Capacitor_THT:C_Radial_D5.0mm_H11.0mm_P2.00mm, F.Cu at (144.8, 53.1)
- added C5: 100nF, Capacitor_THT:C_Radial_D5.0mm_H11.0mm_P2.00mm, F.Cu at (156.2, 53.1)
- added C6: 100nF, Capacitor_THT:C_Radial_D5.0mm_H11.0mm_P2.00mm, F.Cu at (167.6, 53.1)
- added C7: 100nF, Capacitor_THT:C_Radial_D5.0mm_H11.0mm_P2.00mm, F.Cu at (179.1, 53.1)
- added C8: 100nF, Capacitor_THT:C_Radial_D5.0mm_H11.0mm_P2.00mm, F.Cu at (190.5, 53.1)
- added C9: 100nF, Capacitor_THT:C_Radial_D5.0mm_H11.0mm_P2.00mm, F.Cu at (110.5, 68.8)
- added CONTROL: Conn_01x08, Connector_IDC:IDC-Header_2x04_P2.54mm_Vertical, F.Cu at (75.6, 37.5)
- added H4: MountingHole_Pad, MountingHole:MountingHole_3.5mm_Pad, F.Cu at (101.0, 61.0)
- added R12: 1K, Resistor_THT:R_Axial_DIN0207_L6.3mm_D2.5mm_P7.62mm_Horizontal, F.Cu at (201.9, 81.9)
- added R13: 1K, Resistor_THT:R_Axial_DIN0207_L6.3mm_D2.5mm_P7.62mm_Horizontal, F.Cu at (198.8, 81.9)
- added R14: 1K, Resistor_THT:R_Axial_DIN0207_L6.3mm_D2.5mm_P7.62mm_Horizontal, F.Cu at (201.9, 70.5)
- added R15: 1K, Resistor_THT:R_Axial_DIN0207_L6.3mm_D2.5mm_P7.62mm_Horizontal, F.Cu at (198.8, 70.5)
- added R16: 1K, Resistor_THT:R_Axial_DIN0207_L6.3mm_D2.5mm_P7.62mm_Horizontal, F.Cu at (201.9, 59.1)
- added R17: 1K, Resistor_THT:R_Axial_DIN0207_L6.3mm_D2.5mm_P7.62mm_Horizontal, F.Cu at (198.8, 59.1)
- added R18: 1K, Resistor_THT:R_Axial_DIN0207_L6.3mm_D2.5mm_P7.62mm_Horizontal, F.Cu at (201.9, 47.6)
- added R19: 1K, Resistor_THT:R_Axial_DIN0207_L6.3mm_D2.5mm_P7.62mm_Horizontal, F.Cu at (198.8, 47.6)
- added READ: Conn_01x08, Connector_IDC:IDC-Header_2x04_P2.54mm_Vertical, F.Cu at (75.6, 76.8)
- added U24: 74HC00, Package_DIP:DIP-14_W7.62mm_LongPads, F.Cu at (91.5, 90.2)
- added WRITE: Conn_01x08, Connector_IDC:IDC-Header_2x04_P2.54mm_Vertical, F.Cu at (75.6, 57.1)
- Q9: value 2N7000 -> BS250
- moved H2 163.5 mm to (215.3, 90.2)
- moved U7 103.2 mm to (175.2, 31.7), turned to 0 degrees
- moved U6 101.9 mm to (152.4, 31.7), turned to 0 degrees
- moved U3 100.6 mm to (129.5, 31.7), turned to 0 degrees
- moved U1 99.4 mm to (106.6, 31.7), turned to 0 degrees
- moved H1 92.1 mm to (215.3, 31.8)
- moved R8 84.1 mm to (205.1, 40.0), turned to -90 degrees
- moved U9 81.0 mm to (186.7, 31.7), turned to 0 degrees
- moved D8 80.5 mm to (214.0, 40.6), turned to 180 degrees
- moved U12 79.2 mm to (102.9, 90.2), turned to 180 degrees
- moved U8 79.0 mm to (163.8, 31.7), turned to 0 degrees
- moved Q8 77.7 mm to (217.2, 39.4)
- moved R7 77.0 mm to (208.3, 40.0), turned to -90 degrees
- moved U4 76.9 mm to (140.9, 31.7), turned to 0 degrees
- moved U2 75.0 mm to (118.1, 31.7), turned to 0 degrees
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Connections:
- D1 pad 1: GND -> Net-(D1-K)
- D2 pad 1: GND -> Net-(D2-K)
- D3 pad 1: GND -> Net-(D3-K)
- D4 pad 1: GND -> Net-(D4-K)
- D5 pad 1: GND -> Net-(D5-K)
- D6 pad 1: GND -> Net-(D6-K)
- D7 pad 1: GND -> Net-(D7-K)
- D8 pad 1: GND -> Net-(D8-K)
- Q1 pad 1: +5V -> GND
- Q1 pad 2: /READ_6 -> Net-(Q1-G)
- Q1 pad 3: Net-(Q1-D) -> Net-(D1-K)
- Q10 pad 1: +5V -> GND
- Q2 pad 1: +5V -> GND
- Q2 pad 2: /READ_5 -> Net-(Q2-G)
- Q2 pad 3: Net-(Q2-D) -> Net-(D2-K)
- Q3 pad 1: +5V -> GND
- Q3 pad 2: /READ_4 -> Net-(Q3-G)
- Q3 pad 3: Net-(Q3-D) -> Net-(D3-K)
- Q4 pad 1: +5V -> GND
- Q4 pad 2: /READ_3 -> Net-(Q4-G)
- Q4 pad 3: Net-(Q4-D) -> Net-(D4-K)
- Q5 pad 1: +5V -> GND
- Q5 pad 2: /READ_2 -> Net-(Q5-G)
- Q5 pad 3: Net-(Q5-D) -> Net-(D5-K)
- Q6 pad 1: +5V -> GND
- Q6 pad 2: /READ_1 -> Net-(Q6-G)
- Q6 pad 3: Net-(Q6-D) -> Net-(D6-K)
- Q7 pad 1: +5V -> GND
- Q7 pad 2: /READ_0 -> Net-(Q7-G)
- Q7 pad 3: Net-(Q7-D) -> Net-(D7-K)
- Q8 pad 1: +5V -> GND
- Q8 pad 2: /READ_7 -> Net-(Q8-G)
- Q8 pad 3: Net-(Q8-D) -> Net-(D8-K)
- Q9 pad 1: +5V -> Net-(Q10-D)
- Q9 pad 2: Net-(Q9-G) -> Net-(Q10-G)
- Q9 pad 3: Net-(Q9-D) -> +5V
- R1 pad 2: Net-(Q7-D) -> +5V
- R2 pad 2: Net-(Q6-D) -> +5V
- R3 pad 2: Net-(Q5-D) -> +5V
- R4 pad 2: Net-(Q4-D) -> +5V
- R5 pad 2: Net-(Q3-D) -> +5V
- R6 pad 2: Net-(Q2-D) -> +5V
- R7 pad 2: Net-(Q1-D) -> +5V
- R8 pad 2: Net-(Q8-D) -> +5V
- U1 pad 13: Net-(Q9-D) -> Net-(U1-Pad13)
- U1 pad 9: Net-(Q9-D) -> Net-(U1-Pad13)
- U10 pad 10: Net-(Q11-D) -> Net-(Q10-D)
- U10 pad 2: Net-(Q11-D) -> Net-(Q10-D)
- U13 pad 13: Net-(Q9-D) -> Net-(U13-Pad13)
- U13 pad 9: Net-(Q9-D) -> Net-(U13-Pad13)
- U14 pad 13: Net-(Q9-D) -> Net-(U13-Pad13)
- U14 pad 9: Net-(Q9-D) -> Net-(U13-Pad13)
- U15 pad 13: Net-(Q9-D) -> Net-(U13-Pad13)
- U15 pad 9: Net-(Q9-D) -> Net-(U13-Pad13)
- U16 pad 13: Net-(Q9-D) -> Net-(U13-Pad13)
- U16 pad 9: Net-(Q9-D) -> Net-(U13-Pad13)
- U17 pad 1: Net-(Q10-D) -> Net-(U17-Pad1)
- U17 pad 5: Net-(Q10-D) -> Net-(U17-Pad1)
- U18 pad 1: Net-(Q10-D) -> Net-(U17-Pad1)
- U18 pad 5: Net-(Q10-D) -> Net-(U17-Pad1)
- U19 pad 1: Net-(Q10-D) -> Net-(U17-Pad1)
- U19 pad 5: Net-(Q10-D) -> Net-(U17-Pad1)
- U2 pad 1: Net-(Q10-D) -> Net-(U2-Pad1)
- U2 pad 5: Net-(Q10-D) -> Net-(U2-Pad1)
- U20 pad 1: Net-(Q10-D) -> Net-(U17-Pad1)
- U20 pad 5: Net-(Q10-D) -> Net-(U17-Pad1)
- U21 pad 10: Net-(Q11-D) -> Net-(Q10-D)
- U21 pad 2: Net-(Q11-D) -> Net-(Q10-D)
- U22 pad 10: Net-(Q11-D) -> Net-(Q10-D)
- U22 pad 2: Net-(Q11-D) -> Net-(Q10-D)
- U23 pad 12: Net-(Q9-G) -> Net-(J3-Pin_3)
- U23 pad 13: Net-(Q9-G) -> Net-(J3-Pin_3)
- U23 pad 8: Net-(Q9-G) -> Net-(U23-Pad8)
- U3 pad 13: Net-(Q9-D) -> Net-(U1-Pad13)
- U3 pad 9: Net-(Q9-D) -> Net-(U1-Pad13)
- U4 pad 1: Net-(Q10-D) -> Net-(U2-Pad1)
- U4 pad 5: Net-(Q10-D) -> Net-(U2-Pad1)
- U5 pad 10: Net-(Q11-D) -> Net-(Q10-D)
- U5 pad 2: Net-(Q11-D) -> Net-(Q10-D)
- U6 pad 13: Net-(Q9-D) -> Net-(U1-Pad13)
- U6 pad 9: Net-(Q9-D) -> Net-(U1-Pad13)
- U7 pad 13: Net-(Q9-D) -> Net-(U1-Pad13)
- U7 pad 9: Net-(Q9-D) -> Net-(U1-Pad13)
- U8 pad 1: Net-(Q10-D) -> Net-(U2-Pad1)
- U8 pad 5: Net-(Q10-D) -> Net-(U2-Pad1)
- U9 pad 1: Net-(Q10-D) -> Net-(U2-Pad1)
- U9 pad 5: Net-(Q10-D) -> Net-(U2-Pad1)
Routing:
- net +5V: track 188.2 -> 854.0 mm, vias 25 -> 1
- net Net-(Q9-D): track 220.2 -> 0.00 mm
- net Net-(Q11-D): track 216.7 -> 0.00 mm
- net Net-(U2-Pad1): track 0.00 -> 202.9 mm, vias 0 -> 5
- net Net-(U1-Pad13): track 0.00 -> 176.9 mm, vias 0 -> 4
- net Net-(U17-Pad1): track 0.00 -> 174.7 mm, vias 0 -> 3
- net Net-(U13-Pad13): track 0.00 -> 141.5 mm
- net /WRITE_4: track 171.9 -> 65.6 mm, vias 0 -> 1
- net /WRITE_6: track 195.6 -> 95.0 mm, vias 0 -> 1
- net /WRITE_5: track 176.4 -> 77.4 mm, vias 0 -> 3
- net /WRITE_7: track 217.8 -> 138.8 mm, vias 0 -> 6
- net Net-(U11-Pad11): track 32.8 -> 103.0 mm, vias 0 -> 5
- net Net-(U12-Pad11): track 32.8 -> 100.1 mm, vias 0 -> 4
- net /READ_5: track 247.5 -> 196.7 mm, vias 3 -> 5
- net /READ_6: track 256.9 -> 206.7 mm, vias 2 -> 3
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- added copper zone on F.Cu, net GND
- removed copper zone on F.Cu, net +5V
Other:
- board size 213.4 x 66 mm -> 151.8 x 71.1 mm
