File: pcb/register_file/register_file.kicad_pcb (KiCad board)
At the start: 2 copper layers, 141 parts, among them J1 READ1, J10 REG3_CONTROL, J11 REG0_WRITE, J12 REG1_WRITE, J13 REG2_WRITE, J14 REG3_WRITE, J15 REG1_READ, J16 REG2_READ, J17 REG3_READ, J18 READP, J2 READ2, J3 REG0_READ, J4 WRITE, J5 SELECT, J6 CONTROL, J7 REG0_CONTROL, J8 REG1_CONTROL, J9 REG2_CONTROL, Q1 2N7000, Q10 2N7000, Q11 BS250, Q12 2N7000, Q13 BS250, Q14 2N7000, Q15 BS250, Q16 2N7000, Q17 BS250, Q18 2N7000, Q19 BS250, Q2 BS250, Q20 2N7000, Q21 BS250, Q22 2N7000, Q23 BS250, Q24 2N7000, Q25 BS250, Q26 2N7000, Q27 BS250, Q28 2N7000, Q29 BS250, Q3 BS250, Q30 2N7000, Q31 BS250, Q32 2N7000, Q4 2N7000, Q5 BS250, Q6 2N7000, Q7 BS250, Q8 2N7000, Q9 BS250, U1 74HC00, U10 74HC00, U11 74HC00, U12 74HC00, U13 74HC00, U14 74HC00, U15 74HC00, U16 74HC00, U17 74HC00, U18 74HC00, U19 74HC00, U2 74HC00, U20 74HC00, U21 74HC00, U22 74HC00, U23 74HC00, U24 74HC00, U25 74HC00, U26 74HC00, U27 74HC00, U28 74HC00, U29 74HC00, U3 74HC00, U30 74HC00, U31 74HC00, U32 74HC00, U33 74HC00, U34 74HC00, U35 74HC00, U36 74HC00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

Commit message: V2
Parts:
- added H1: MountingHole_Pad, MountingHole:MountingHole_3.5mm_Pad, F.Cu at (341.0, 108.6)
- added H2: MountingHole_Pad, MountingHole:MountingHole_3.5mm_Pad, F.Cu at (340.4, 151.1)
- added H3: MountingHole_Pad, MountingHole:MountingHole_3.5mm_Pad, F.Cu at (53.3, 108.6)
- added H4: MountingHole_Pad, MountingHole:MountingHole_3.5mm_Pad, F.Cu at (53.3, 151.1)
Routing:
- added copper zone on F.Cu, net +5V
Other:
- board outline added: 299.7 x 55.2 mm
Changed lines of the file:
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@@
     (thickness 1.6)
   )
-  (paper "A4")
+  (paper "A3")
   (layers
     (0 "F.Cu" signal)
@@
     )
   )
+  (footprint "MountingHole:MountingHole_3.5mm_Pad" (layer "F.Cu")
+    (at 340.995 108.585)
+    (descr "Mounting Hole 3.5mm")
+    (tags "mounting hole 3.5mm")
+    (property "Sheetfile" "register_file.kicad_sch")
+    (property "Sheetname" "")
+    (property "ki_description" "Mounting Hole with connection")
+    (property "ki_keywords" "mounting hole")
+    (attr exclude_from_pos_files)
+    (fp_text reference "H1" (at 0 -4.5) (layer "F.SilkS")
+        (effects (font (size 1 1) (thickness 0.15)))
+    )
+    (fp_text value "MountingHole_Pad" (at 0 4.5) (layer "F.Fab")
+        (effects (font (size 1 1) (thickness 0.15)))
+    )
+    (fp_text user "${REFERENCE}" (at 0 0) (layer "F.Fab")
+        (effects (font (size 1 1) (thickness 0.15)))
+    )
+    (fp_circle (center 0 0) (end 3.5 0)
+      (stroke (width 0.15) (type solid)) (fill none) (layer "Cmts.User"))
+    (fp_circle (center 0 0) (end 3.75 0)
+      (stroke (width 0.05) (type solid)) (fill none) (layer "F.CrtYd"))
+    (pad "1" thru_hole circle (at 0 0) (size 7 7) (drill 3.5) (layers "*.Cu" "*.Mask")
+      (net 2 "GND") (pinfunction "1") (pintype "input"))
+  )
   (footprint "Package_DIP:DIP-14_W7.62mm_LongPads" (layer "F.Cu")
     (at -50.905 -84.615)
@@
     )
   )
+  (footprint "MountingHole:MountingHole_3.5mm_Pad" (layer "F.Cu")
+    (at 340.36 151.13)
+    (descr "Mounting Hole 3.5mm")
+    (tags "mounting hole 3.5mm")
+    (property "Sheetfile" "register_file.kicad_sch")
+    (property "Sheetname" "")
+    (property "ki_description" "Mounting Hole with connection")
+    (property "ki_keywords" "mounting hole")
+    (attr exclude_from_pos_files)
+    (fp_text reference "H2" (at 0 -4.5) (layer "F.SilkS")
+        (effects (font (size 1 1) (thickness 0.15)))
+    )
+    (fp_text value "MountingHole_Pad" (at 0 4.5) (layer "F.Fab")
+        (effects (font (size 1 1) (thickness 0.15)))
+    )
+    (fp_text user "${REFERENCE}" (at 0 0) (layer "F.Fab")
+        (effects (font (size 1 1) (thickness 0.15)))
+    )
+    (fp_circle (center 0 0) (end 3.5 0)
+      (stroke (width 0.15) (type solid)) (fill none) (layer "Cmts.User"))
+    (fp_circle (center 0 0) (end 3.75 0)
+      (stroke (width 0.05) (type solid)) (fill none) (layer "F.CrtYd"))
+    (pad "1" thru_hole circle (at 0 0) (size 7 7) (drill 3.5) (layers "*.Cu" "*.Mask")
+      (net 2 "GND") (pinfunction "1") (pintype "input"))
+  )
   (footprint "Package_DIP:DIP-14_W7.62mm_LongPads" (layer "F.Cu")
     (at -74.105 -123.415)
@@
     )
   )
+  (footprint "MountingHole:MountingHole_3.5mm_Pad" (layer "F.Cu")
+    (at 53.34 108.585)
+    (descr "Mounting Hole 3.5mm")
+    (tags "mounting hole 3.5mm")
+    (property "Sheetfile" "register_file.kicad_sch")
+    (property "Sheetname" "")
+    (property "ki_description" "Mounting Hole with connection")
+    (property "ki_keywords" "mounting hole")
+    (attr exclude_from_pos_files)
+    (fp_text reference "H3" (at 0 -4.5) (layer "F.SilkS")
+        (effects (font (size 1 1) (thickness 0.15)))
+    )
+    (fp_text value "MountingHole_Pad" (at 0 4.5) (layer "F.Fab")
+        (effects (font (size 1 1) (thickness 0.15)))
+    )
+    (fp_text user "${REFERENCE}" (at 0 0) (layer "F.Fab")
+        (effects (font (size 1 1) (thickness 0.15)))
+    )
+    (fp_circle (center 0 0) (end 3.5 0)
+      (stroke (width 0.15) (type solid)) (fill none) (layer "Cmts.User"))
+    (fp_circle (center 0 0) (end 3.75 0)
+      (stroke (width 0.05) (type solid)) (fill none) (layer "F.CrtYd"))
+    (pad "1" thru_hole circle (at 0 0) (size 7 7) (drill 3.5) (layers "*.Cu" "*.Mask")
+      (net 2 "GND") (pinfunction "1") (pintype "input"))
+  )
   (footprint "Capacitor_THT:C_Radial_D5.0mm_H11.0mm_P2.00mm" (layer "F.Cu")
     (at -39.865 -5.315)
@@
     )
   )
+  (footprint "MountingHole:MountingHole_3.5mm_Pad" (layer "F.Cu")
+    (at 53.34 151.13)
+    (descr "Mounting Hole 3.5mm")
+    (tags "mounting hole 3.5mm")
+    (property "Sheetfile" "register_file.kicad_sch")
+    (property "Sheetname" "")
+    (property "ki_description" "Mounting Hole with connection")
+    (property "ki_keywords" "mounting hole")
+    (attr exclude_from_pos_files)
+    (fp_text reference "H4" (at 0 -4.5) (layer "F.SilkS")
+        (effects (font (size 1 1) (thickness 0.15)))
+    )
+    (fp_text value "MountingHole_Pad" (at 0 4.5) (layer "F.Fab")
+        (effects (font (size 1 1) (thickness 0.15)))
+    )
+    (fp_text user "${REFERENCE}" (at 0 0) (layer "F.Fab")
+        (effects (font (size 1 1) (thickness 0.15)))
+    )
+    (fp_circle (center 0 0) (end 3.5 0)
+      (stroke (width 0.15) (type solid)) (fill none) (layer "Cmts.User"))
+    (fp_circle (center 0 0) (end 3.75 0)
+      (stroke (width 0.05) (type solid)) (fill none) (layer "F.CrtYd"))
+    (pad "1" thru_hole circle (at 0 0) (size 7 7) (drill 3.5) (layers "*.Cu" "*.Mask")
+      (net 2 "GND") (pinfunction "1") (pintype "input"))
+  )
   (footprint "Connector_IDC:IDC-Header_2x04_P2.54mm_Vertical" (layer "F.Cu")
     (at -104.485 -21.895)
@@
     )
   )
+  (gr_arc (start 346.71 151.13) (mid 344.850128 155.620128) (end 340.36 157.48)
+    (stroke (width 0.1) (type default)) (layer "Edge.Cuts"))
+  (gr_arc (start 46.99 108.585) (mid 48.849872 104.094872) (end 53.34 102.235)
+    (stroke (width 0.1) (type default)) (layer "Edge.Cuts"))
+  (gr_line (start 346.71 108.585) (end 346.71 151.13)
+    (stroke (width 0.1) (type default)) (layer "Edge.Cuts"))
+  (gr_arc (start 53.34 157.48) (mid 48.849872 155.620128) (end 46.99 151.13)
+    (stroke (width 0.1) (type default)) (layer "Edge.Cuts"))
+  (gr_line (start 53.34 102.235) (end 340.36 102.235)
+    (stroke (width 0.1) (type default)) (layer "Edge.Cuts"))
+  (gr_line (start 46.99 108.585) (end 46.99 151.13)
+    (stroke (width 0.1) (type default)) (layer "Edge.Cuts"))
+  (gr_arc (start 340.36 102.235) (mid 344.850128 104.094872) (end 346.71 108.585)
+    (stroke (width 0.1) (type default)) (layer "Edge.Cuts"))
+  (gr_line (start 340.36 157.48) (end 53.34 157.48)
+    (stroke (width 0.1) (type default)) (layer "Edge.Cuts"))
+  (zone (net 1) (net_name "+5V") (layer "F.Cu") (hatch edge 0.5)
+    (connect_pads (clearance 0.5))
+    (min_thickness 0.25) (filled_areas_thickness no)
+    (fill yes (thermal_gap 0.5) (thermal_bridge_width 0.5))
+    (polygon
+      (pts
+        (xy 347.98 101.6)
+        (xy 347.98 160.02)
+        (xy 44.45 158.75)
+        (xy 44.45 99.06)
+      )
+    )
+  )
