File: pcb/register_file/register_file.kicad_sch (KiCad schematic)
At the start: 141 parts, among them J1 READ1, J10 REG3_CONTROL, J11 REG0_WRITE, J12 REG1_WRITE, J13 REG2_WRITE, J14 REG3_WRITE, J15 REG1_READ, J16 REG2_READ, J17 REG3_READ, J18 READP, J2 READ2, J3 REG0_READ, J4 WRITE, J5 SELECT, J6 CONTROL, J7 REG0_CONTROL, J8 REG1_CONTROL, J9 REG2_CONTROL, Q1 2N7000, Q10 2N7000, Q11 BS250, Q12 2N7000, Q13 BS250, Q14 2N7000, Q15 BS250, Q16 2N7000, Q17 BS250, Q18 2N7000, Q19 BS250, Q2 BS250, Q20 2N7000, Q21 BS250, Q22 2N7000, Q23 BS250, Q24 2N7000, Q25 BS250, Q26 2N7000, Q27 BS250, Q28 2N7000, Q29 BS250, Q3 BS250, Q30 2N7000, Q31 BS250, Q32 2N7000, Q4 2N7000, Q5 BS250, Q6 2N7000, Q7 BS250, Q8 2N7000, Q9 BS250, U1 74HC00, U10 74HC00, U11 74HC00, U12 74HC00, U13 74HC00, U14 74HC00, U15 74HC00, U16 74HC00, U17 74HC00, U18 74HC00, U19 74HC00, U2 74HC00, U20 74HC00, U21 74HC00, U22 74HC00, U23 74HC00, U24 74HC00, U25 74HC00, U26 74HC00, U27 74HC00, U28 74HC00, U29 74HC00, U3 74HC00, U30 74HC00, U31 74HC00, U32 74HC00, U33 74HC00, U34 74HC00, U35 74HC00, U36 74HC00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

Commit message: V2
Parts:
- added C3, C4, C48, C49, C50, C51, C52, C53: 100 nF, Capacitor_THT:C_Radial_D5.0mm_H11.0mm_P2.00mm, symbol Device:C_Small
- added H1, H2, H3, H4: MountingHole_Pad, MountingHole:MountingHole_3.5mm_Pad, symbol Mechanical:MountingHole_Pad
- C1, C10, C11, C12, C13, C14, C15, C16, C17, C18, C19, C2, C20, C21, C22, C23, C24, C25, C26, C27, C28, C29, C30, C31, C32, C33, C34, C35, C36, C37, C38, C39, C40, C41, C42, C43, C44, C45, C46, C47, C5, C6, C7, C8, C9: value C_Small -> 100 nF
Connections:
- net +5V: now also C45.2, C3.1, C4.1, C48.1, C49.1, C50.1, C51.2, C52.2, C53.2; no longer C45.1
- net GND: now also C45.1, C3.2, C4.2, C48.2, C49.2, C50.2, C51.1, C52.1, C53.1, H1.1, H2.1, H3.1, H4.1; no longer C45.2
