File: hardware/register/register.kicad_sch (KiCad schematic)
At the start: 91 parts, among them J1 Conn_02x04_Odd_Even, J2 Conn_02x04_Odd_Even, J3 Conn_02x04_Odd_Even, Q1 BS170, Q10 BS170, Q11 BS170, Q2 BS170, Q3 BS170, Q4 BS170, Q5 BS170, Q6 BS170, Q7 BS170, Q8 BS170, Q9 BS170, U1 74HC00, U10 74HC00, U11 74HC00, U12 74HC00, U13 74HC00, U14 74HC00, U15 74HC00, U16 74LS00, U17 74HC00, U18 74HC00, U19 74HC00, U2 74HC00, U20 74HC00, U21 74HC00, U22 74HC00, U23 74HC00, U24 74HC00, U25 74HC00, U3 74HC00, U4 74HC00, U5 74HC00, U6 74HC00, U7 74HC00, U8 74HC00, U9 74HC00

Commit message: redesigned register PCB with SMD components
Parts:
- removed H1: MountingHole_Pad, MountingHole:MountingHole_2.2mm_M2_Pad, symbol Mechanical:MountingHole_Pad
- removed Q1, Q10, Q11, Q2, Q3, Q4, Q5, Q6, Q7, Q8, Q9: BS170, Package_TO_SOT_THT:TO-92_Inline_Wide, symbol Transistor_FET:BS170
- added Q1, Q10, Q11, Q12, Q13, Q14, Q2, Q3, Q4, Q5, Q6, Q7, Q8, Q9: IRLML6244, Package_TO_SOT_SMD:SOT-23_Handsoldering, symbol Transistor_FET:IRLML6244
- added R13, R14, R15: 400, Resistor_SMD:R_1206_3216Metric_Pad1.30x1.75mm_HandSolder, symbol Device:R
- D1, D10, D11, D12, D2, D3, D4, D5, D6, D7, D8, D9: footprint LED_THT:LED_D3.0mm -> LED_SMD:LED_1206_3216Metric_Pad1.42x1.75mm_HandSolder
- R1, R10, R11, R12, R2, R3, R4, R5, R6, R7, R8, R9: value 200 -> 400; footprint Resistor_THT:R_Axial_DIN0207_L6.3mm_D2.5mm_P7.62mm_Horizontal -> Resistor_SMD:R_1206_3216Metric_Pad1.30x1.75mm_HandSolder
Connections:
- net +5V: now also Q1.3 (D), Q10.3 (D), Q11.3 (D), Q12.3 (D), Q13.3 (D), Q14.3 (D), Q2.3 (D), Q3.3 (D), Q4.3 (D), Q5.3 (D), Q6.3 (D), Q7.3 (D), Q8.3 (D), Q9.3 (D)
- net GND: now also R13.2, R14.2, R15.2
- net at D9.2 (A), J3.6 (Pin_6): now also Q8.2 (S)
- net at U1.9, U11.9, U12.10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: now also R2.1, Q1.2 (S); no longer D2.2 (A)
- net at R1.1: now also U1.2, U11.2, U12.1, U14.2, U15.1, U18.2, U19.1, U2.1, U21.2, U22.1, U24.2, U25.1, U5.2, U6.1, U8.2, U9.1, Q12.2 (S); no longer D1.1 (K)
- net at U18.11, U19.12: now also Q8.1 (G)
- net at D6.2 (A), J3.3 (Pin_3): now also Q5.2 (S)
- net at U10.5, U13.5, U17.5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: now also R3.1, Q2.2 (S); no longer D3.2 (A)
- net at U14.11, U15.12: now also Q7.1 (G)
- net at U16.12, U16.13, U16.8: now also Q12.1 (G)
- net at U21.11, U22.12: now also Q9.1 (G)
- net at D4.2 (A), J3.1 (Pin_1): now also Q3.2 (S)
- net at D5.2 (A), J3.2 (Pin_2): now also Q4.2 (S)
- net at D7.2 (A), J3.4 (Pin_4): now also Q6.2 (S)
- net at D8.2 (A), J3.5 (Pin_5): now also Q7.2 (S)
- net at D10.2 (A), J3.7 (Pin_7): now also Q9.2 (S)
- net at D11.2 (A), J3.8 (Pin_8): now also Q10.2 (S)
- net at U11.11, U12.12: now also Q6.1 (G)
- net at U8.11, U9.12: now also Q5.1 (G)
- net at D3.1 (K): now also R15.1; no longer R3.1
- net WEN: now reaches J1.1 (Pin_1), U16.2
- net WEN: now also Q13.1 (G)
- net !CLR: now reaches J1.3 (Pin_3), U16.1
- net !CLR: now also Q14.1 (G), Q2.1 (G)
- net CLK: now reaches J1.4 (Pin_4), U16.10
- net CLK: now also Q11.1 (G)
- net at U5.11, U6.12: now also Q4.1 (G)
- net at U1.11, U2.12: now also Q3.1 (G)
- net at U24.11, U25.12: now also Q10.1 (G)
- net at U16.11: now also Q1.1 (G)
- net at D2.1 (K): now also R14.1; no longer R2.1
- new net: D3.2 (A), Q14.2 (S)
- new net: D1.1 (K), R13.1
- new net: D1.2 (A), Q11.2 (S)
- new net: D2.2 (A), Q13.2 (S)
Other:
- moved on the sheet: C25, J1, U16E
