File: hardware/register/register.kicad_sch (KiCad schematic)
At the start: 123 parts, among them J1 Conn_02x04_Odd_Even, J2 Conn_02x04_Odd_Even, J3 Conn_02x04_Odd_Even, Q1 IRLML6244, Q10 IRLML6244, Q11 IRLML6244, Q12 IRLML6244, Q13 IRLML6244, Q14 IRLML6244, Q2 IRLML6244, Q3 IRLML6244, Q4 IRLML6244, Q5 IRLML6244, Q6 IRLML6244, Q7 IRLML6244, Q8 IRLML6244, Q9 IRLML6244, U1 74HC00, U10 74HC00, U11 74HC00, U12 74HC00, U13 74HC00, U14 74HC00, U15 74HC00, U16 74HC00, U17 74HC00, U18 74HC00, U19 74HC00, U2 74HC00, U20 74HC00, U21 74HC00, U22 74HC00, U23 74HC00, U24 74HC00, U25 74HC00, U3 74HC00, U4 74HC00, U5 74HC00, U6 74HC00, U7 74HC00, U8 74HC00, U9 74HC00

Commit message: redesigned register using SMD components
Parts:
- removed H2: MountingHole_Pad, MountingHole:MountingHole_2.2mm_M2_Pad, symbol Mechanical:MountingHole_Pad
- removed J1, J2, J3: Conn_02x04_Odd_Even, Connector_PinHeader_2.54mm:PinHeader_2x04_P2.54mm_Horizontal, symbol Connector_Generic:Conn_02x04_Odd_Even
- added C26, C27: 10uF, Capacitor_SMD:C_0603_1608Metric_Pad1.08x0.95mm_HandSolder, symbol Device:C
- added J4: Conn_02x16_Odd_Even, Connector_PinHeader_2.54mm:PinHeader_2x16_P2.54mm_Horizontal, symbol Connector_Generic:Conn_02x16_Odd_Even
- C1, C10, C11, C12, C13, C14, C15, C16, C17, C18, C19, C2, C20, C21, C22, C23, C24, C25, C3, C4, C5, C6, C7, C8, C9: value 100nF -> 330nF; footprint Capacitor_SMD:C_1206_3216Metric_Pad1.33x1.80mm_HandSolder -> Capacitor_SMD:C_0603_1608Metric_Pad1.08x0.95mm_HandSolder; LCSC C920964 -> C2918485
- D1, D10, D11, D12, D2, D3, D4, D5, D6, D7, D8, D9: footprint LED_SMD:LED_1206_3216Metric_Pad1.42x1.75mm_HandSolder -> LED_SMD:LED_0603_1608Metric_Pad1.05x0.95mm_HandSolder; LCSC C6577912 -> C84267
- R1, R2, R3: footprint Resistor_SMD:R_1206_3216Metric_Pad1.30x1.75mm_HandSolder -> Resistor_SMD:R_0603_1608Metric_Pad0.98x0.95mm_HandSolder; LCSC C4410 -> C21190
- R10, R11, R12, R13, R14, R15, R4, R5, R6, R7, R8, R9: value 100 -> 1000; footprint Resistor_SMD:R_1206_3216Metric_Pad1.30x1.75mm_HandSolder -> Resistor_SMD:R_0603_1608Metric_Pad0.98x0.95mm_HandSolder; LCSC C17901 -> C21190
Connections:
- net !CLR: now also J4.29 (Pin_29)
- net +5V: now also C26.1, C27.1, J4.24 (Pin_24), J4.26 (Pin_26), J4.28 (Pin_28), J4.30 (Pin_30)
- net CLK: now also J4.25 (Pin_25)
- net GND: now also C26.2, C27.2, J4.1 (Pin_1), J4.11 (Pin_11), J4.12 (Pin_12), J4.2 (Pin_2), J4.21 (Pin_21), J4.22 (Pin_22), J4.23 (Pin_23), J4.31 (Pin_31), J4.32 (Pin_32)
- net WEN: now also J4.27 (Pin_27)
- net at D9.2 (A), Q8.2 (S): now also J4.8 (Pin_8)
- net at TP6.1, U17.1, U17.2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: now also J4.18 (Pin_18)
- net at D5.2 (A), Q4.2 (S): now also J4.4 (Pin_4)
- net at D10.2 (A), Q9.2 (S): now also J4.9 (Pin_9)
- net at TP1.1, U1.1, U3.1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: now also J4.13 (Pin_13)
- net at D6.2 (A), Q5.2 (S): now also J4.5 (Pin_5)
- net at D4.2 (A), Q3.2 (S): now also J4.3 (Pin_3)
- net at D7.2 (A), Q6.2 (S): now also J4.6 (Pin_6)
- net at D8.2 (A), Q7.2 (S): now also J4.7 (Pin_7)
- net at D11.2 (A), Q10.2 (S): now also J4.10 (Pin_10)
- net at TP4.1, U10.1, U10.2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: now also J4.16 (Pin_16)
- net at TP5.1, U13.1, U13.2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: now also J4.17 (Pin_17)
- net at TP2.1, U4.1, U4.2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: now also J4.14 (Pin_14)
- net at TP7.1, U20.1, U20.2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: now also J4.19 (Pin_19)
- net at TP3.1, U7.1, U7.2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: now also J4.15 (Pin_15)
- net at TP8.1, U23.1, U23.2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: now also J4.20 (Pin_20)
Other:
- moved on the sheet: C25, D1, D12, D2, D3, Q11, Q13, Q14, U16E
