File: hardware/register/register.kicad_sch (KiCad schematic)
At the start: 122 parts, among them J4 Conn_02x16_Odd_Even, Q1 IRLML6244, Q10 IRLML6244, Q11 IRLML6244, Q12 IRLML6244, Q13 IRLML6244, Q14 IRLML6244, Q2 IRLML6244, Q3 IRLML6244, Q4 IRLML6244, Q5 IRLML6244, Q6 IRLML6244, Q7 IRLML6244, Q8 IRLML6244, Q9 IRLML6244, U1 74HC00, U10 74HC00, U11 74HC00, U12 74HC00, U13 74HC00, U14 74HC00, U15 74HC00, U16 74HC00, U17 74HC00, U18 74HC00, U19 74HC00, U2 74HC00, U20 74HC00, U21 74HC00, U22 74HC00, U23 74HC00, U24 74HC00, U25 74HC00, U3 74HC00, U4 74HC00, U5 74HC00, U6 74HC00, U7 74HC00, U8 74HC00, U9 74HC00

Commit message: did a good chunk of IO PCB schematic
Connections:
- net R5: now reaches D9.2 (A), J4.8 (Pin_8), Q8.2 (S)
- net W5: now reaches J4.18 (Pin_18), TP6.1, U17.1, U17.2, U18.1
- net R1: now reaches D5.2 (A), J4.4 (Pin_4), Q4.2 (S)
- net R6: now reaches D10.2 (A), J4.9 (Pin_9), Q9.2 (S)
- net W0: now reaches J4.13 (Pin_13), TP1.1, U1.1, U3.1, U3.2
- net R2: now reaches D6.2 (A), J4.5 (Pin_5), Q5.2 (S)
- net R7: now reaches D11.2 (A), J4.10 (Pin_10), Q10.2 (S)
- net W1: now reaches J4.14 (Pin_14), TP2.1, U4.1, U4.2, U5.1
- net W2: now reaches J4.15 (Pin_15), TP3.1, U7.1, U7.2, U8.1
- net W3: now reaches J4.16 (Pin_16), TP4.1, U10.1, U10.2, U11.1
- net W4: now reaches J4.17 (Pin_17), TP5.1, U13.1, U13.2, U14.1
- net W6: now reaches J4.19 (Pin_19), TP7.1, U20.1, U20.2, U21.1
- net W7: now reaches J4.20 (Pin_20), TP8.1, U23.1, U23.2, U24.1
- net R0: now reaches D4.2 (A), J4.3 (Pin_3), Q3.2 (S)
- net R3: now reaches D7.2 (A), J4.6 (Pin_6), Q6.2 (S)
- net R4: now reaches D8.2 (A), J4.7 (Pin_7), Q7.2 (S)
Changed lines of the file:
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@@
+		)
+	)
+	(label "W5"
+		(at 111.76 53.34 0)
+		(effects
+			(font
+				(size 1.27 1.27)
+			)
+			(justify left bottom)
+		)
+	)
+	(label "W1"
+		(at 111.76 58.42 0)
+		(effects
+			(font
+				(size 1.27 1.27)
+			)
+			(justify left bottom)
+		)
+	)
+	(label "W4"
+		(at 133.35 53.34 0)
+		(effects
+			(font
+				(size 1.27 1.27)
+			)
+			(justify left bottom)
+		)
+	)
+	(label "R3"
+		(at 111.76 68.58 0)
+		(effects
+			(font
+				(size 1.27 1.27)
+			)
+			(justify left bottom)
+		)
+	)
+	(label "W2"
+		(at 133.35 55.88 0)
+		(effects
+			(font
+				(size 1.27 1.27)
+			)
+			(justify left bottom)
+		)
+	)
+	(label "R6"
+		(at 133.35 63.5 0)
+		(effects
+			(font
+				(size 1.27 1.27)
+			)
+			(justify left bottom)
+		)
+	)
+	(label "R5"
+		(at 111.76 66.04 0)
+		(effects
+			(font
+				(size 1.27 1.27)
+			)
+			(justify left bottom)
+		)
+	)
+	(label "W0"
+		(at 133.35 58.42 0)
+		(effects
+			(font
+				(size 1.27 1.27)
+			)
+			(justify left bottom)
+		)
+	)
+	(label "W3"
+		(at 111.76 55.88 0)
+		(effects
+			(font
+				(size 1.27 1.27)
+			)
+			(justify left bottom)
 		)
 	)
@@
 		)
 	)
+	(label "R2"
+		(at 133.35 68.58 0)
+		(effects
+			(font
+				(size 1.27 1.27)
+			)
+			(justify left bottom)
+		)
+	)
+	(label "R0"
+		(at 133.35 71.12 0)
+		(effects
+			(font
+				(size 1.27 1.27)
+			)
+			(justify left bottom)
+		)
+	)
+	(label "W7"
+		(at 111.76 50.8 0)
+		(effects
+			(font
+				(size 1.27 1.27)
+			)
+			(justify left bottom)
+		)
+	)
 	(label "CLK"
 		(at 218.44 49.53 0)
@@
 		)
 	)
+	(label "CLK"
+		(at 133.35 43.18 0)
+		(effects
+			(font
+				(size 1.27 1.27)
+			)
+			(justify left bottom)
+		)
+	)
+	(label "R4"
+		(at 133.35 66.04 0)
+		(effects
+			(font
+				(size 1.27 1.27)
+			)
+			(justify left bottom)
+		)
+	)
+	(label "!CLR"
+		(at 137.16 38.1 180)
+		(effects
+			(font
+				(size 1.27 1.27)
+			)
+			(justify right bottom)
+		)
+	)
+	(label "R1"
+		(at 111.76 71.12 0)
+		(effects
+			(font
+				(size 1.27 1.27)
+			)
+			(justify left bottom)
+		)
+	)
+	(label "WEN"
+		(at 137.16 40.64 180)
+		(effects
+			(font
+				(size 1.27 1.27)
+			)
+			(justify right bottom)
+		)
+	)
+	(label "R7"
+		(at 111.76 63.5 0)
+		(effects
+			(font
+				(size 1.27 1.27)
+			)
+			(justify left bottom)
+		)
+	)
 	(label "!CLR"
 		(at 226.06 39.37 180)
@@
 		)
 	)
+	(label "W6"
+		(at 133.35 50.8 0)
+		(effects
+			(font
+				(size 1.27 1.27)
+			)
+			(justify left bottom)
+		)
+	)
