File: hardware/alu_add_sub/alu_add_sub.kicad_sch (KiCad schematic)
At the start: 158 parts, among them J1 Conn_02x22_Odd_Even, Q1 IRLML6244, Q10 IRLML6244, Q11 IRLML6244, Q12 IRLML6244, Q13 IRLML6244, Q14 IRLML6244, Q15 IRLML6244, Q16 IRLML6244, Q17 IRLML6244, Q18 IRLML6244, Q19 IRLML6244, Q2 IRLML6244, Q20 IRLML6244, Q21 IRLML6244, Q22 IRLML6244, Q23 IRLML6244, Q24 IRLML6244, Q25 IRLML6244, Q26 IRLML6244, Q27 IRLML6244, Q28 IRLML6244, Q3 IRLML6244, Q4 IRLML6244, Q5 IRLML6244, Q6 IRLML6244, Q7 IRLML6244, Q8 IRLML6244, Q9 IRLML6244, U1 74HC00, U10 74HC00, U11 74HC00, U12 74HC00, U13 74HC00, U14 74HC00, U15 74HC00, U16 74HC00, U17 74HC00, U18 74HC00, U19 74HC00, U2 74HC00, U20 74HC00, U21 74HC00, U22 74HC00, U23 74HC00, U24 74HC00, U25 74HC00, U26 74HC00, U27 74HC00, U28 74HC00, U29 74HC00, U3 74HC00, U30 74HC00, U31 74HC00, U32 74HC00, U33 74HC00, U34 74HC00, U35 74HC00, U4 74HC00, U5 74HC00, U6 74HC00, U7 74HC00, U8 74HC00, U9 74HC00

Commit message: layout done for alu add sub (missing test points)
Parts:
- added D29: LED, LED_SMD:LED_0603_1608Metric_Pad1.05x0.95mm_HandSolder, symbol Device:LED
- added H3, H4: MountingHole_Pad, MountingHole:MountingHole_2.2mm_M2_Pad, symbol Mechanical:MountingHole_Pad
- added R29: 1000, Resistor_SMD:R_0603_1608Metric_Pad0.98x0.95mm_HandSolder, symbol Device:R
- C1, C10, C11, C12, C13, C14, C15, C16, C17, C18, C19, C2, C20, C21, C22, C23, C24, C25, C26, C27, C28, C29, C3, C30, C31, C32, C33, C34, C35, C36, C37, C38, C4, C5, C6, C7, C8, C9: footprint (none) -> Capacitor_SMD:C_0603_1608Metric_Pad1.08x0.95mm_HandSolder
- D1, D10, D11, D12, D13, D14, D15, D16, D17, D18, D19, D2, D20, D21, D22, D23, D24, D25, D26, D27, D28, D3, D4, D5, D6, D7, D8, D9: footprint (none) -> LED_SMD:LED_0603_1608Metric_Pad1.05x0.95mm_HandSolder
- J1: footprint (none) -> Connector_PinHeader_2.54mm:PinHeader_2x22_P2.54mm_Horizontal
- Q1, Q10, Q11, Q12, Q13, Q14, Q15, Q16, Q17, Q18, Q19, Q2, Q20, Q21, Q22, Q23, Q24, Q25, Q26, Q27, Q28, Q3, Q4, Q5, Q6, Q7, Q8, Q9: footprint Package_TO_SOT_SMD:SOT-23 -> Package_TO_SOT_SMD:SOT-23_Handsoldering
- R1, R10, R11, R12, R13, R14, R15, R16, R17, R18, R19, R2, R20, R21, R22, R23, R24, R25, R26, R27, R28, R3, R4, R5, R6, R7, R8, R9: footprint (none) -> Resistor_SMD:R_0603_1608Metric_Pad0.98x0.95mm_HandSolder
- U1, U10, U11, U12, U13, U14, U15, U16, U17, U18, U19, U2, U20, U21, U22, U23, U24, U25, U26, U27, U28, U29, U3, U30, U31, U32, U33, U34, U35, U4, U5, U6, U7, U8, U9: footprint (none) -> Package_SO:SOIC-14_3.9x8.7mm_P1.27mm
Connections:
- net +5V: now also D29.2 (A)
- net GND: now also H3.1, H4.1, R29.2
- new net: D29.1 (K), R29.1
