File: hardware/alu_add_sub/alu_add_sub.kicad_sch (KiCad schematic)
At the start: 186 parts, among them J1 Conn_02x22_Odd_Even, Q1 IRLML6244, Q10 IRLML6244, Q11 IRLML6244, Q12 IRLML6244, Q13 IRLML6244, Q14 IRLML6244, Q15 IRLML6244, Q16 IRLML6244, Q17 IRLML6244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

Commit message: finished design of ALU binary logic module
Parts:
- J1: now not fitted
Changed lines of the file:
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@@
 		(in_bom no)
 		(on_board yes)
-		(dnp no)
+		(dnp yes)
 		(fields_autoplaced yes)
 		(property "Reference" "J1"
