File: hardware/alu_bitops/alu_bitops.kicad_sch (KiCad schematic)
At the start: 230 parts, among them J1 Conn_02x21_Odd_Even, Q1 IRLML6244, Q10 IRLML6244, Q11 IRLML6244, Q12 IRLML6244, Q13 IRLML6244, Q14 IRLML6244, Q15 IRLML6244, Q16 IRLML6244, Q17 IRLML6244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

Commit message: added 8 bit mux pcb, started work on ALU shifter
Parts:
- U1, U10, U11, U12, U13, U14, U15, U16, U17, U18, U19, U2, U20, U21, U22, U23, U24, U25, U26, U27, U28, U29, U3, U30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: LCSC (none) -> C5586
