File: hardware/alu_motherboard/alu_motherboard.kicad_sch (KiCad schematic)
At the start: 43 parts, among them J1 OUT, J3 ADD_SUB, J4 BITOPS, J5 SHIFT, J6 IN, Q3 IRLML6244, Q4 IRLML6244, Q5 IRLML6244, Q6 IRLML6244, U2 74HC00, U3 74HC00, U4 74HC00, U5 74HC00, U53 74HC00, U6 74HC00

Commit message: fixed schematic of ALU motherboard
Parts:
- removed J1: OUT, Connector_PinHeader_2.54mm:PinHeader_2x15_P2.54mm_Horizontal, symbol Connector_Generic:Conn_02x15_Odd_Even
- removed J6: IN, Connector_PinHeader_2.54mm:PinHeader_2x15_P2.54mm_Horizontal, symbol Connector_Generic:Conn_02x15_Odd_Even
- added J2: Conn_02x26_Odd_Even, Connector_PinHeader_2.54mm:PinHeader_2x26_P2.54mm_Horizontal, symbol Connector_Generic:Conn_02x26_Odd_Even
Connections:
- net +5V: now also J2.44 (Pin_44), J2.46 (Pin_46), J2.47 (Pin_47), J2.48 (Pin_48), J2.49 (Pin_49), J2.50 (Pin_50)
- net A0: now also J2.3 (Pin_3); no longer J3.41 (Pin_41), J4.20 (Pin_20)
- net A1: now also J2.5 (Pin_5)
- net A2: now also J2.7 (Pin_7)
- net A3: now also J2.9 (Pin_9)
- net A4: now also J2.13 (Pin_13)
- net A5: now also J2.15 (Pin_15)
- net A6: now also J2.17 (Pin_17)
- net A7: now also J2.19 (Pin_19)
- net ASS: now also J2.39 (Pin_39)
- net B0: now also J2.4 (Pin_4)
- net B1: now also J2.6 (Pin_6)
- net B2: now also J2.8 (Pin_8)
- net B3: now also J2.10 (Pin_10)
- net B4: now also J2.14 (Pin_14)
- net B5: now also J2.16 (Pin_16)
- net B6: now also J2.18 (Pin_18)
- net CEN: now also J2.35 (Pin_35)
- net CIN: now also J2.33 (Pin_33)
- net COUT: now also J2.27 (Pin_27)
- net GND: now also J2.1 (Pin_1), J2.11 (Pin_11), J2.12 (Pin_12), J2.2 (Pin_2), J2.21 (Pin_21), J2.22 (Pin_22), J2.31 (Pin_31), J2.32 (Pin_32), J2.37 (Pin_37), J2.42 (Pin_42), J2.45 (Pin_45), J2.51 (Pin_51), J2.52 (Pin_52)
- net NEG: now also J2.25 (Pin_25)
- net OP1: now also U5.4, U5.5, J2.41 (Pin_41); no longer U5.1, U5.2
- net OP2: now also U5.1, U5.2, J2.43 (Pin_43); no longer U5.4, U5.5
- net OVF: now also J2.29 (Pin_29)
- net RES0: now also D8.2 (A), J2.24 (Pin_24); no longer D1.2 (A)
- net RES1: now also D7.2 (A), J2.26 (Pin_26); no longer D2.2 (A)
- net RES2: now also D6.2 (A), J2.28 (Pin_28); no longer D3.2 (A)
- net RES3: now also D5.2 (A), J2.30 (Pin_30); no longer D4.2 (A)
- net RES4: now also D4.2 (A), J2.34 (Pin_34); no longer D5.2 (A)
- net RES5: now also D3.2 (A), J2.36 (Pin_36); no longer D6.2 (A)
- net RES6: now also D2.2 (A), J2.38 (Pin_38); no longer D7.2 (A)
- net RES7: now also D1.2 (A), J2.40 (Pin_40); no longer D8.2 (A)
- net ZERO: now also J2.23 (Pin_23)
- new net B7: J2.20 (Pin_20), J3.41 (Pin_41), J4.20 (Pin_20)
Other:
- moved on the sheet: C17, C18, C19, C20, C21, C22, C23, C24, C25, C26, C27, D1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

Commit message: finished schematic and draft of ALU motherboard
Parts:
- added D13, D14, D15, D16, D17, D18, D19, D20: LED, LED_SMD:LED_0603_1608Metric_Pad1.05x0.95mm_HandSolder, symbol Device:LED
- added Q10, Q11, Q12, Q13, Q14, Q15, Q16, Q9: IRLML6244, Package_TO_SOT_SMD:SOT-23-3, symbol Transistor_FET:IRLML6244
- added R12, R13, R14, R15, R16, R17, R18, R19: 1000, Resistor_SMD:R_0603_1608Metric_Pad0.98x0.95mm_HandSolder, symbol Device:R
- Q3, Q4, Q5, Q6: footprint Package_TO_SOT_SMD:SOT-23_Handsoldering -> Package_TO_SOT_SMD:SOT-23-3
- U2, U3, U4, U5, U6: footprint (none) -> Package_SO:SOIC-14_3.9x8.7mm_P1.27mm
- U6: renamed from U53; footprint (none) -> Package_SO:SOIC-14_3.9x8.7mm_P1.27mm
Connections:
- net +5V: now also Q10.3 (D), Q11.3 (D), Q12.3 (D), Q13.3 (D), Q14.3 (D), Q15.3 (D), Q16.3 (D), Q9.3 (D)
- net CIN: no longer J3.42 (Pin_42), U6.6
- net COUT: no longer J3.36 (Pin_36), U2.5
- net GND: now also R12.2, R13.2, R14.2, R15.2, R16.2, R17.2, R18.2, R19.2
- net OVF: no longer J3.34 (Pin_34), U4.5
- net ASS renamed AASS
- net B0 renamed ABY0
- net B1 renamed ABY1
- net B2 renamed ABY2
- net OP1 renamed BS1
- removed net RES0: D8.2 (A), J2.24 (Pin_24), J3.4 (Pin_4), J4.3 (Pin_3), J5.3 (Pin_3)
- removed net RES1: D7.2 (A), J2.26 (Pin_26), J3.6 (Pin_6), J4.4 (Pin_4), J5.4 (Pin_4)
- removed net RES2: D6.2 (A), J2.28 (Pin_28), J3.8 (Pin_8), J4.5 (Pin_5), J5.5 (Pin_5)
- removed net RES3: D5.2 (A), J2.30 (Pin_30), J3.10 (Pin_10), J4.6 (Pin_6), J5.6 (Pin_6)
- removed net RES4: D4.2 (A), J2.34 (Pin_34), J3.14 (Pin_14), J4.7 (Pin_7), J5.7 (Pin_7)
- removed net RES5: D3.2 (A), J2.36 (Pin_36), J3.16 (Pin_16), J4.8 (Pin_8), J5.8 (Pin_8)
- removed net RES6: D2.2 (A), J2.38 (Pin_38), J3.18 (Pin_18), J4.9 (Pin_9), J5.9 (Pin_9)
- removed net RES7: D1.2 (A), J2.40 (Pin_40), J3.20 (Pin_20), J4.10 (Pin_10), J5.10 (Pin_10), Q6.1 (G)
- net SOB renamed ASOB
- new net: D19.1 (K), R18.1
- new net: D18.1 (K), R17.1
- new net: D20.1 (K), R19.1
- new net: D15.1 (K), R14.1
- new net: D14.1 (K), R13.1
- new net: D16.1 (K), R15.1
- new net: D17.1 (K), R16.1
- new net: D13.1 (K), R12.1
- new net 8Bit_Mux1/RES0: Q9.1 (G)
- new net 8Bit_Mux1/RES1: Q10.1 (G)
- new net 8Bit_Mux1/RES2: Q11.1 (G)
- new net 8Bit_Mux1/RES3: Q12.1 (G)
- new net 8Bit_Mux1/RES4: Q13.1 (G)
- new net 8Bit_Mux1/RES5: Q14.1 (G)
- new net 8Bit_Mux1/RES6: Q15.1 (G)
- new net 8Bit_Mux1/RES7: Q16.1 (G), Q6.1 (G)
- new net ACIN: J3.42 (Pin_42), U6.6
- new net ACOUT: J3.36 (Pin_36), U2.5
- new net AOVF: J3.34 (Pin_34), U4.5
- new net ARES0: J3.4 (Pin_4)
- new net ARES1: J3.6 (Pin_6)
- new net ARES2: J3.8 (Pin_8)
- new net ARES3: J3.10 (Pin_10)
- new net ARES4: J3.14 (Pin_14)
- new net ARES5: J3.16 (Pin_16)
- new net ARES6: J3.18 (Pin_18)
- new net ARES7: J3.20 (Pin_20)
- new net BRES0: J4.3 (Pin_3)
- new net BRES1: J4.4 (Pin_4)
- new net BRES2: J4.5 (Pin_5)
- new net BRES3: J4.6 (Pin_6)
- new net BRES4: J4.7 (Pin_7)
- new net BRES5: J4.8 (Pin_8)
- new net BRES6: J4.9 (Pin_9)
- new net BRES7: J4.10 (Pin_10)
- new net ORES0: D13.2 (A), D8.2 (A), J2.24 (Pin_24), Q9.2 (S)
- new net ORES1: D14.2 (A), D7.2 (A), J2.26 (Pin_26), Q10.2 (S)
- new net ORES2: D15.2 (A), D6.2 (A), J2.28 (Pin_28), Q11.2 (S)
- new net ORES3: D16.2 (A), D5.2 (A), J2.30 (Pin_30), Q12.2 (S)
- new net ORES4: D17.2 (A), D4.2 (A), J2.34 (Pin_34), Q13.2 (S)
- new net ORES5: D18.2 (A), D3.2 (A), J2.36 (Pin_36), Q14.2 (S)
- new net ORES6: D19.2 (A), D2.2 (A), J2.38 (Pin_38), Q15.2 (S)
- new net ORES7: D1.2 (A), D20.2 (A), J2.40 (Pin_40), Q16.2 (S)
- new net SRES0: J5.3 (Pin_3)
- new net SRES1: J5.4 (Pin_4)
- new net SRES2: J5.5 (Pin_5)
- new net SRES3: J5.6 (Pin_6)
- new net SRES4: J5.7 (Pin_7)
- new net SRES5: J5.8 (Pin_8)
- new net SRES6: J5.9 (Pin_9)
- new net SRES7: J5.10 (Pin_10)
Other:
- moved on the sheet: D1, D2, D3, D4, D5, D6, D7, D8, R4, U5D
