File: hardware/alu_shift/mux.kicad_sch (KiCad schematic)
At the start: 22 parts, among them Q1 IRLML6244, Q2 IRLML6244, U2 74HC00, U3 74HC00, U4 74HC00, U5 74HC00, U6 74HC00, U7 74HC00, U8 74HC00, U9 74HC00

Commit message: added LED indicators for ALU shift module
Parts:
- renumbered C2 to C42, C3 to C43, C4 to C44, C5 to C45, C6 to C46, C7 to C47, C8 to C48, C9 to C49, D1 to D6, Q1 to Q11, Q2 to Q12, R1 to R16, R2 to R17, R3 to R18, U2 to U42, U3 to U43, U4 to U44, U5 to U45, U6 to U46, U7 to U47, U8 to U48, U9 to U49

Commit message: added 8 bit mux pcb, started work on ALU shifter
Parts:
- removed C42, C43, C44, C45, C46, C47, C48, C49: 330nF, Capacitor_SMD:C_0603_1608Metric_Pad1.08x0.95mm_HandSolder, symbol Device:C
- removed D6: LED, LED_SMD:LED_0603_1608Metric_Pad1.05x0.95mm_HandSolder, symbol Device:LED
- removed Q11, Q12: IRLML6244, Package_TO_SOT_SMD:SOT-23_Handsoldering, symbol Transistor_FET:IRLML6244
- removed R16, R17, R18: 1000, Resistor_SMD:R_0603_1608Metric_Pad0.98x0.95mm_HandSolder, symbol Device:R
- removed U42, U43, U44, U45, U46, U47, U48, U49: 74HC00, Package_SO:SOIC-14_3.9x8.7mm_P1.27mm, symbol 74xx:74HC00
- added C10, C11, C4, C5, C6, C7, C8, C9: 330nF, Capacitor_SMD:C_0603_1608Metric_Pad1.08x0.95mm_HandSolder, symbol Device:C
- added Q22, Q23: IRLML6244, Package_TO_SOT_SMD:SOT-23-3, symbol Transistor_FET:IRLML6244
- added R22, R23, R24: 1000, Resistor_SMD:R_0603_1608Metric_Pad0.98x0.95mm_HandSolder, symbol Device:R
- added U2, U3, U4, U5, U6, U7, U8, U9: 74HC00, Package_SO:SOIC-14_3.9x8.7mm_P1.27mm, symbol 74xx:74HC00
Connections:
- net +5V: now also C10.1, C11.1, C4.1, C5.1, C6.1, C7.1, C8.1, C9.1, Q23.3 (D), R22.1, U2.14 (VCC), U3.14 (VCC), U4.14 (VCC), U5.14 (VCC), U6.14 (VCC), U7.14 (VCC), U8.14 (VCC), U9.14 (VCC)
- net A0: now also U2.9
- net A1: now also U3.9
- net A2: now also U4.9
- net A3: now also U5.9
- net A4: now also U6.9
- net A5: now also U7.9
- net A6: now also U8.9
- net A7: now also U9.9
- net B0: now also U2.1
- net B1: now also U3.1
- net B2: now also U4.1
- net B3: now also U5.1
- net B4: now also U6.1
- net B5: now also U7.1
- net B6: now also U8.1
- net B7: now also U9.1
- net GND: now also C10.2, C11.2, C4.2, C5.2, C6.2, C7.2, C8.2, C9.2, Q22.2 (S), R23.2, U2.12, U2.13, U2.7 (GND), U3.12, U3.13, U3.7 (GND), U4.12, U4.13, U4.7 (GND), U5.12, U5.13, U5.7 (GND), U6.12, U6.13, U6.7 (GND), U7.12, U7.13, U7.7 (GND), U8.12, U8.13, U8.7 (GND), U9.12, U9.13, U9.7 (GND)
- net SEL: now also R24.2
- new net: U6.3, U6.4
- new net: U6.5, U6.8
- new net: U5.3, U5.4
- new net: U5.5, U5.8
- new net: Q22.3 (D), R22.2, U2.10, U3.10, U4.10, U5.10, U6.10, U7.10, U8.10, U9.10
- new net: U2.5, U2.8
- new net: Q23.2 (S), R23.1, U2.2, U3.2, U4.2, U5.2, U6.2, U7.2, U8.2, U9.2
- new net: U7.3, U7.4
- new net: U4.3, U4.4
- new net: U4.5, U4.8
- new net: U9.3, U9.4
- new net: U9.5, U9.8
- new net: U7.5, U7.8
- new net: U2.3, U2.4
- new net: Q22.1 (G), Q23.1 (G), R24.1
- new net: U8.5, U8.8
- new net: U8.3, U8.4
- new net: U3.3, U3.4
- new net: U3.5, U3.8
- new net RES0: U2.6
- new net RES1: U3.6
- new net RES2: U4.6
- new net RES3: U5.6
- new net RES4: U6.6
- new net RES5: U7.6
- new net RES6: U8.6
- new net RES7: U9.6

Commit message: started work on ALU motherboard
Parts:
- renumbered C4 to C1, C7 to C12, C8 to C13, C9 to C14, C10 to C15, C11 to C16, C5 to C2, C6 to C3, Q22 to Q1, Q23 to Q2, R24 to R1, R22 to R2, R23 to R3, U2 to U1, U3 to U10, U4 to U11, U5 to U12, U6 to U13, U7 to U14, U8 to U15, U9 to U16

Commit message: fixed schematic of ALU motherboard
Parts:
- renumbered C15 to C10, C16 to C11, C1 to C4, C2 to C5, C3 to C6, C12 to C7, C13 to C8, C14 to C9, Q1 to Q7, Q2 to Q8, R2 to R10, R3 to R11, R1 to R9, U12 to U17, U13 to U18, U14 to U19, U15 to U20, U16 to U21, U1 to U7, U10 to U8, U11 to U9

Commit message: reverted changes to alu_shift
Parts:
- renumbered Q7 to Q22, Q8 to Q23, R10 to R22, R11 to R23, R9 to R24, U7 to U2, U8 to U3, U9 to U4, U17 to U5, U18 to U6, U19 to U7, U20 to U8, U21 to U9
