File: hardware/alu/alu.kicad_pcb (KiCad board)
At the start: 4 copper layers, 140 x 160 mm, 405 parts, among them J8 Conn_02x24_Odd_Even, Q100 IRLML6402, Q101 IRLML6244, Q102 IRLML6402, Q103 IRLML6244, Q104 IRLML6402, Q105 IRLML6244, Q106 IRLML6402, Q107 IRLML6244, Q108 IRLML6402, Q109 IRLML6244, Q110 IRLML6402, Q111 IRLML6244, Q112 IRLML6402, Q113 IRLML6244, Q114 IRLML6402, Q115 IRLML6244, Q116 IRLML6402, Q117 IRLML6244, Q118 IRLML6402, Q119 IRLML6244, Q120 IRLML6402, Q121 IRLML6244, Q122 IRLML6402, Q123 IRLML6244, Q124 IRLML6402, Q125 IRLML6244, Q126 IRLML6402, Q127 IRLML6244, Q128 IRLML6402, Q129 IRLML6244, Q130 IRLML6402, Q131 IRLML6244, Q132 IRLML6402, Q133 IRLML6244, Q134 IRLML6402, Q135 IRLML6244, Q136 IRLML6402, Q137 IRLML6244, Q138 IRLML6402, Q139 IRLML6244, Q140 IRLML6402, Q141 IRLML6244, Q142 IRLML6402, Q143 IRLML6244, Q144 IRLML6402, Q145 IRLML6244, Q146 IRLML6402, Q147 IRLML6244, Q148 IRLML6402, Q149 IRLML6244, Q150 IRLML6402, Q151 IRLML6244, Q152 IRLML6402, Q153 IRLML6244, Q154 IRLML6402, Q155 IRLML6244, Q156 IRLML6402, Q157 IRLML6244, Q158 IRLML6402, Q159 IRLML6244, Q160 IRLML6402, Q161 IRLML6244, Q162 IRLML6402, Q163 IRLML6244, Q164 IRLML6402, Q165 IRLML6244, Q166 IRLML6402, Q167 IRLML6244, Q168 IRLML6402, Q169 IRLML6244, Q170 IRLML6402, Q171 IRLML6244, Q172 IRLML6402, Q173 IRLML6244, Q174 IRLML6402, Q175 IRLML6244, Q176 IRLML6402, Q93 IRLML6402, Q94 IRLML6244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

Commit message: more WIP work on ALU V2
Parts:
- added C91: 330nF, Capacitor_SMD:C_0402_1005Metric, F.Cu at (74.6, 150.2)
- added C93: 330nF, Capacitor_SMD:C_0402_1005Metric, F.Cu at (66.9, 150.2)
- added C94: 330nF, Capacitor_SMD:C_0402_1005Metric, F.Cu at (66.9, 138.8)
- added C95: 330nF, Capacitor_SMD:C_0402_1005Metric, F.Cu at (74.7, 138.8)
- J8: footprint Connector_PinSocket_2.54mm:PinSocket_2x24_P2.54mm_Horizontal -> Connector_PinHeader_2.54mm:PinHeader_2x24_P2.54mm_Horizontal
- moved Q176 528.9 mm to (67.0, 123.2), turned to 180 degrees
- moved Q174 527.2 mm to (67.0, 119.6), turned to 180 degrees
- moved Q172 525.5 mm to (67.0, 116.1), turned to 180 degrees
- moved D145 525.2 mm to (48.7, 67.5)
- moved D147 525.2 mm to (55.8, 67.5)
- moved D148 525.2 mm to (59.4, 67.5)
- moved D149 525.2 mm to (62.9, 67.5)
- moved D47 525.2 mm to (70.0, 67.5)
- moved D48 525.2 mm to (73.6, 67.5)
- moved Q153 525.2 mm to (48.7, 72.0)
- moved Q157 525.2 mm to (55.8, 72.0)
- moved Q159 525.2 mm to (59.4, 72.0)
- moved Q161 525.2 mm to (62.9, 72.0)
- moved Q165 525.2 mm to (70.0, 72.0)
- moved Q167 525.2 mm to (73.6, 72.0)
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Routing:
- net /IA7: track 32.5 -> 249.9 mm, vias 5 -> 13
- net /IA6: track 32.6 -> 237.8 mm, vias 5 -> 13
- net /IA5: track 32.6 -> 225.9 mm, vias 5 -> 13
- net /IA4: track 32.6 -> 214.2 mm, vias 5 -> 13
- net /IB7: track 36.3 -> 211.1 mm, vias 6 -> 9
- net /IA3: track 32.6 -> 202.9 mm, vias 5 -> 13
- net /IB6: track 36.3 -> 199.7 mm, vias 6 -> 9
- net /IA2: track 32.6 -> 192.1 mm, vias 5 -> 13
- net /IB5: track 36.3 -> 188.5 mm, vias 6 -> 9
- net /IA1: track 32.6 -> 181.1 mm, vias 5 -> 13
- net /IB4: track 36.3 -> 177.1 mm, vias 6 -> 9
- net /IA0: track 32.6 -> 172.2 mm, vias 5 -> 13
- net /IB3: track 36.3 -> 165.6 mm, vias 6 -> 9
- net /IB2: track 65.4 -> 183.4 mm, vias 10 -> 13
- net /IB1: track 64.9 -> 172.0 mm, vias 10 -> 13
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Other:
- board size 140 x 160 mm -> 140 x 130 mm
- board text added: "A"
- board text added: "ADD"
- board text added: "AND"
- board text added: "B"
- board text added: "CEN"
- board text added: "CIN"
- board text added: "COUT"
- board text added: "CRY"
- board text added: "NAND"
- board text added: "NEG"
- board text added: "OP"
- board text added: "OR"
- board text added: "OVF"
- board text added: "RES"
- board text added: "SHL"
- board text added: "SHR"
- board text added: "SUB"
- board text added: "XOR"
- board text added: "ZERO"

Commit message: further WIP on ALU V2 pcb
Parts:
- moved C88 0.20 mm to (38.2, 47.5)
- moved C86 0.20 mm to (38.0, 41.5)
- moved C87 0.20 mm to (38.2, 53.6)
Routing:
- net Net-(U91-I0d): track 0.00 -> 162.0 mm, vias 0 -> 5
- net Net-(U91-I0c): track 0.00 -> 153.1 mm, vias 0 -> 5
- net Net-(U91-I0b): track 0.00 -> 140.9 mm, vias 0 -> 5
- net Net-(U91-I0a): track 0.00 -> 135.4 mm, vias 0 -> 5
- net Net-(U90-I0d): track 0.00 -> 123.4 mm, vias 0 -> 5
- net Net-(U52-Za): track 0.00 -> 111.9 mm, vias 0 -> 4
- net Net-(U90-I0c): track 0.00 -> 109.9 mm, vias 0 -> 5
- net Net-(U85-Za): track 0.00 -> 107.1 mm, vias 0 -> 3
- net Net-(U85-Zd): track 0.00 -> 104.7 mm, vias 0 -> 3
- net Net-(U52-Zd): track 0.00 -> 102.3 mm, vias 0 -> 4
- net Net-(U85-Zb): track 0.00 -> 100.1 mm, vias 0 -> 3
- net Net-(U52-Zb): track 0.00 -> 99.6 mm, vias 0 -> 4
- net +5V: track 1118.0 -> 1216.1 mm, vias 156 -> 162
- net Net-(U90-I0b): track 0.00 -> 96.7 mm, vias 0 -> 5
- net Net-(U85-Zc): track 0.00 -> 96.5 mm, vias 0 -> 3
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