File: hardware/alu/alu.kicad_pcb (KiCad board)
At the start: 4 copper layers, 140 x 130 mm, 409 parts, among them J8 Conn_02x24_Odd_Even, Q100 IRLML6402, Q101 IRLML6244, Q102 IRLML6402, Q103 IRLML6244, Q104 IRLML6402, Q105 IRLML6244, Q106 IRLML6402, Q107 IRLML6244, Q108 IRLML6402, Q109 IRLML6244, Q110 IRLML6402, Q111 IRLML6244, Q112 IRLML6402, Q113 IRLML6244, Q114 IRLML6402, Q115 IRLML6244, Q116 IRLML6402, Q117 IRLML6244, Q118 IRLML6402, Q119 IRLML6244, Q120 IRLML6402, Q121 IRLML6244, Q122 IRLML6402, Q123 IRLML6244, Q124 IRLML6402, Q125 IRLML6244, Q126 IRLML6402, Q127 IRLML6244, Q128 IRLML6402, Q129 IRLML6244, Q130 IRLML6402, Q131 IRLML6244, Q132 IRLML6402, Q133 IRLML6244, Q134 IRLML6402, Q135 IRLML6244, Q136 IRLML6402, Q137 IRLML6244, Q138 IRLML6402, Q139 IRLML6244, Q140 IRLML6402, Q141 IRLML6244, Q142 IRLML6402, Q143 IRLML6244, Q144 IRLML6402, Q145 IRLML6244, Q146 IRLML6402, Q147 IRLML6244, Q148 IRLML6402, Q149 IRLML6244, Q150 IRLML6402, Q151 IRLML6244, Q152 IRLML6402, Q153 IRLML6244, Q154 IRLML6402, Q155 IRLML6244, Q156 IRLML6402, Q157 IRLML6244, Q158 IRLML6402, Q159 IRLML6244, Q160 IRLML6402, Q161 IRLML6244, Q162 IRLML6402, Q163 IRLML6244, Q164 IRLML6402, Q165 IRLML6244, Q166 IRLML6402, Q167 IRLML6244, Q168 IRLML6402, Q169 IRLML6244, Q170 IRLML6402, Q171 IRLML6244, Q172 IRLML6402, Q173 IRLML6244, Q174 IRLML6402, Q175 IRLML6244, Q176 IRLML6402, Q93 IRLML6402, Q94 IRLML6244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

Commit message: ALU V2 done?
Routing:
- net /IOP1: track 31.1 -> 265.9 mm, vias 2 -> 9
- net /IOP0: track 245.0 -> 471.8 mm, vias 28 -> 33
- net +5V: track 1216.1 -> 1421.1 mm, vias 162 -> 170
- net /ICRY: track 89.1 -> 279.8 mm, vias 9 -> 17
- net /IOP2: track 35.6 -> 221.7 mm, vias 3 -> 8
- net Net-(U34-Pad11): track 0.00 -> 147.5 mm, vias 0 -> 5
- net Net-(U35-Pad11): track 0.00 -> 125.6 mm, vias 0 -> 4
- net Net-(Q161-G): track 0.00 -> 125.0 mm, vias 0 -> 4
- net Net-(Q163-G): track 0.00 -> 123.7 mm, vias 0 -> 4
- net Net-(Q165-G): track 0.00 -> 113.6 mm, vias 0 -> 4
- net Net-(Q153-G): track 0.00 -> 112.6 mm, vias 0 -> 3
- net Net-(Q167-G): track 0.00 -> 102.2 mm, vias 0 -> 3
- net Net-(Q155-G): track 0.00 -> 101.5 mm, vias 0 -> 2
- net Net-(D124-K): track 21.9 -> 117.5 mm, vias 0 -> 2
- net Net-(Q159-G): track 0.00 -> 94.9 mm, vias 0 -> 2
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- added copper zone on F.Cu, net +5V

Commit message: small fixes in ALU V2, started work on register fabric, schematic done (?)
Parts:
- added D52: LED, LED_SMD:LED_0402_1005Metric, F.Cu at (38.0, 34.7)
- added R192: 1000, Resistor_SMD:R_0402_1005Metric, F.Cu at (36.8, 34.7)
Routing:
- net Net-(D52-K): track 0.00 -> 1.20 mm
- net GND: track 615.2 -> 616.2 mm, vias 245 -> 246
Other:
- board text added: "PWR"
