File: hardware/alu/alu.kicad_pcb (KiCad board)
At the start: 4 copper layers, 140 x 130 mm, 414 parts, among them J8 Conn_02x24_Odd_Even, Q100 IRLML6402, Q101 IRLML6244, Q102 IRLML6402, Q103 IRLML6244, Q104 IRLML6402, Q105 IRLML6244, Q106 IRLML6402, Q107 IRLML6244, Q108 IRLML6402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

Commit message: all PCBs passing all CRC & vibe checks
Parts:
- R1, R10, R11, R12, R13, R14, R15, R16, R17, R18, R19, R2, R20, R21, R3, R4, R5, R6, R7, R8, R9: value 10K -> 100K
