File: hardware/register_fabric/register_fabric.kicad_pcb (KiCad board)
At the start: 2 copper layers, 356 x 52.6 mm, 417 parts, among them J2 Conn_02x40_Odd_Even, J3 Conn_02x16_Odd_Even, J4 Conn_02x16_Odd_Even, J5 Conn_02x16_Odd_Even, J6 Conn_02x16_Odd_Even, J7 Conn_02x16_Odd_Even, J8 Conn_02x16_Odd_Even, J9 Conn_02x16_Odd_Even, Q109 IRLML6244, Q110 IRLML6402, Q111 IRLML6244, Q112 IRLML6402, Q113 IRLML6244, Q114 IRLML6402, Q115 IRLML6244, Q116 IRLML6402, Q117 IRLML6244, Q118 IRLML6402, Q119 IRLML6244, Q120 IRLML6402, Q121 IRLML6244, Q122 IRLML6402, Q123 IRLML6244, Q124 IRLML6402, Q125 IRLML6244, Q126 IRLML6402, Q127 IRLML6244, Q128 IRLML6402, Q129 IRLML6244, Q130 IRLML6402, Q131 IRLML6244, Q132 IRLML6402, Q133 IRLML6244, Q134 IRLML6402, Q135 IRLML6244, Q136 IRLML6402, Q137 IRLML6244, Q138 IRLML6402, Q139 IRLML6244, Q140 IRLML6402, Q141 IRLML6244, Q142 IRLML6402, Q143 IRLML6244, Q144 IRLML6402, Q145 IRLML6244, Q146 IRLML6402, Q147 IRLML6244, Q148 IRLML6402, Q149 IRLML6244, Q150 IRLML6402, Q151 IRLML6244, Q152 IRLML6402, Q153 IRLML6244, Q154 IRLML6402, Q155 IRLML6244, Q156 IRLML6402, Q157 IRLML6244, Q158 IRLML6402, Q159 IRLML6244, Q160 IRLML6402, Q161 IRLML6244, Q162 IRLML6402, Q163 IRLML6244, Q164 IRLML6402, Q165 IRLML6244, Q166 IRLML6402, Q167 IRLML6244, Q168 IRLML6402, Q169 IRLML6244, Q170 IRLML6402, Q171 IRLML6244, Q172 IRLML6402, Q173 IRLML6244, Q174 IRLML6402, Q175 IRLML6244, Q176 IRLML6402, Q177 IRLML6244, Q178 IRLML6402, Q179 IRLML6244, Q180 IRLML6402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

Commit message: started work on register fabric PCB layout, grouped LEDs
Parts:
- removed R244, R245, R246, R247, R248, R249, R250, R251, R252, R253, R254, R255, R256, R257, R258, R259: 1000, Resistor_SMD:R_0402_1005Metric
- added R1: 10K, Resistor_SMD:R_0402_1005Metric, F.Cu at (-108.0, -21.4)
- added R10: 10K, Resistor_SMD:R_0402_1005Metric, F.Cu at (298.1, 144.7)
- added R11: 10K, Resistor_SMD:R_0402_1005Metric, F.Cu at (255.2, 144.7)
- added R12: 10K, Resistor_SMD:R_0402_1005Metric, F.Cu at (247.1, 144.7)
- added R13: 10K, Resistor_SMD:R_0402_1005Metric, F.Cu at (204.2, 144.7)
- added R14: 10K, Resistor_SMD:R_0402_1005Metric, F.Cu at (196.1, 144.7)
- added R15: 10K, Resistor_SMD:R_0402_1005Metric, F.Cu at (153.2, 144.7)
- added R16: 10K, Resistor_SMD:R_0402_1005Metric, F.Cu at (145.1, 144.7)
- added R2: 10K, Resistor_SMD:R_0402_1005Metric, F.Cu at (-108.0, -19.4)
- added R3: 10K, Resistor_SMD:R_0402_1005Metric, F.Cu at (459.2, 144.7)
- added R4: 10K, Resistor_SMD:R_0402_1005Metric, F.Cu at (451.1, 144.7)
- added R5: 10K, Resistor_SMD:R_0402_1005Metric, F.Cu at (408.2, 144.7)
- added R6: 10K, Resistor_SMD:R_0402_1005Metric, F.Cu at (400.1, 144.7)
- added R7: 10K, Resistor_SMD:R_0402_1005Metric, F.Cu at (357.2, 144.7)
- added R8: 10K, Resistor_SMD:R_0402_1005Metric, F.Cu at (349.1, 144.7)
- added R9: 10K, Resistor_SMD:R_0402_1005Metric, F.Cu at (306.2, 144.7)
- U1, U10, U11, U12, U13, U14, U15, U16, U17, U3, U4, U5, U6, U7, U8, U9: footprint Package_SO:SO-20_12.8x7.5mm_P1.27mm -> Package_SO:TSSOP-20_4.4x6.5mm_P0.65mm
- moved J4 403.3 mm to (414.0, 140.8), turned to -90 degrees
- moved J3 380.5 mm to (465.0, 140.8)
- moved U19 363.5 mm to (437.7, 146.7), turned to -90 degrees
- moved J5 361.7 mm to (363.0, 140.8), turned to -90 degrees
- moved U4 348.2 mm to (455.1, 146.9), turned to -90 degrees
- moved D198 346.1 mm to (-104.4, -197.4), turned to 90 degrees
- moved D199 345.3 mm to (-104.4, -193.8), turned to 90 degrees
- moved D200 344.5 mm to (-104.4, -190.2), turned to 90 degrees
- moved D201 343.8 mm to (-104.4, -186.6), turned to 90 degrees
- moved C4 335.3 mm to (429.3, 146.7), turned to 180 degrees
- moved U5 334.0 mm to (447.0, 146.9), turned to -90 degrees
- moved J6 328.6 mm to (312.0, 140.8), turned to -90 degrees
- moved D195 325.2 mm to (-83.6, -197.8), turned to 180 degrees
- moved U21 324.5 mm to (386.7, 146.7), turned to -90 degrees
- moved U3 323.3 mm to (-113.8, -10.3)
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Connections:
- net Net-(D141-A) renamed /DII7
- net Net-(D142-A) renamed /DII6
- net Net-(D143-A) renamed /DII5
- net Net-(D144-A) renamed /DII4
- net Net-(D145-A) renamed /DII3
- net Net-(D146-A) renamed /DII2
- net Net-(D147-A) renamed /DII1
- net Net-(D148-A) renamed /DII0
- net Net-(D165-A) renamed /FII7
- net Net-(D166-A) renamed /FII6
- net Net-(D167-A) renamed /FII5
- net Net-(D168-A) renamed /FII4
- net Net-(D169-A) renamed /FII3
- net Net-(D170-A) renamed /FII2
- net Net-(D171-A) renamed /FII1
- net Net-(D172-A) renamed /FII0
- net Net-(D189-A) renamed /RSI02
- net Net-(D190-A) renamed /RSI01
- net Net-(D191-A) renamed /RSI00
- net Net-(D192-A) renamed /RSI12
- net Net-(D193-A) renamed /RSI11
- net Net-(D194-A) renamed /RSI10
- net Net-(D195-A) renamed /WSI2
- net Net-(D196-A) renamed /WSI1
- net Net-(D197-A) renamed /WSI0
- net Net-(D199-A) renamed /IFWEN
- net Net-(D200-A) renamed /ICLK
- net Net-(D201-A) renamed /I!CLR
- net Net-(Q125-G) renamed /RI07
- net Net-(Q127-G) renamed /RI06
- net Net-(Q129-G) renamed /RI05
- net Net-(Q131-G) renamed /RI04
- net Net-(Q133-G) renamed /RI03
- net Net-(Q135-G) renamed /RI02
- net Net-(Q137-G) renamed /RI01
- net Net-(Q139-G) renamed /RI00
- net Net-(Q141-G) renamed /RI17
- net Net-(Q143-G) renamed /RI16
- net Net-(Q145-G) renamed /RI15
- net Net-(Q147-G) renamed /RI14
- net Net-(Q149-G) renamed /RI13
- net Net-(Q151-G) renamed /RI12
- net Net-(Q153-G) renamed /RI11
- net Net-(Q155-G) renamed /RI10
- D198 pad 2: Net-(D198-A) -> /IRWEN
- J2 pad 74: /RWEN -> /COUT
- J2 pad 76: Net-(J2-Pin_2) -> /RWEN
- J7 pad 5: Net-(J7-Pin_5) -> /COUT
- J8 pad 10: Net-(J8-Pin_10) -> /RAI7
- J8 pad 3: Net-(J8-Pin_3) -> /RAI0
- J8 pad 4: Net-(J8-Pin_4) -> /RAI1
- J8 pad 5: Net-(J8-Pin_5) -> /RAI2
- J8 pad 6: Net-(J8-Pin_6) -> /RAI3
- J8 pad 7: Net-(J8-Pin_7) -> /RAI4
- J8 pad 8: Net-(J8-Pin_8) -> /RAI5
- J8 pad 9: Net-(J8-Pin_9) -> /RAI6
- J9 pad 10: Net-(J9-Pin_10) -> /RAI15
- J9 pad 3: Net-(J9-Pin_3) -> /RAI8
- J9 pad 4: Net-(J9-Pin_4) -> /RAI9
- J9 pad 5: Net-(J9-Pin_5) -> /RAI10
- J9 pad 6: Net-(J9-Pin_6) -> /RAI11
- J9 pad 7: Net-(J9-Pin_7) -> /RAI12
- J9 pad 8: Net-(J9-Pin_8) -> /RAI13
- J9 pad 9: Net-(J9-Pin_9) -> /RAI14
- Q173 pad 1: unconnected-(Q173-G-Pad1) -> /RAI15
- Q175 pad 1: unconnected-(Q175-G-Pad1) -> /RAI14
- Q177 pad 1: unconnected-(Q177-G-Pad1) -> /RAI13
- Q179 pad 1: unconnected-(Q179-G-Pad1) -> /RAI12
- Q181 pad 1: unconnected-(Q181-G-Pad1) -> /RAI11
- Q183 pad 1: unconnected-(Q183-G-Pad1) -> /RAI10
- Q185 pad 1: unconnected-(Q185-G-Pad1) -> /RAI9
- Q187 pad 1: unconnected-(Q187-G-Pad1) -> /RAI8
- Q189 pad 1: unconnected-(Q189-G-Pad1) -> /RAI7
- Q191 pad 1: unconnected-(Q191-G-Pad1) -> /RAI6
- Q193 pad 1: unconnected-(Q193-G-Pad1) -> /RAI5
- Q195 pad 1: unconnected-(Q195-G-Pad1) -> /RAI4
- Q197 pad 1: unconnected-(Q197-G-Pad1) -> /RAI3
- Q199 pad 1: unconnected-(Q199-G-Pad1) -> /RAI2
- Q201 pad 1: unconnected-(Q201-G-Pad1) -> /RAI1
- Q203 pad 1: unconnected-(Q203-G-Pad1) -> /RAI0
- Q224 pad 3: Net-(D198-A) -> /IRWEN
- U12 pad 4: Net-(J7-Pin_5) -> /COUT
- U13 pad 4: Net-(J7-Pin_5) -> /COUT
- U14 pad 2: Net-(J8-Pin_3) -> /RAI0
- U14 pad 3: Net-(J8-Pin_4) -> /RAI1
- U14 pad 4: Net-(J8-Pin_5) -> /RAI2
- U14 pad 5: Net-(J8-Pin_6) -> /RAI3
- U14 pad 6: Net-(J8-Pin_7) -> /RAI4
- U14 pad 7: Net-(J8-Pin_8) -> /RAI5
- U14 pad 8: Net-(J8-Pin_9) -> /RAI6
- U14 pad 9: Net-(J8-Pin_10) -> /RAI7
- U15 pad 2: Net-(J8-Pin_3) -> /RAI0
- U15 pad 3: Net-(J8-Pin_4) -> /RAI1
- U15 pad 4: Net-(J8-Pin_5) -> /RAI2
- U15 pad 5: Net-(J8-Pin_6) -> /RAI3
- U15 pad 6: Net-(J8-Pin_7) -> /RAI4
- U15 pad 7: Net-(J8-Pin_8) -> /RAI5
- U15 pad 8: Net-(J8-Pin_9) -> /RAI6
- U15 pad 9: Net-(J8-Pin_10) -> /RAI7
- U16 pad 2: Net-(J9-Pin_3) -> /RAI8
- U16 pad 3: Net-(J9-Pin_4) -> /RAI9
- U16 pad 4: Net-(J9-Pin_5) -> /RAI10
- U16 pad 5: Net-(J9-Pin_6) -> /RAI11
- U16 pad 6: Net-(J9-Pin_7) -> /RAI12
- U16 pad 7: Net-(J9-Pin_8) -> /RAI13
- U16 pad 8: Net-(J9-Pin_9) -> /RAI14
- U16 pad 9: Net-(J9-Pin_10) -> /RAI15
- U17 pad 2: Net-(J9-Pin_3) -> /RAI8
- U17 pad 3: Net-(J9-Pin_4) -> /RAI9
- U17 pad 4: Net-(J9-Pin_5) -> /RAI10
- U17 pad 5: Net-(J9-Pin_6) -> /RAI11
- U17 pad 6: Net-(J9-Pin_7) -> /RAI12
- U17 pad 7: Net-(J9-Pin_8) -> /RAI13
- U17 pad 8: Net-(J9-Pin_9) -> /RAI14
- U17 pad 9: Net-(J9-Pin_10) -> /RAI15
- U19 pad 1: Net-(U19-Pad1) -> /IRWEN
- U21 pad 1: Net-(U19-Pad1) -> /IRWEN
- U22 pad 1: Net-(U19-Pad1) -> /IRWEN
- U23 pad 1: Net-(U19-Pad1) -> /IRWEN
- U24 pad 1: Net-(U19-Pad1) -> /IRWEN
- U25 pad 1: Net-(U19-Pad1) -> /IRWEN
- U26 pad 1: Net-(U19-Pad1) -> /IRWEN
Routing:
- net +5V: track 0.00 -> 723.4 mm, vias 0 -> 129
- net GND: track 0.00 -> 595.7 mm, vias 0 -> 145
- net /RI00: track 0.00 -> 368.8 mm, vias 0 -> 7
- net /RI01: track 0.00 -> 365.2 mm, vias 0 -> 7
- net /RI02: track 0.00 -> 361.6 mm, vias 0 -> 7
- net /RI03: track 0.00 -> 358.2 mm, vias 0 -> 7
- net /RI04: track 0.00 -> 354.7 mm, vias 0 -> 7
- net /RI05: track 0.00 -> 351.1 mm, vias 0 -> 7
- net /RI06: track 0.00 -> 347.6 mm, vias 0 -> 7
- net /RI07: track 0.00 -> 343.9 mm, vias 0 -> 7
- net /RI10: track 0.00 -> 340.4 mm, vias 0 -> 7
- net /RI11: track 0.00 -> 336.8 mm, vias 0 -> 7
- net /RI12: track 0.00 -> 333.5 mm, vias 0 -> 7
- net /RI13: track 0.00 -> 329.7 mm, vias 0 -> 7
- net /RI14: track 0.00 -> 326.1 mm, vias 0 -> 7
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- added copper zone on F.Cu, net +5V
- added copper zone on B.Cu, net GND
- added copper zone on In1.Cu, net GND
- added copper zone on In2.Cu, net GND
Other:
- copper layers 2 -> 4

Commit message: finished Rev A of register fabric pcb
Parts:
- added C33: 330nF, Capacitor_SMD:C_0402_1005Metric, F.Cu at (255.3, 166.1)
- added C34: 330nF, Capacitor_SMD:C_0402_1005Metric, F.Cu at (264.0, 166.1)
- added C35: 330nF, Capacitor_SMD:C_0402_1005Metric, F.Cu at (220.2, 148.6)
- added C36: 330nF, Capacitor_SMD:C_0402_1005Metric, F.Cu at (266.7, 148.7)
- added D202: LED, LED_SMD:LED_0402_1005Metric, F.Cu at (339.1, 180.0)
- added R244: 1000, Resistor_SMD:R_0402_1005Metric, F.Cu at (338.1, 180.0)
- moved D198 573.1 mm to (339.2, 165.5)
- moved D199 573.1 mm to (339.2, 169.1)
- moved D200 573.1 mm to (339.2, 172.7)
- moved Q223 573.1 mm to (334.7, 165.5)
- moved Q224 573.1 mm to (330.7, 165.5)
- moved Q225 573.1 mm to (334.7, 169.1)
- moved Q226 573.1 mm to (330.7, 169.1)
- moved Q227 573.1 mm to (334.7, 172.7)
- moved Q228 573.1 mm to (330.7, 172.7)
- moved R236 573.1 mm to (337.7, 165.5)
- moved R237 573.1 mm to (337.7, 166.5)
- moved R238 573.1 mm to (337.7, 169.1)
- moved R240 573.1 mm to (337.7, 172.7)
- moved R243 573.1 mm to (337.7, 177.3)
- moved R39 573.1 mm to (337.7, 168.0)
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Connections:
- J2 pad 1: Net-(J2-Pin_1) -> GND
- J2 pad 19: Net-(J2-Pin_1) -> GND
- J2 pad 2: Net-(J2-Pin_2) -> GND
- J2 pad 20: Net-(J2-Pin_2) -> GND
- J2 pad 37: Net-(J2-Pin_1) -> GND
- J2 pad 38: Net-(J2-Pin_2) -> GND
- J2 pad 55: Net-(J2-Pin_1) -> GND
- J2 pad 56: Net-(J2-Pin_2) -> GND
- J2 pad 63: Net-(J2-Pin_1) -> GND
- J2 pad 64: Net-(J2-Pin_2) -> GND
- J2 pad 69: Net-(J2-Pin_1) -> GND
- J2 pad 72: Net-(J2-Pin_2) -> GND
- J2 pad 79: Net-(J2-Pin_1) -> GND
- J2 pad 80: Net-(J2-Pin_2) -> GND
Routing:
- net +5V: track 723.4 -> 1822.9 mm, vias 129 -> 171
- net /DII1: track 9.66 -> 528.5 mm, vias 0 -> 9
- net /DII0: track 9.66 -> 519.2 mm, vias 0 -> 9
- net /DII3: track 9.66 -> 503.3 mm, vias 0 -> 8
- net /DII2: track 9.66 -> 493.0 mm, vias 0 -> 8
- net /DII5: track 9.66 -> 488.1 mm, vias 0 -> 8
- net /DII7: track 9.66 -> 479.6 mm, vias 0 -> 8
- net /DII4: track 9.66 -> 474.5 mm, vias 0 -> 8
- net /DII6: track 9.66 -> 462.1 mm, vias 0 -> 8
- net Net-(U2-~{Y1}): track 5.31 -> 456.2 mm, vias 0 -> 3
- net Net-(U18-~{Y1}): track 5.31 -> 442.0 mm, vias 0 -> 2
- net /ICLK: track 9.66 -> 441.1 mm, vias 0 -> 1
- net Net-(U20-Y1): track 0.00 -> 407.7 mm, vias 0 -> 2
- net /I!CLR: track 9.66 -> 407.2 mm, vias 0 -> 2
- net Net-(U2-~{Y2}): track 5.31 -> 402.3 mm, vias 0 -> 4
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Other:
- board size 356 x 52.6 mm -> 356 x 62.3 mm
- board text added: "8x8 bit register fabric | REV A"
- board text added: "ADDR"
- board text added: "CLK"
- board text added: "CLR"
- board text added: "DIN"
- board text added: "FIN"
- board text added: "FWEN"
- board text added: "PWR"
- board text added: "READ0"
- board text added: "READ1"
- board text added: "RSEL0"
- board text added: "RSEL1"
- board text added: "RWEN"
- board text added: "WSEL"
- board text added: "mrab"
