File: hardware/register_fabric/register_fabric.kicad_pcb (KiCad board)
At the start: 4 copper layers, 356 x 62.3 mm, 423 parts, among them J2 Conn_02x40_Odd_Even, J3 Conn_02x16_Odd_Even, J4 Conn_02x16_Odd_Even, J5 Conn_02x16_Odd_Even, J6 Conn_02x16_Odd_Even, J7 Conn_02x16_Odd_Even, J8 Conn_02x16_Odd_Even, J9 Conn_02x16_Odd_Even, Q109 IRLML6244, Q110 IRLML6402, Q111 IRLML6244, Q112 IRLML6402, Q113 IRLML6244, Q114 IRLML6402, Q115 IRLML6244, Q116 IRLML6402, Q117 IRLML6244, Q118 IRLML6402, Q119 IRLML6244, Q120 IRLML6402, Q121 IRLML6244, Q122 IRLML6402, Q123 IRLML6244, Q124 IRLML6402, Q125 IRLML6244, Q126 IRLML6402, Q127 IRLML6244, Q128 IRLML6402, Q129 IRLML6244, Q130 IRLML6402, Q131 IRLML6244, Q132 IRLML6402, Q133 IRLML6244, Q134 IRLML6402, Q135 IRLML6244, Q136 IRLML6402, Q137 IRLML6244, Q138 IRLML6402, Q139 IRLML6244, Q140 IRLML6402, Q141 IRLML6244, Q142 IRLML6402, Q143 IRLML6244, Q144 IRLML6402, Q145 IRLML6244, Q146 IRLML6402, Q147 IRLML6244, Q148 IRLML6402, Q149 IRLML6244, Q150 IRLML6402, Q151 IRLML6244, Q152 IRLML6402, Q153 IRLML6244, Q154 IRLML6402, Q155 IRLML6244, Q156 IRLML6402, Q157 IRLML6244, Q158 IRLML6402, Q159 IRLML6244, Q160 IRLML6402, Q161 IRLML6244, Q162 IRLML6402, Q163 IRLML6244, Q164 IRLML6402, Q165 IRLML6244, Q166 IRLML6402, Q167 IRLML6244, Q168 IRLML6402, Q169 IRLML6244, Q170 IRLML6402, Q171 IRLML6244, Q172 IRLML6402, Q173 IRLML6244, Q174 IRLML6402, Q175 IRLML6244, Q176 IRLML6402, Q177 IRLML6244, Q178 IRLML6402, Q179 IRLML6244, Q180 IRLML6402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

Commit message: added fiducials and markers to ALU, started on register fabric
Parts:
- added H1: MountingHole_Pad, MountingHole:MountingHole_3.2mm_M3_ISO7380_Pad_TopBottom, F.Cu at (165.5, 139.4)
- added H2: MountingHole_Pad, MountingHole:MountingHole_3.2mm_M3_ISO7380_Pad_TopBottom, F.Cu at (216.5, 139.4)
- added H3: MountingHole_Pad, MountingHole:MountingHole_3.2mm_M3_ISO7380_Pad_TopBottom, F.Cu at (125.3, 157.9)
- added H4: MountingHole_Pad, MountingHole:MountingHole_3.2mm_M3_ISO7380_Pad_TopBottom, F.Cu at (267.5, 139.4)
- added H5: MountingHole_Pad, MountingHole:MountingHole_3.2mm_M3_ISO7380_Pad_TopBottom, F.Cu at (461.2, 181.6)
- added H6: MountingHole_Pad, MountingHole:MountingHole_3.2mm_M3_ISO7380_Pad_TopBottom, F.Cu at (318.4, 139.4)
- added H7: MountingHole_Pad, MountingHole:MountingHole_3.2mm_M3_ISO7380_Pad_TopBottom, F.Cu at (420.4, 139.4)
- added H8: MountingHole_Pad, MountingHole:MountingHole_3.2mm_M3_ISO7380_Pad_TopBottom, F.Cu at (369.4, 139.4)
Routing:
- net Net-(J7-Pin_18): track 35.0 -> 37.3 mm, vias 1 -> 3
- net Net-(J7-Pin_20): track 34.3 -> 36.0 mm
- net Net-(J7-Pin_19): track 35.6 -> 36.9 mm
Other:
- board text added: "GND"
- board text added: "Wer das liest, ist doof"
