File: hardware/register_fabric/register_fabric.kicad_sch (KiCad schematic)
At the start: 431 parts, among them J2 Conn_02x40_Odd_Even, J3 Conn_02x16_Odd_Even, J4 Conn_02x16_Odd_Even, J5 Conn_02x16_Odd_Even, J6 Conn_02x16_Odd_Even, J7 Conn_02x16_Odd_Even, J8 Conn_02x16_Odd_Even, J9 Conn_02x16_Odd_Even, Q109 IRLML6244, Q110 IRLML6402, Q111 IRLML6244, Q112 IRLML6402, Q113 IRLML6244, Q114 IRLML6402, Q115 IRLML6244, Q116 IRLML6402, Q117 IRLML6244, Q118 IRLML6402, Q119 IRLML6244, Q120 IRLML6402, Q121 IRLML6244, Q122 IRLML6402, Q123 IRLML6244, Q124 IRLML6402, Q125 IRLML6244, Q126 IRLML6402, Q127 IRLML6244, Q128 IRLML6402, Q129 IRLML6244, Q130 IRLML6402, Q131 IRLML6244, Q132 IRLML6402, Q133 IRLML6244, Q134 IRLML6402, Q135 IRLML6244, Q136 IRLML6402, Q137 IRLML6244, Q138 IRLML6402, Q139 IRLML6244, Q140 IRLML6402, Q141 IRLML6244, Q142 IRLML6402, Q143 IRLML6244, Q144 IRLML6402, Q145 IRLML6244, Q146 IRLML6402, Q147 IRLML6244, Q148 IRLML6402, Q149 IRLML6244, Q150 IRLML6402, Q151 IRLML6244, Q152 IRLML6402, Q153 IRLML6244, Q154 IRLML6402, Q155 IRLML6244, Q156 IRLML6402, Q157 IRLML6244, Q158 IRLML6402, Q159 IRLML6244, Q160 IRLML6402, Q161 IRLML6244, Q162 IRLML6402, Q163 IRLML6244, Q164 IRLML6402, Q165 IRLML6244, Q166 IRLML6402, Q167 IRLML6244, Q168 IRLML6402, Q169 IRLML6244, Q170 IRLML6402, Q171 IRLML6244, Q172 IRLML6402, Q173 IRLML6244, Q174 IRLML6402, Q175 IRLML6244, Q176 IRLML6402, Q177 IRLML6244, Q178 IRLML6402, Q179 IRLML6244, Q180 IRLML6402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

Commit message: as ordered
Parts:
- C11, C12, C14, C15, C17, C18, C2, C20, C21, C23, C24, C25, C26, C27, C28, C29, C3, C30, C31, C32, C33, C34, C35, C36, C5, C6, C8, C9: LCSC (none) -> C77020
- R1, R10, R11, R12, R13, R14, R15, R16, R2, R3, R4, R5, R6, R7, R8, R9: LCSC (none) -> C60491
- R21, R22, R23, R24, R25, R26, R27, R28, R29, R30, R31, R32, R33, R34, R35, R36, R37, R38, R39, R40, R41, R45, R46, R47, R48, R49, R50, R51, R52: LCSC C60490 -> C60491
- U1, U10, U11, U12, U13, U14, U15, U16, U17, U3, U4, U5, U6, U7, U8, U9: LCSC (none) -> C5626
- U18, U2: LCSC (none) -> C5602
- U19, U21, U22, U23, U24, U25, U26: LCSC (none) -> C5586
- U20: LCSC (none) -> C5620
