File: hardware/io/io.kicad_pcb (KiCad board)
At the start: 2 copper layers, 215 x 160 mm, 0 parts

Commit message: almost done with placement for IO board
Parts:
- added C1: 22pF, Capacitor_SMD:C_0402_1005Metric, F.Cu at (287.3, 469.7)
- added C100: 100nF, Capacitor_SMD:C_0402_1005Metric, F.Cu at (286.3, 449.8)
- added C101: 100nF, Capacitor_SMD:C_0402_1005Metric, F.Cu at (295.8, 449.8)
- added C102: 100nF, Capacitor_SMD:C_0402_1005Metric, F.Cu at (282.8, 457.8)
- added C103: 100nF, Capacitor_SMD:C_0402_1005Metric, F.Cu at (286.8, 468.2)
- added C104: 100nF, Capacitor_SMD:C_0402_1005Metric, F.Cu at (273.7, 428.1)
- added C105: 100nF, Capacitor_SMD:C_0402_1005Metric, F.Cu at (265.8, 428.1)
- added C106: 100nF, Capacitor_SMD:C_0402_1005Metric, F.Cu at (286.4, 434.2)
- added C107: 100nF, Capacitor_SMD:C_0402_1005Metric, F.Cu at (-199.4, 455.7)
- added C108: 100nF, Capacitor_SMD:C_0402_1005Metric, F.Cu at (396.0, 410.8)
- added C109: 100nF, Capacitor_SMD:C_0402_1005Metric, F.Cu at (396.0, 400.7)
- added C11: 100nF, Capacitor_SMD:C_0402_1005Metric, F.Cu at (288.3, 449.8)
- added C110: 100nF, Capacitor_SMD:C_0402_1005Metric, F.Cu at (396.0, 390.6)
- added C111: 100nF, Capacitor_SMD:C_0402_1005Metric, F.Cu at (396.0, 420.9)
- added C12: 100nF, Capacitor_SMD:C_0402_1005Metric, F.Cu at (298.2, 299.4)
- added C13: 100nF, Capacitor_SMD:C_0402_1005Metric, F.Cu at (290.5, 299.4)
- added C14: 100nF, Capacitor_SMD:C_0402_1005Metric, F.Cu at (290.9, 379.6)
- added C15: 100nF, Capacitor_SMD:C_0402_1005Metric, F.Cu at (290.5, 371.3)
- added C16: 100nF, Capacitor_SMD:C_0402_1005Metric, F.Cu at (298.3, 415.4)
- added C17: 100nF, Capacitor_SMD:C_0402_1005Metric, F.Cu at (298.3, 407.2)
- added C18: 100nF, Capacitor_SMD:C_0402_1005Metric, F.Cu at (268.8, 342.5)
- added C19: 100nF, Capacitor_SMD:C_0402_1005Metric, F.Cu at (268.8, 353.7)
- added C2: 22pF, Capacitor_SMD:C_0402_1005Metric, F.Cu at (292.7, 469.6)
- added C20: 100nF, Capacitor_SMD:C_0402_1005Metric, F.Cu at (268.8, 306.5)
- added C21: 100nF, Capacitor_SMD:C_0402_1005Metric, F.Cu at (268.8, 282.8)
- added C22: 100nF, Capacitor_SMD:C_0402_1005Metric, F.Cu at (268.8, 271.7)
- added C23: 100nF, Capacitor_SMD:C_0402_1005Metric, F.Cu at (306.3, 265.4)
- added C24: 100nF, Capacitor_SMD:C_0402_1005Metric, F.Cu at (268.8, 377.3)
- added C25: 100nF, Capacitor_SMD:C_0402_1005Metric, F.Cu at (268.8, 366.1)
- added C26: 22uF, Capacitor_THT:C_Radial_D5.0mm_H11.0mm_P2.00mm, F.Cu at (264.0, 478.0)
- added C27: 100nF, Capacitor_SMD:C_0402_1005Metric, F.Cu at (298.3, 307.6)
- added C28: 100nF, Capacitor_SMD:C_0402_1005Metric, F.Cu at (290.5, 307.6)
- added C29: 100nF, Capacitor_SMD:C_0402_1005Metric, F.Cu at (298.3, 379.6)
- added C3: 100nF, Capacitor_SMD:C_0402_1005Metric, F.Cu at (244.9, 449.6)
- added C30: 100nF, Capacitor_SMD:C_0402_1005Metric, F.Cu at (298.3, 371.3)
- added C31: 100nF, Capacitor_SMD:C_0402_1005Metric, F.Cu at (290.5, 407.2)
- added C32: 100nF, Capacitor_SMD:C_0402_1005Metric, F.Cu at (290.4, 415.4)
- added C33: 100nF, Capacitor_SMD:C_0402_1005Metric, F.Cu at (268.8, 295.3)
- added C34: 100nF, Capacitor_SMD:C_0402_1005Metric, F.Cu at (314.3, 265.4)
- added C35: 100nF, Capacitor_SMD:C_0402_1005Metric, F.Cu at (298.4, 265.4)
- added C36: 100nF, Capacitor_SMD:C_0402_1005Metric, F.Cu at (290.3, 265.5)
- added C37: 100nF, Capacitor_SMD:C_0402_1005Metric, F.Cu at (268.8, 400.9)
- added C38: 100nF, Capacitor_SMD:C_0402_1005Metric, F.Cu at (268.9, 389.7)
- added C39: 100nF, Capacitor_SMD:C_0402_1005Metric, F.Cu at (268.8, 330.1)
- added C4: 100nF, Capacitor_SMD:C_0402_1005Metric, F.Cu at (401.9, 452.2)
- added C40: 100nF, Capacitor_SMD:C_0402_1005Metric, F.Cu at (268.8, 318.9)
- added C41: 22uF, Capacitor_THT:C_Radial_D5.0mm_H11.0mm_P2.00mm, F.Cu at (264.0, 474.0)
- added C42: 100nF, Capacitor_SMD:C_0402_1005Metric, F.Cu at (397.5, 348.3)
- added C43: 100nF, Capacitor_SMD:C_0402_1005Metric, F.Cu at (397.5, 340.1)
- added C44: 100nF, Capacitor_SMD:C_0402_1005Metric, F.Cu at (373.7, 271.3)
- added C45: 100nF, Capacitor_SMD:C_0402_1005Metric, F.Cu at (382.2, 271.3)
- added C46: 100nF, Capacitor_SMD:C_0402_1005Metric, F.Cu at (390.6, 271.3)
- added C47: 100nF, Capacitor_SMD:C_0402_1005Metric, F.Cu at (399.0, 271.3)
- added C48: 100nF, Capacitor_SMD:C_0402_1005Metric, F.Cu at (397.5, 314.5)
- added C49: 100nF, Capacitor_SMD:C_0402_1005Metric, F.Cu at (397.5, 322.9)
- added C5: 100nF, Capacitor_SMD:C_0402_1005Metric, F.Cu at (326.9, 452.2)
- added C50: 100nF, Capacitor_SMD:C_0402_1005Metric, F.Cu at (311.5, 460.3)
- added C51: 100nF, Capacitor_SMD:C_0402_1005Metric, F.Cu at (-213.8, 467.5)
- added C52: 100nF, Capacitor_SMD:C_0402_1005Metric, F.Cu at (-210.9, 445.9)
- added C53: 100nF, Capacitor_SMD:C_0402_1005Metric, F.Cu at (-210.9, 447.8)
- added C54: 100nF, Capacitor_SMD:C_0402_1005Metric, F.Cu at (-210.9, 449.8)
- added C55: 100nF, Capacitor_SMD:C_0402_1005Metric, F.Cu at (-210.9, 451.8)
- added C56: 100nF, Capacitor_SMD:C_0402_1005Metric, F.Cu at (-210.9, 453.7)
- added C57: 100nF, Capacitor_SMD:C_0402_1005Metric, F.Cu at (-210.9, 455.7)
- added C58: 100nF, Capacitor_SMD:C_0402_1005Metric, F.Cu at (244.9, 448.3)
- added C59: 100nF, Capacitor_SMD:C_0402_1005Metric, F.Cu at (386.8, 387.8)
- added C6: 100nF, Capacitor_SMD:C_0402_1005Metric, F.Cu at (341.9, 452.2)
- added C60: 100nF, Capacitor_SMD:C_0402_1005Metric, F.Cu at (382.8, 407.5)
- added C61: 100nF, Capacitor_SMD:C_0402_1005Metric, F.Cu at (378.8, 387.8)
- added C62: 100nF, Capacitor_SMD:C_0402_1005Metric, F.Cu at (374.8, 407.5)
- added C63: 100nF, Capacitor_SMD:C_0402_1005Metric, F.Cu at (370.8, 387.8)
- added C64: 100nF, Capacitor_SMD:C_0402_1005Metric, F.Cu at (366.8, 407.5)
- added C65: 100nF, Capacitor_SMD:C_0402_1005Metric, F.Cu at (362.8, 387.8)
- added C66: 100nF, Capacitor_SMD:C_0402_1005Metric, F.Cu at (358.8, 407.5)
- added C67: 100nF, Capacitor_SMD:C_0402_1005Metric, F.Cu at (354.8, 387.8)
- added C68: 100nF, Capacitor_SMD:C_0402_1005Metric, F.Cu at (350.8, 407.5)
- added C69: 100nF, Capacitor_SMD:C_0402_1005Metric, F.Cu at (346.8, 387.8)
- added C7: 100nF, Capacitor_SMD:C_0402_1005Metric, F.Cu at (356.9, 452.2)
- added C70: 100nF, Capacitor_SMD:C_0402_1005Metric, F.Cu at (342.8, 407.5)
- added C71: 100nF, Capacitor_SMD:C_0402_1005Metric, F.Cu at (338.8, 387.8)
- added C72: 100nF, Capacitor_SMD:C_0402_1005Metric, F.Cu at (334.8, 407.5)
- added C73: 100nF, Capacitor_SMD:C_0402_1005Metric, F.Cu at (330.8, 387.8)
- added C74: 100nF, Capacitor_SMD:C_0402_1005Metric, F.Cu at (326.8, 407.5)
- added C75: 100nF, Capacitor_SMD:C_0402_1005Metric, F.Cu at (386.8, 407.5)
- added C76: 100nF, Capacitor_SMD:C_0402_1005Metric, F.Cu at (382.8, 427.2)
- added C77: 100nF, Capacitor_SMD:C_0402_1005Metric, F.Cu at (378.8, 407.5)
- added C78: 100nF, Capacitor_SMD:C_0402_1005Metric, F.Cu at (374.8, 427.2)
- added C79: 100nF, Capacitor_SMD:C_0402_1005Metric, F.Cu at (370.8, 407.5)
- added C8: 100nF, Capacitor_SMD:C_0402_1005Metric, F.Cu at (371.9, 452.2)
- added C80: 100nF, Capacitor_SMD:C_0402_1005Metric, F.Cu at (366.8, 427.2)
- added C81: 100nF, Capacitor_SMD:C_0402_1005Metric, F.Cu at (362.8, 407.5)
- added C82: 100nF, Capacitor_SMD:C_0402_1005Metric, F.Cu at (358.8, 427.2)
- added C83: 100nF, Capacitor_SMD:C_0402_1005Metric, F.Cu at (354.8, 407.5)
- added C84: 100nF, Capacitor_SMD:C_0402_1005Metric, F.Cu at (350.8, 427.2)
- added C85: 100nF, Capacitor_SMD:C_0402_1005Metric, F.Cu at (346.8, 407.5)
- added C86: 100nF, Capacitor_SMD:C_0402_1005Metric, F.Cu at (342.8, 427.2)
- added C87: 100nF, Capacitor_SMD:C_0402_1005Metric, F.Cu at (338.8, 407.5)
- added C88: 100nF, Capacitor_SMD:C_0402_1005Metric, F.Cu at (334.8, 427.2)
- added C89: 100nF, Capacitor_SMD:C_0402_1005Metric, F.Cu at (330.8, 407.5)
- added C9: 100nF, Capacitor_SMD:C_0402_1005Metric, F.Cu at (386.9, 452.2)
- added C90: 100nF, Capacitor_SMD:C_0402_1005Metric, F.Cu at (326.8, 427.2)
- added C91: 100nF, Capacitor_SMD:C_0402_1005Metric, F.Cu at (-202.3, 451.8)
- added C92: 100nF, Capacitor_SMD:C_0402_1005Metric, F.Cu at (-202.3, 453.7)
- added C93: 100nF, Capacitor_SMD:C_0402_1005Metric, F.Cu at (-202.3, 455.7)
- added C94: 100nF, Capacitor_SMD:C_0402_1005Metric, F.Cu at (-202.3, 457.7)
- added C95: 100nF, Capacitor_SMD:C_0402_1005Metric, F.Cu at (-202.3, 459.6)
- added C96: 100nF, Capacitor_SMD:C_0402_1005Metric, F.Cu at (-202.3, 461.6)
- added C97: 22uF, Capacitor_THT:C_Radial_D5.0mm_H11.0mm_P2.00mm, F.Cu at (258.0, 478.0)
- added C98: 22uF, Capacitor_THT:C_Radial_D5.0mm_H11.0mm_P2.00mm, F.Cu at (258.0, 474.0)
- added C99: 100nF, Capacitor_SMD:C_0402_1005Metric, F.Cu at (301.2, 459.8)
- added D1: RX, LED_SMD:LED_0402_1005Metric, F.Cu at (236.5, 432.7)
- added D100: LED, LED_SMD:LED_0402_1005Metric, F.Cu at (358.7, 291.8)
- added D101: LED, LED_SMD:LED_0402_1005Metric, F.Cu at (355.2, 291.8)
- added D102: LED, LED_SMD:LED_0402_1005Metric, F.Cu at (351.7, 291.8)
- added D103: LED, LED_SMD:LED_0402_1005Metric, F.Cu at (348.2, 291.8)
- added D104: LED, LED_SMD:LED_0402_1005Metric, F.Cu at (344.7, 291.8)
- added D105: LED, LED_SMD:LED_0402_1005Metric, F.Cu at (341.2, 291.8)
- added D106: LED, LED_SMD:LED_0402_1005Metric, F.Cu at (337.7, 291.8)
- added D107: LED, LED_SMD:LED_0402_1005Metric, F.Cu at (334.2, 291.8)
- added D108: LED, LED_SMD:LED_0402_1005Metric, F.Cu at (330.7, 291.8)
- added D109: LED, LED_SMD:LED_0402_1005Metric, F.Cu at (327.2, 291.8)
- added D110: LED, LED_SMD:LED_0402_1005Metric, F.Cu at (323.7, 291.8)
- added D111: LED, LED_SMD:LED_0402_1005Metric, F.Cu at (320.2, 291.8)
- added D112: LED, LED_SMD:LED_0402_1005Metric, F.Cu at (316.7, 291.8)
- added D113: LED, LED_SMD:LED_0402_1005Metric, F.Cu at (313.2, 291.8)
- added D2: TX, LED_SMD:LED_0402_1005Metric, F.Cu at (236.5, 437.2)
- added D3: IND1, LED_SMD:LED_0402_1005Metric, F.Cu at (269.4, 456.5)
- added D30: LED, LED_SMD:LED_0402_1005Metric, F.Cu at (365.6, 337.4)
- added D31: LED, LED_SMD:LED_0402_1005Metric, F.Cu at (362.1, 337.4)
- added D32: LED, LED_SMD:LED_0402_1005Metric, F.Cu at (358.6, 337.4)
- added D33: LED, LED_SMD:LED_0402_1005Metric, F.Cu at (355.1, 337.4)
- added D34: LED, LED_SMD:LED_0402_1005Metric, F.Cu at (351.6, 337.4)
- added D35: LED, LED_SMD:LED_0402_1005Metric, F.Cu at (348.1, 337.4)
- added D36: LED, LED_SMD:LED_0402_1005Metric, F.Cu at (344.6, 337.4)
- added D37: LED, LED_SMD:LED_0402_1005Metric, F.Cu at (341.1, 337.4)
- added D38: LED, LED_SMD:LED_0402_1005Metric, F.Cu at (337.6, 337.4)
- added D39: LED, LED_SMD:LED_0402_1005Metric, F.Cu at (334.1, 337.4)
- added D4: PWR, LED_SMD:LED_0402_1005Metric, F.Cu at (237.2, 461.0)
- added D40: LED, LED_SMD:LED_0402_1005Metric, F.Cu at (330.6, 337.4)
- added D41: LED, LED_SMD:LED_0402_1005Metric, F.Cu at (327.1, 337.4)
- added D42: LED, LED_SMD:LED_0402_1005Metric, F.Cu at (323.6, 337.4)
- added D43: LED, LED_SMD:LED_0402_1005Metric, F.Cu at (320.1, 337.4)
- added D44: LED, LED_SMD:LED_0402_1005Metric, F.Cu at (316.6, 337.4)
- added D45: LED, LED_SMD:LED_0402_1005Metric, F.Cu at (313.1, 337.4)
- added D46: LED, LED_SMD:LED_0402_1005Metric, F.Cu at (365.6, 314.5)
- added D47: LED, LED_SMD:LED_0402_1005Metric, F.Cu at (362.1, 314.5)
- added D48: LED, LED_SMD:LED_0402_1005Metric, F.Cu at (358.6, 314.5)
- added D49: LED, LED_SMD:LED_0402_1005Metric, F.Cu at (355.1, 314.5)
- added D5: IND0, LED_SMD:LED_0402_1005Metric, F.Cu at (269.4, 461.0)
- added D50: LED, LED_SMD:LED_0402_1005Metric, F.Cu at (351.6, 314.5)
- added D51: LED, LED_SMD:LED_0402_1005Metric, F.Cu at (348.1, 314.5)
- added D52: LED, LED_SMD:LED_0402_1005Metric, F.Cu at (344.6, 314.5)
- added D53: LED, LED_SMD:LED_0402_1005Metric, F.Cu at (341.1, 314.5)
- added D54: LED, LED_SMD:LED_0402_1005Metric, F.Cu at (337.6, 314.5)
- added D55: LED, LED_SMD:LED_0402_1005Metric, F.Cu at (334.1, 314.5)
- added D56: LED, LED_SMD:LED_0402_1005Metric, F.Cu at (330.6, 314.5)
- added D57: LED, LED_SMD:LED_0402_1005Metric, F.Cu at (327.1, 314.5)
- added D58: LED, LED_SMD:LED_0402_1005Metric, F.Cu at (323.6, 314.5)
- added D59: LED, LED_SMD:LED_0402_1005Metric, F.Cu at (320.1, 314.5)
- added D6: D_Zener, Diode_SMD:D_SOD-123, F.Cu at (240.0, 473.0)
- added D60: LED, LED_SMD:LED_0402_1005Metric, F.Cu at (316.6, 314.5)
- added D61: LED, LED_SMD:LED_0402_1005Metric, F.Cu at (313.1, 314.5)
- added D62: LED, LED_SMD:LED_0402_1005Metric, F.Cu at (362.6, 378.5)
- added D63: LED, LED_SMD:LED_0402_1005Metric, F.Cu at (362.6, 375.0)
- added D64: LED, LED_SMD:LED_0402_1005Metric, F.Cu at (362.6, 371.5)
- added D65: LED, LED_SMD:LED_0402_1005Metric, F.Cu at (362.6, 368.0)
- added D66: LED, LED_SMD:LED_0402_1005Metric, F.Cu at (362.6, 364.5)
- added D67: LED, LED_SMD:LED_0402_1005Metric, F.Cu at (362.6, 361.0)
- added D68: LED, LED_SMD:LED_0402_1005Metric, F.Cu at (362.6, 357.5)
- added D69: LED, LED_SMD:LED_0402_1005Metric, F.Cu at (325.7, 378.5)
- added D7: PWR_USB, LED_SMD:LED_0402_1005Metric, F.Cu at (237.2, 456.5)
- added D70: LED, LED_SMD:LED_0402_1005Metric, F.Cu at (325.7, 375.0)
- added D71: LED, LED_SMD:LED_0402_1005Metric, F.Cu at (325.7, 371.5)
- added D72: LED, LED_SMD:LED_0402_1005Metric, F.Cu at (325.7, 368.0)
- added D73: LED, LED_SMD:LED_0402_1005Metric, F.Cu at (325.7, 364.5)
- added D74: LED, LED_SMD:LED_0402_1005Metric, F.Cu at (325.7, 361.0)
- added D75: LED, LED_SMD:LED_0402_1005Metric, F.Cu at (325.7, 357.5)
- added D76: LED, LED_SMD:LED_0402_1005Metric, F.Cu at (395.1, 436.7)
- added D77: LED, LED_SMD:LED_0402_1005Metric, F.Cu at (391.6, 436.7)
- added D78: LED, LED_SMD:LED_0402_1005Metric, F.Cu at (388.1, 436.7)
- added D79: LED, LED_SMD:LED_0402_1005Metric, F.Cu at (384.6, 436.7)
- added D80: LED, LED_SMD:LED_0402_1005Metric, F.Cu at (381.1, 436.7)
- added D81: LED, LED_SMD:LED_0402_1005Metric, F.Cu at (377.6, 436.7)
- added D82: LED, LED_SMD:LED_0402_1005Metric, F.Cu at (374.1, 436.7)
- added D83: LED, LED_SMD:LED_0402_1005Metric, F.Cu at (370.6, 436.7)
- added D84: LED, LED_SMD:LED_0402_1005Metric, F.Cu at (367.1, 436.7)
- added D85: LED, LED_SMD:LED_0402_1005Metric, F.Cu at (363.6, 436.7)
- added D86: LED, LED_SMD:LED_0402_1005Metric, F.Cu at (360.1, 436.7)
- added D87: LED, LED_SMD:LED_0402_1005Metric, F.Cu at (356.6, 436.7)
- added D88: LED, LED_SMD:LED_0402_1005Metric, F.Cu at (353.1, 436.7)
- added D89: LED, LED_SMD:LED_0402_1005Metric, F.Cu at (349.6, 436.7)
- added D90: LED, LED_SMD:LED_0402_1005Metric, F.Cu at (346.1, 436.7)
- added D91: LED, LED_SMD:LED_0402_1005Metric, F.Cu at (342.6, 436.7)
- added D92: LED, LED_SMD:LED_0402_1005Metric, F.Cu at (-82.2, 493.9)
- added D93: LED, LED_SMD:LED_0402_1005Metric, F.Cu at (289.1, 429.9)
- added D94: LED, LED_SMD:LED_0402_1005Metric, F.Cu at (289.1, 433.4)
- added D95: LED, LED_SMD:LED_0402_1005Metric, F.Cu at (289.1, 436.9)
- added D96: LED, LED_SMD:LED_0402_1005Metric, F.Cu at (289.1, 440.4)
- added D98: LED, LED_SMD:LED_0402_1005Metric, F.Cu at (365.7, 291.8)
- added D99: LED, LED_SMD:LED_0402_1005Metric, F.Cu at (362.2, 291.8)
- added F1: Fuse, Fuse:Fuseholder_Clip-5x20mm_Littelfuse_520_Inline_P20.50x5.80mm_D1.30mm_Horizontal, F.Cu at (231.8, 480.0)
- added J1: USB_B, Connector_USB:USB_B_OST_USB-B1HSxx_Horizontal, F.Cu at (231.6, 447.2)
- added J10: Conn_02x18_Odd_Even, Connector_PinSocket_2.54mm:PinSocket_2x18_P2.54mm_Horizontal, F.Cu at (342.7, 478.9)
- added J2: Conn_02x03_Odd_Even, Connector_PinHeader_2.54mm:PinHeader_2x03_P2.54mm_Vertical, F.Cu at (293.9, 481.2)
- added J3: Conn_02x08_Odd_Even, Connector_PinHeader_2.54mm:PinHeader_2x08_P2.54mm_Vertical, F.Cu at (246.3, 444.8)
- added J4: Conn_02x40_Odd_Even, Connector_PinHeader_2.54mm:PinHeader_2x40_P2.54mm_Horizontal, F.Cu at (325.8, 264.6)
- added J5: Conn_02x16_Odd_Even, Connector_PinSocket_2.54mm:PinSocket_2x16_P2.54mm_Horizontal, F.Cu at (420.5, 433.1)
- added J6: Conn_02x16_Odd_Even, Connector_PinSocket_2.54mm:PinSocket_2x16_P2.54mm_Horizontal, F.Cu at (420.5, 484.1)
- added J7: Conn_02x12_Odd_Even, Connector_PinSocket_2.54mm:PinSocket_2x12_P2.54mm_Vertical, F.Cu at (328.4, 560.1)
- added J8: Conn_02x24_Odd_Even, Connector_PinSocket_2.54mm:PinSocket_2x24_P2.54mm_Horizontal, F.Cu at (420.5, 354.4)
- added J9: Barrel_Jack_MountingPin, Connector_BarrelJack:BarrelJack_Horizontal, F.Cu at (231.0, 468.0)
- added Q129: IRLML6244, Package_TO_SOT_SMD:SOT-23, F.Cu at (365.6, 341.8)
- added Q130: IRLML6402, Package_TO_SOT_SMD:SOT-23, F.Cu at (365.6, 345.8)
- added Q131: IRLML6244, Package_TO_SOT_SMD:SOT-23, F.Cu at (362.1, 341.8)
- added Q132: IRLML6402, Package_TO_SOT_SMD:SOT-23, F.Cu at (362.1, 345.8)
- added Q133: IRLML6244, Package_TO_SOT_SMD:SOT-23, F.Cu at (358.6, 341.8)
- added Q134: IRLML6402, Package_TO_SOT_SMD:SOT-23, F.Cu at (358.6, 345.8)
- added Q135: IRLML6244, Package_TO_SOT_SMD:SOT-23, F.Cu at (355.1, 341.8)
- added Q136: IRLML6402, Package_TO_SOT_SMD:SOT-23, F.Cu at (355.1, 345.8)
- added Q137: IRLML6244, Package_TO_SOT_SMD:SOT-23, F.Cu at (351.6, 341.8)
- added Q138: IRLML6402, Package_TO_SOT_SMD:SOT-23, F.Cu at (351.6, 345.8)
- added Q139: IRLML6244, Package_TO_SOT_SMD:SOT-23, F.Cu at (348.1, 341.8)
- added Q140: IRLML6402, Package_TO_SOT_SMD:SOT-23, F.Cu at (348.1, 345.8)
- added Q141: IRLML6244, Package_TO_SOT_SMD:SOT-23, F.Cu at (344.6, 341.8)
- added Q142: IRLML6402, Package_TO_SOT_SMD:SOT-23, F.Cu at (344.6, 345.8)
- added Q143: IRLML6244, Package_TO_SOT_SMD:SOT-23, F.Cu at (341.1, 341.8)
- added Q144: IRLML6402, Package_TO_SOT_SMD:SOT-23, F.Cu at (341.1, 345.8)
- added Q145: IRLML6244, Package_TO_SOT_SMD:SOT-23, F.Cu at (337.6, 341.8)
- added Q146: IRLML6402, Package_TO_SOT_SMD:SOT-23, F.Cu at (337.6, 345.8)
- added Q147: IRLML6244, Package_TO_SOT_SMD:SOT-23, F.Cu at (334.1, 341.8)
- added Q148: IRLML6402, Package_TO_SOT_SMD:SOT-23, F.Cu at (334.1, 345.8)
- added Q149: IRLML6244, Package_TO_SOT_SMD:SOT-23, F.Cu at (330.6, 341.8)
- added Q150: IRLML6402, Package_TO_SOT_SMD:SOT-23, F.Cu at (330.6, 345.8)
- added Q151: IRLML6244, Package_TO_SOT_SMD:SOT-23, F.Cu at (327.1, 341.8)
- added Q152: IRLML6402, Package_TO_SOT_SMD:SOT-23, F.Cu at (327.1, 345.8)
- added Q153: IRLML6244, Package_TO_SOT_SMD:SOT-23, F.Cu at (323.6, 341.8)
- added Q154: IRLML6402, Package_TO_SOT_SMD:SOT-23, F.Cu at (323.6, 345.8)
- added Q155: IRLML6244, Package_TO_SOT_SMD:SOT-23, F.Cu at (320.1, 341.8)
- added Q156: IRLML6402, Package_TO_SOT_SMD:SOT-23, F.Cu at (320.1, 345.8)
- added Q157: IRLML6244, Package_TO_SOT_SMD:SOT-23, F.Cu at (316.6, 341.8)
- added Q158: IRLML6402, Package_TO_SOT_SMD:SOT-23, F.Cu at (316.6, 345.8)
- added Q159: IRLML6244, Package_TO_SOT_SMD:SOT-23, F.Cu at (313.1, 341.8)
- added Q160: IRLML6402, Package_TO_SOT_SMD:SOT-23, F.Cu at (313.1, 345.8)
- added Q161: IRLML6244, Package_TO_SOT_SMD:SOT-23, F.Cu at (365.6, 318.9)
- added Q162: IRLML6402, Package_TO_SOT_SMD:SOT-23, F.Cu at (365.6, 322.8)
- added Q163: IRLML6244, Package_TO_SOT_SMD:SOT-23, F.Cu at (362.1, 318.9)
- added Q164: IRLML6402, Package_TO_SOT_SMD:SOT-23, F.Cu at (362.1, 322.8)
- added Q165: IRLML6244, Package_TO_SOT_SMD:SOT-23, F.Cu at (358.6, 318.9)
- added Q166: IRLML6402, Package_TO_SOT_SMD:SOT-23, F.Cu at (358.6, 322.8)
- added Q167: IRLML6244, Package_TO_SOT_SMD:SOT-23, F.Cu at (355.1, 318.9)
- added Q168: IRLML6402, Package_TO_SOT_SMD:SOT-23, F.Cu at (355.1, 322.8)
- added Q169: IRLML6244, Package_TO_SOT_SMD:SOT-23, F.Cu at (351.6, 318.9)
- added Q170: IRLML6402, Package_TO_SOT_SMD:SOT-23, F.Cu at (351.6, 322.8)
- added Q171: IRLML6244, Package_TO_SOT_SMD:SOT-23, F.Cu at (348.1, 318.9)
- added Q172: IRLML6402, Package_TO_SOT_SMD:SOT-23, F.Cu at (348.1, 322.8)
- added Q173: IRLML6244, Package_TO_SOT_SMD:SOT-23, F.Cu at (344.6, 318.9)
- added Q174: IRLML6402, Package_TO_SOT_SMD:SOT-23, F.Cu at (344.6, 322.8)
- added Q175: IRLML6244, Package_TO_SOT_SMD:SOT-23, F.Cu at (341.1, 318.9)
- added Q176: IRLML6402, Package_TO_SOT_SMD:SOT-23, F.Cu at (341.1, 322.8)
- added Q177: IRLML6244, Package_TO_SOT_SMD:SOT-23, F.Cu at (337.6, 318.9)
- added Q178: IRLML6402, Package_TO_SOT_SMD:SOT-23, F.Cu at (337.6, 322.8)
- added Q179: IRLML6244, Package_TO_SOT_SMD:SOT-23, F.Cu at (334.1, 318.9)
- added Q180: IRLML6402, Package_TO_SOT_SMD:SOT-23, F.Cu at (334.1, 322.8)
- added Q181: IRLML6244, Package_TO_SOT_SMD:SOT-23, F.Cu at (330.6, 318.9)
- added Q182: IRLML6402, Package_TO_SOT_SMD:SOT-23, F.Cu at (330.6, 322.8)
- added Q183: IRLML6244, Package_TO_SOT_SMD:SOT-23, F.Cu at (327.1, 318.9)
- added Q184: IRLML6402, Package_TO_SOT_SMD:SOT-23, F.Cu at (327.1, 322.8)
- added Q185: IRLML6244, Package_TO_SOT_SMD:SOT-23, F.Cu at (323.6, 318.9)
- added Q186: IRLML6402, Package_TO_SOT_SMD:SOT-23, F.Cu at (323.6, 322.8)
- added Q187: IRLML6244, Package_TO_SOT_SMD:SOT-23, F.Cu at (320.1, 318.9)
- added Q188: IRLML6402, Package_TO_SOT_SMD:SOT-23, F.Cu at (320.1, 322.8)
- added Q189: IRLML6244, Package_TO_SOT_SMD:SOT-23, F.Cu at (316.6, 318.9)
- added Q190: IRLML6402, Package_TO_SOT_SMD:SOT-23, F.Cu at (316.6, 322.8)
- added Q191: IRLML6244, Package_TO_SOT_SMD:SOT-23, F.Cu at (313.1, 318.9)
- added Q192: IRLML6402, Package_TO_SOT_SMD:SOT-23, F.Cu at (313.1, 322.8)
- added Q193: IRLML6244, Package_TO_SOT_SMD:SOT-23, F.Cu at (358.2, 378.5)
- added Q194: IRLML6402, Package_TO_SOT_SMD:SOT-23, F.Cu at (354.3, 378.5)
- added Q195: IRLML6244, Package_TO_SOT_SMD:SOT-23, F.Cu at (358.2, 375.0)
- added Q196: IRLML6402, Package_TO_SOT_SMD:SOT-23, F.Cu at (354.3, 375.0)
- added Q197: IRLML6244, Package_TO_SOT_SMD:SOT-23, F.Cu at (358.2, 371.5)
- added Q198: IRLML6402, Package_TO_SOT_SMD:SOT-23, F.Cu at (354.3, 371.5)
- added Q199: IRLML6244, Package_TO_SOT_SMD:SOT-23, F.Cu at (358.2, 368.0)
- added Q2: IRF4905, Package_TO_SOT_THT:TO-220-3_Vertical, F.Cu at (244.5, 473.9)
- added Q200: IRLML6402, Package_TO_SOT_SMD:SOT-23, F.Cu at (354.3, 368.0)
- added Q201: IRLML6244, Package_TO_SOT_SMD:SOT-23, F.Cu at (358.2, 364.5)
- added Q202: IRLML6402, Package_TO_SOT_SMD:SOT-23, F.Cu at (354.3, 364.5)
- added Q203: IRLML6244, Package_TO_SOT_SMD:SOT-23, F.Cu at (358.2, 361.0)
- added Q204: IRLML6402, Package_TO_SOT_SMD:SOT-23, F.Cu at (354.3, 361.0)
- added Q205: IRLML6244, Package_TO_SOT_SMD:SOT-23, F.Cu at (358.2, 357.5)
- added Q206: IRLML6402, Package_TO_SOT_SMD:SOT-23, F.Cu at (354.3, 357.5)
- added Q207: IRLML6244, Package_TO_SOT_SMD:SOT-23, F.Cu at (321.3, 378.5)
- added Q208: IRLML6402, Package_TO_SOT_SMD:SOT-23, F.Cu at (317.4, 378.5)
- added Q209: IRLML6244, Package_TO_SOT_SMD:SOT-23, F.Cu at (321.3, 375.0)
- added Q210: IRLML6402, Package_TO_SOT_SMD:SOT-23, F.Cu at (317.4, 375.0)
- added Q211: IRLML6244, Package_TO_SOT_SMD:SOT-23, F.Cu at (321.3, 371.5)
- added Q212: IRLML6402, Package_TO_SOT_SMD:SOT-23, F.Cu at (317.4, 371.5)
- added Q213: IRLML6244, Package_TO_SOT_SMD:SOT-23, F.Cu at (321.3, 368.0)
- added Q214: IRLML6402, Package_TO_SOT_SMD:SOT-23, F.Cu at (317.4, 368.0)
- added Q215: IRLML6244, Package_TO_SOT_SMD:SOT-23, F.Cu at (321.3, 364.5)
- added Q216: IRLML6402, Package_TO_SOT_SMD:SOT-23, F.Cu at (317.4, 364.5)
- added Q217: IRLML6244, Package_TO_SOT_SMD:SOT-23, F.Cu at (321.3, 361.0)
- added Q218: IRLML6402, Package_TO_SOT_SMD:SOT-23, F.Cu at (317.4, 361.0)
- added Q219: IRLML6244, Package_TO_SOT_SMD:SOT-23, F.Cu at (321.3, 357.5)
- added Q220: IRLML6402, Package_TO_SOT_SMD:SOT-23, F.Cu at (317.4, 357.5)
- added Q221: IRLML6244, Package_TO_SOT_SMD:SOT-23, F.Cu at (395.1, 441.1)
- added Q222: IRLML6402, Package_TO_SOT_SMD:SOT-23, F.Cu at (395.1, 445.0)
- added Q223: IRLML6244, Package_TO_SOT_SMD:SOT-23, F.Cu at (391.6, 441.1)
- added Q224: IRLML6402, Package_TO_SOT_SMD:SOT-23, F.Cu at (391.6, 445.0)
- added Q225: IRLML6244, Package_TO_SOT_SMD:SOT-23, F.Cu at (388.1, 441.1)
- added Q226: IRLML6402, Package_TO_SOT_SMD:SOT-23, F.Cu at (388.1, 445.0)
- added Q227: IRLML6244, Package_TO_SOT_SMD:SOT-23, F.Cu at (384.6, 441.1)
- added Q228: IRLML6402, Package_TO_SOT_SMD:SOT-23, F.Cu at (384.6, 445.0)
- added Q229: IRLML6244, Package_TO_SOT_SMD:SOT-23, F.Cu at (381.1, 441.1)
- added Q230: IRLML6402, Package_TO_SOT_SMD:SOT-23, F.Cu at (381.1, 445.0)
- added Q231: IRLML6244, Package_TO_SOT_SMD:SOT-23, F.Cu at (377.6, 441.1)
- added Q232: IRLML6402, Package_TO_SOT_SMD:SOT-23, F.Cu at (377.6, 445.0)
- added Q233: IRLML6244, Package_TO_SOT_SMD:SOT-23, F.Cu at (374.1, 441.1)
- added Q234: IRLML6402, Package_TO_SOT_SMD:SOT-23, F.Cu at (374.1, 445.0)
- added Q235: IRLML6244, Package_TO_SOT_SMD:SOT-23, F.Cu at (370.6, 441.1)
- added Q236: IRLML6402, Package_TO_SOT_SMD:SOT-23, F.Cu at (370.6, 445.0)
- added Q237: IRLML6244, Package_TO_SOT_SMD:SOT-23, F.Cu at (367.1, 441.1)
- added Q238: IRLML6402, Package_TO_SOT_SMD:SOT-23, F.Cu at (367.1, 445.0)
- added Q239: IRLML6244, Package_TO_SOT_SMD:SOT-23, F.Cu at (363.6, 441.1)
- added Q240: IRLML6402, Package_TO_SOT_SMD:SOT-23, F.Cu at (363.6, 445.0)
- added Q241: IRLML6244, Package_TO_SOT_SMD:SOT-23, F.Cu at (360.1, 441.1)
- added Q242: IRLML6402, Package_TO_SOT_SMD:SOT-23, F.Cu at (360.1, 445.0)
- added Q243: IRLML6244, Package_TO_SOT_SMD:SOT-23, F.Cu at (356.6, 441.1)
- added Q244: IRLML6402, Package_TO_SOT_SMD:SOT-23, F.Cu at (356.6, 445.0)
- added Q245: IRLML6244, Package_TO_SOT_SMD:SOT-23, F.Cu at (353.1, 441.1)
- added Q246: IRLML6402, Package_TO_SOT_SMD:SOT-23, F.Cu at (353.1, 445.0)
- added Q247: IRLML6244, Package_TO_SOT_SMD:SOT-23, F.Cu at (349.6, 441.1)
- added Q248: IRLML6402, Package_TO_SOT_SMD:SOT-23, F.Cu at (349.6, 445.0)
- added Q249: IRLML6244, Package_TO_SOT_SMD:SOT-23, F.Cu at (346.1, 441.1)
- added Q250: IRLML6402, Package_TO_SOT_SMD:SOT-23, F.Cu at (346.1, 445.0)
- added Q251: IRLML6244, Package_TO_SOT_SMD:SOT-23, F.Cu at (342.6, 441.1)
- added Q252: IRLML6402, Package_TO_SOT_SMD:SOT-23, F.Cu at (342.6, 445.0)
- added Q253: IRLML6244, Package_TO_SOT_SMD:SOT-23, F.Cu at (-86.3, 495.3)
- added Q254: IRLML6244, Package_TO_SOT_SMD:SOT-23, F.Cu at (293.5, 429.9)
- added Q255: IRLML6402, Package_TO_SOT_SMD:SOT-23, F.Cu at (297.4, 429.9)
- added Q256: IRLML6244, Package_TO_SOT_SMD:SOT-23, F.Cu at (293.5, 433.4)
- added Q257: IRLML6402, Package_TO_SOT_SMD:SOT-23, F.Cu at (297.4, 433.4)
- added Q258: IRLML6244, Package_TO_SOT_SMD:SOT-23, F.Cu at (293.5, 436.9)
- added Q259: IRLML6402, Package_TO_SOT_SMD:SOT-23, F.Cu at (297.4, 436.9)
- added Q260: IRLML6244, Package_TO_SOT_SMD:SOT-23, F.Cu at (293.5, 440.4)
- added Q261: IRLML6402, Package_TO_SOT_SMD:SOT-23, F.Cu at (297.4, 440.4)
- added Q264: IRLML6244, Package_TO_SOT_SMD:SOT-23, F.Cu at (365.7, 296.2)
- added Q265: IRLML6402, Package_TO_SOT_SMD:SOT-23, F.Cu at (365.7, 300.1)
- added Q266: IRLML6244, Package_TO_SOT_SMD:SOT-23, F.Cu at (362.2, 296.2)
- added Q267: IRLML6402, Package_TO_SOT_SMD:SOT-23, F.Cu at (362.2, 300.1)
- added Q268: IRLML6244, Package_TO_SOT_SMD:SOT-23, F.Cu at (358.7, 296.2)
- added Q269: IRLML6402, Package_TO_SOT_SMD:SOT-23, F.Cu at (358.7, 300.1)
- added Q270: IRLML6244, Package_TO_SOT_SMD:SOT-23, F.Cu at (355.2, 296.2)
- added Q271: IRLML6402, Package_TO_SOT_SMD:SOT-23, F.Cu at (355.2, 300.1)
- added Q272: IRLML6244, Package_TO_SOT_SMD:SOT-23, F.Cu at (351.7, 296.2)
- added Q273: IRLML6402, Package_TO_SOT_SMD:SOT-23, F.Cu at (351.7, 300.1)
- added Q274: IRLML6244, Package_TO_SOT_SMD:SOT-23, F.Cu at (348.2, 296.2)
- added Q275: IRLML6402, Package_TO_SOT_SMD:SOT-23, F.Cu at (348.2, 300.1)
- added Q276: IRLML6244, Package_TO_SOT_SMD:SOT-23, F.Cu at (344.7, 296.2)
- added Q277: IRLML6402, Package_TO_SOT_SMD:SOT-23, F.Cu at (344.7, 300.1)
- added Q278: IRLML6244, Package_TO_SOT_SMD:SOT-23, F.Cu at (341.2, 296.2)
- added Q279: IRLML6402, Package_TO_SOT_SMD:SOT-23, F.Cu at (341.2, 300.1)
- added Q280: IRLML6244, Package_TO_SOT_SMD:SOT-23, F.Cu at (337.7, 296.2)
- added Q281: IRLML6402, Package_TO_SOT_SMD:SOT-23, F.Cu at (337.7, 300.1)
- added Q282: IRLML6244, Package_TO_SOT_SMD:SOT-23, F.Cu at (334.2, 296.2)
- added Q283: IRLML6402, Package_TO_SOT_SMD:SOT-23, F.Cu at (334.2, 300.1)
- added Q284: IRLML6244, Package_TO_SOT_SMD:SOT-23, F.Cu at (330.7, 296.2)
- added Q285: IRLML6402, Package_TO_SOT_SMD:SOT-23, F.Cu at (330.7, 300.1)
- added Q286: IRLML6244, Package_TO_SOT_SMD:SOT-23, F.Cu at (327.2, 296.2)
- added Q287: IRLML6402, Package_TO_SOT_SMD:SOT-23, F.Cu at (327.2, 300.1)
- added Q288: IRLML6244, Package_TO_SOT_SMD:SOT-23, F.Cu at (323.7, 296.2)
- added Q289: IRLML6402, Package_TO_SOT_SMD:SOT-23, F.Cu at (323.7, 300.1)
- added Q290: IRLML6244, Package_TO_SOT_SMD:SOT-23, F.Cu at (320.2, 296.2)
- added Q291: IRLML6402, Package_TO_SOT_SMD:SOT-23, F.Cu at (320.2, 300.1)
- added Q292: IRLML6244, Package_TO_SOT_SMD:SOT-23, F.Cu at (316.7, 296.2)
- added Q293: IRLML6402, Package_TO_SOT_SMD:SOT-23, F.Cu at (316.7, 300.1)
- added Q294: IRLML6244, Package_TO_SOT_SMD:SOT-23, F.Cu at (313.2, 296.2)
- added Q295: IRLML6402, Package_TO_SOT_SMD:SOT-23, F.Cu at (313.2, 300.1)
- added R1: 1K, Resistor_SMD:R_0402_1005Metric, F.Cu at (235.4, 432.7)
- added R10: 1K, Resistor_SMD:R_0402_1005Metric, F.Cu at (264.1, 439.2)
- added R100: 100K, Resistor_SMD:R_0402_1005Metric, F.Cu at (376.6, 438.2)
- added R101: 100K, Resistor_SMD:R_0402_1005Metric, F.Cu at (373.1, 438.2)
- added R102: 100K, Resistor_SMD:R_0402_1005Metric, F.Cu at (369.6, 438.2)
- added R103: 100K, Resistor_SMD:R_0402_1005Metric, F.Cu at (366.1, 438.2)
- added R104: 100K, Resistor_SMD:R_0402_1005Metric, F.Cu at (362.6, 438.2)
- added R105: 100K, Resistor_SMD:R_0402_1005Metric, F.Cu at (359.1, 438.2)
- added R106: 100K, Resistor_SMD:R_0402_1005Metric, F.Cu at (355.6, 438.2)
- added R107: 100K, Resistor_SMD:R_0402_1005Metric, F.Cu at (352.1, 438.2)
- added R108: 100K, Resistor_SMD:R_0402_1005Metric, F.Cu at (348.6, 438.2)
- added R109: 100K, Resistor_SMD:R_0402_1005Metric, F.Cu at (345.1, 438.2)
- added R11: 1K, Resistor_SMD:R_0402_1005Metric, F.Cu at (403.9, 452.2)
- added R110: 100K, Resistor_SMD:R_0402_1005Metric, F.Cu at (341.6, 438.2)
- added R111: 100K, Resistor_SMD:R_0402_1005Metric, F.Cu at (290.6, 430.9)
- added R112: 100K, Resistor_SMD:R_0402_1005Metric, F.Cu at (290.6, 434.4)
- added R113: 100K, Resistor_SMD:R_0402_1005Metric, F.Cu at (290.6, 437.9)
- added R114: 100K, Resistor_SMD:R_0402_1005Metric, F.Cu at (290.6, 441.4)
- added R115: 10K, Resistor_THT:R_Axial_DIN0207_L6.3mm_D2.5mm_P10.16mm_Horizontal, F.Cu at (240.9, 468.0)
- added R116: 10K, Resistor_SMD:R_0402_1005Metric, F.Cu at (-88.3, 317.2)
- added R117: 10K, Resistor_SMD:R_0402_1005Metric, F.Cu at (268.3, 436.3)
- added R118: 10K, Resistor_SMD:R_0402_1005Metric, F.Cu at (260.4, 436.3)
- added R119: 100K, Resistor_SMD:R_0402_1005Metric, F.Cu at (-88.3, 323.2)
- added R12: 10K, Resistor_SMD:R_0402_1005Metric, F.Cu at (405.9, 452.2)
- added R120: 100K, Resistor_SMD:R_0402_1005Metric, F.Cu at (-88.3, 325.2)
- added R121: 100K, Resistor_SMD:R_0402_1005Metric, F.Cu at (-88.3, 327.2)
- added R122: 100K, Resistor_SMD:R_0402_1005Metric, F.Cu at (-88.3, 329.2)
- added R123: 100K, Resistor_SMD:R_0402_1005Metric, F.Cu at (-88.3, 331.1)
- added R124: 100K, Resistor_SMD:R_0402_1005Metric, F.Cu at (-88.3, 333.1)
- added R125: 100K, Resistor_SMD:R_0402_1005Metric, F.Cu at (-88.3, 335.1)
- added R126: 100K, Resistor_SMD:R_0402_1005Metric, F.Cu at (-88.3, 337.1)
- added R127: 100K, Resistor_SMD:R_0402_1005Metric, F.Cu at (364.7, 293.3)
- added R128: 100K, Resistor_SMD:R_0402_1005Metric, F.Cu at (361.2, 293.3)
- added R129: 100K, Resistor_SMD:R_0402_1005Metric, F.Cu at (357.7, 293.3)
- added R13: 10K, Resistor_SMD:R_0402_1005Metric, F.Cu at (330.9, 452.2)
- added R130: 100K, Resistor_SMD:R_0402_1005Metric, F.Cu at (354.2, 293.3)
- added R131: 100K, Resistor_SMD:R_0402_1005Metric, F.Cu at (350.7, 293.3)
- added R132: 100K, Resistor_SMD:R_0402_1005Metric, F.Cu at (347.2, 293.3)
- added R133: 100K, Resistor_SMD:R_0402_1005Metric, F.Cu at (343.7, 293.3)
- added R134: 100K, Resistor_SMD:R_0402_1005Metric, F.Cu at (340.2, 293.3)
- added R135: 100K, Resistor_SMD:R_0402_1005Metric, F.Cu at (336.7, 293.3)
- added R136: 100K, Resistor_SMD:R_0402_1005Metric, F.Cu at (333.2, 293.3)
- added R137: 100K, Resistor_SMD:R_0402_1005Metric, F.Cu at (329.7, 293.3)
- added R138: 100K, Resistor_SMD:R_0402_1005Metric, F.Cu at (326.2, 293.3)
- added R139: 100K, Resistor_SMD:R_0402_1005Metric, F.Cu at (322.7, 293.3)
- added R14: 1K, Resistor_SMD:R_0402_1005Metric, F.Cu at (328.9, 452.2)
- added R140: 100K, Resistor_SMD:R_0402_1005Metric, F.Cu at (319.2, 293.3)
- added R141: 100K, Resistor_SMD:R_0402_1005Metric, F.Cu at (315.7, 293.3)
- added R142: 1000, Resistor_SMD:R_0402_1005Metric, F.Cu at (365.6, 338.9)
- added R143: 1000, Resistor_SMD:R_0402_1005Metric, F.Cu at (366.6, 339.0)
- added R144: 1000, Resistor_SMD:R_0402_1005Metric, F.Cu at (362.1, 338.9)
- added R145: 1000, Resistor_SMD:R_0402_1005Metric, F.Cu at (363.1, 339.0)
- added R146: 1000, Resistor_SMD:R_0402_1005Metric, F.Cu at (358.6, 338.9)
- added R147: 1000, Resistor_SMD:R_0402_1005Metric, F.Cu at (359.6, 339.0)
- added R148: 1000, Resistor_SMD:R_0402_1005Metric, F.Cu at (355.1, 338.9)
- added R149: 1000, Resistor_SMD:R_0402_1005Metric, F.Cu at (356.1, 339.0)
- added R15: 10K, Resistor_SMD:R_0402_1005Metric, F.Cu at (345.9, 452.2)
- added R150: 1000, Resistor_SMD:R_0402_1005Metric, F.Cu at (351.6, 338.9)
- added R151: 1000, Resistor_SMD:R_0402_1005Metric, F.Cu at (352.6, 339.0)
- added R152: 1000, Resistor_SMD:R_0402_1005Metric, F.Cu at (348.1, 338.9)
- added R153: 1000, Resistor_SMD:R_0402_1005Metric, F.Cu at (349.1, 339.0)
- added R154: 1000, Resistor_SMD:R_0402_1005Metric, F.Cu at (344.6, 338.9)
- added R155: 1000, Resistor_SMD:R_0402_1005Metric, F.Cu at (345.6, 339.0)
- added R156: 1000, Resistor_SMD:R_0402_1005Metric, F.Cu at (341.1, 338.9)
- added R157: 1000, Resistor_SMD:R_0402_1005Metric, F.Cu at (342.1, 339.0)
- added R158: 1000, Resistor_SMD:R_0402_1005Metric, F.Cu at (337.6, 338.9)
- added R159: 1000, Resistor_SMD:R_0402_1005Metric, F.Cu at (338.6, 339.0)
- added R16: 1K, Resistor_SMD:R_0402_1005Metric, F.Cu at (343.9, 452.2)
- added R160: 1000, Resistor_SMD:R_0402_1005Metric, F.Cu at (334.1, 338.9)
- added R161: 1000, Resistor_SMD:R_0402_1005Metric, F.Cu at (335.1, 339.0)
- added R162: 1000, Resistor_SMD:R_0402_1005Metric, F.Cu at (330.6, 338.9)
- added R163: 1000, Resistor_SMD:R_0402_1005Metric, F.Cu at (331.6, 339.0)
- added R164: 1000, Resistor_SMD:R_0402_1005Metric, F.Cu at (327.1, 338.9)
- added R165: 1000, Resistor_SMD:R_0402_1005Metric, F.Cu at (328.1, 339.0)
- added R166: 1000, Resistor_SMD:R_0402_1005Metric, F.Cu at (323.6, 338.9)
- added R167: 1000, Resistor_SMD:R_0402_1005Metric, F.Cu at (324.6, 339.0)
- added R168: 1000, Resistor_SMD:R_0402_1005Metric, F.Cu at (320.1, 338.9)
- added R169: 1000, Resistor_SMD:R_0402_1005Metric, F.Cu at (321.1, 339.0)
- added R17: 10K, Resistor_SMD:R_0402_1005Metric, F.Cu at (360.9, 452.2)
- added R170: 1000, Resistor_SMD:R_0402_1005Metric, F.Cu at (316.6, 338.9)
- added R171: 1000, Resistor_SMD:R_0402_1005Metric, F.Cu at (317.6, 339.0)
- added R172: 1000, Resistor_SMD:R_0402_1005Metric, F.Cu at (313.1, 338.9)
- added R173: 1000, Resistor_SMD:R_0402_1005Metric, F.Cu at (314.1, 339.0)
- added R174: 1000, Resistor_SMD:R_0402_1005Metric, F.Cu at (365.6, 316.0)
- added R175: 1000, Resistor_SMD:R_0402_1005Metric, F.Cu at (366.6, 316.0)
- added R176: 1000, Resistor_SMD:R_0402_1005Metric, F.Cu at (362.1, 316.0)
- added R177: 1000, Resistor_SMD:R_0402_1005Metric, F.Cu at (363.1, 316.0)
- added R178: 1000, Resistor_SMD:R_0402_1005Metric, F.Cu at (358.6, 316.0)
- added R179: 1000, Resistor_SMD:R_0402_1005Metric, F.Cu at (359.6, 316.0)
- added R18: 1K, Resistor_SMD:R_0402_1005Metric, F.Cu at (358.9, 452.2)
- added R180: 1000, Resistor_SMD:R_0402_1005Metric, F.Cu at (355.1, 316.0)
- added R181: 1000, Resistor_SMD:R_0402_1005Metric, F.Cu at (356.1, 316.0)
- added R182: 1000, Resistor_SMD:R_0402_1005Metric, F.Cu at (351.6, 316.0)
- added R183: 1000, Resistor_SMD:R_0402_1005Metric, F.Cu at (352.6, 316.0)
- added R184: 1000, Resistor_SMD:R_0402_1005Metric, F.Cu at (348.1, 316.0)
- added R185: 1000, Resistor_SMD:R_0402_1005Metric, F.Cu at (349.1, 316.0)
- added R186: 1000, Resistor_SMD:R_0402_1005Metric, F.Cu at (344.6, 316.0)
- added R187: 1000, Resistor_SMD:R_0402_1005Metric, F.Cu at (345.6, 316.0)
- added R188: 1000, Resistor_SMD:R_0402_1005Metric, F.Cu at (341.1, 316.0)
- added R189: 1000, Resistor_SMD:R_0402_1005Metric, F.Cu at (342.1, 316.0)
- added R19: 10K, Resistor_SMD:R_0402_1005Metric, F.Cu at (375.9, 452.2)
- added R190: 1000, Resistor_SMD:R_0402_1005Metric, F.Cu at (337.6, 316.0)
- added R191: 1000, Resistor_SMD:R_0402_1005Metric, F.Cu at (338.6, 316.0)
- added R192: 1000, Resistor_SMD:R_0402_1005Metric, F.Cu at (334.1, 316.0)
- added R193: 1000, Resistor_SMD:R_0402_1005Metric, F.Cu at (335.1, 316.0)
- added R194: 1000, Resistor_SMD:R_0402_1005Metric, F.Cu at (330.6, 316.0)
- added R195: 1000, Resistor_SMD:R_0402_1005Metric, F.Cu at (331.6, 316.0)
- added R196: 1000, Resistor_SMD:R_0402_1005Metric, F.Cu at (327.1, 316.0)
- added R197: 1000, Resistor_SMD:R_0402_1005Metric, F.Cu at (328.1, 316.0)
- added R198: 1000, Resistor_SMD:R_0402_1005Metric, F.Cu at (323.6, 316.0)
- added R199: 1000, Resistor_SMD:R_0402_1005Metric, F.Cu at (324.6, 316.0)
- added R2: 1K, Resistor_SMD:R_0402_1005Metric, F.Cu at (235.4, 437.2)
- added R20: 1K, Resistor_SMD:R_0402_1005Metric, F.Cu at (373.9, 452.2)
- added R200: 1000, Resistor_SMD:R_0402_1005Metric, F.Cu at (320.1, 316.0)
- added R201: 1000, Resistor_SMD:R_0402_1005Metric, F.Cu at (321.1, 316.0)
- added R202: 1000, Resistor_SMD:R_0402_1005Metric, F.Cu at (316.6, 316.0)
- added R203: 1000, Resistor_SMD:R_0402_1005Metric, F.Cu at (317.6, 316.0)
- added R204: 1000, Resistor_SMD:R_0402_1005Metric, F.Cu at (313.1, 316.0)
- added R205: 1000, Resistor_SMD:R_0402_1005Metric, F.Cu at (314.1, 316.0)
- added R206: 1000, Resistor_SMD:R_0402_1005Metric, F.Cu at (361.1, 378.5)
- added R207: 1000, Resistor_SMD:R_0402_1005Metric, F.Cu at (361.1, 379.5)
- added R208: 1000, Resistor_SMD:R_0402_1005Metric, F.Cu at (361.1, 375.0)
- added R209: 1000, Resistor_SMD:R_0402_1005Metric, F.Cu at (361.1, 376.0)
- added R21: 10K, Resistor_SMD:R_0402_1005Metric, F.Cu at (390.9, 452.2)
- added R210: 1000, Resistor_SMD:R_0402_1005Metric, F.Cu at (361.1, 371.5)
- added R211: 1000, Resistor_SMD:R_0402_1005Metric, F.Cu at (361.1, 372.5)
- added R212: 1000, Resistor_SMD:R_0402_1005Metric, F.Cu at (361.1, 368.0)
- added R213: 1000, Resistor_SMD:R_0402_1005Metric, F.Cu at (361.1, 369.0)
- added R214: 1000, Resistor_SMD:R_0402_1005Metric, F.Cu at (361.1, 364.5)
- added R215: 1000, Resistor_SMD:R_0402_1005Metric, F.Cu at (361.1, 365.5)
- added R216: 1000, Resistor_SMD:R_0402_1005Metric, F.Cu at (361.1, 361.0)
- added R217: 1000, Resistor_SMD:R_0402_1005Metric, F.Cu at (361.1, 362.0)
- added R218: 1000, Resistor_SMD:R_0402_1005Metric, F.Cu at (361.1, 357.5)
- added R219: 1000, Resistor_SMD:R_0402_1005Metric, F.Cu at (361.1, 358.5)
- added R22: 1K, Resistor_SMD:R_0402_1005Metric, F.Cu at (388.9, 452.2)
- added R220: 1000, Resistor_SMD:R_0402_1005Metric, F.Cu at (324.2, 378.5)
- added R221: 1000, Resistor_SMD:R_0402_1005Metric, F.Cu at (324.2, 379.5)
- added R222: 1000, Resistor_SMD:R_0402_1005Metric, F.Cu at (324.2, 375.0)
- added R223: 1000, Resistor_SMD:R_0402_1005Metric, F.Cu at (324.2, 376.0)
- added R224: 1000, Resistor_SMD:R_0402_1005Metric, F.Cu at (324.2, 371.5)
- added R225: 1000, Resistor_SMD:R_0402_1005Metric, F.Cu at (324.2, 372.5)
- added R226: 1000, Resistor_SMD:R_0402_1005Metric, F.Cu at (324.2, 368.0)
- added R227: 1000, Resistor_SMD:R_0402_1005Metric, F.Cu at (324.2, 369.0)
- added R228: 1000, Resistor_SMD:R_0402_1005Metric, F.Cu at (324.2, 364.5)
- added R229: 1000, Resistor_SMD:R_0402_1005Metric, F.Cu at (324.2, 365.5)
- added R23: 1K, Resistor_SMD:R_0402_1005Metric, F.Cu at (286.2, 469.7)
- added R230: 1000, Resistor_SMD:R_0402_1005Metric, F.Cu at (324.2, 361.0)
- added R231: 1000, Resistor_SMD:R_0402_1005Metric, F.Cu at (324.2, 362.0)
- added R232: 1000, Resistor_SMD:R_0402_1005Metric, F.Cu at (324.2, 357.5)
- added R233: 1000, Resistor_SMD:R_0402_1005Metric, F.Cu at (324.2, 358.5)
- added R234: 1000, Resistor_SMD:R_0402_1005Metric, F.Cu at (395.1, 438.2)
- added R235: 1000, Resistor_SMD:R_0402_1005Metric, F.Cu at (396.1, 438.2)
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Routing:
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- added copper zone on B.Cu, net GND
- added copper zone on F.Cu, net GND
- added copper zone on In1.Cu, net GND
- added copper zone on In2.Cu, net GND
Other:
- board size 215 x 160 mm -> 215 x 232 mm
- copper layers 2 -> 4

Commit message: finished IO PCB placement
Parts:
- moved C107 613.1 mm to (400.9, 331.2), turned to 90 degrees
- moved C92 604.9 mm to (397.3, 373.7), turned to 90 degrees
- moved C91 603.6 mm to (397.3, 382.2), turned to 90 degrees
- moved C94 541.3 mm to (338.6, 437.2)
- moved C93 533.0 mm to (330.4, 437.2)
- moved U87 523.7 mm to (405.0, 333.5), turned to 90 degrees
- moved U17 503.5 mm to (328.4, 442.4)
- moved Q253 498.5 mm to (396.1, 369.6), turned to 90 degrees
- moved U85 497.9 mm to (402.5, 384.1), turned to 90 degrees
- moved D92 495.7 mm to (396.6, 365.6), turned to -90 degrees
- moved R266 495.4 mm to (395.6, 365.6), turned to 90 degrees
- moved U86 491.5 mm to (402.5, 375.6), turned to 90 degrees
- moved R116 489.6 mm to (400.9, 335.8), turned to 90 degrees
- moved C51 471.8 mm to (223.2, 289.7), turned to 90 degrees
- moved C53 470.5 mm to (223.0, 266.0), turned to 90 degrees
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