File: hardware/io/io.kicad_sch (KiCad schematic)
At the start: 13 parts, among them U1 AS6C4008-55PCN, U10 SST39SF040, U2 SST39SF040, U3 74HC245, U4 ATmega2560-16A, U5 FT232RL, U6 SST39SF040, U7 SST39SF040, U8 SST39SF040, U9 SST39SF040, Y1 Crystal_GND24

Commit message: small fixes on register fabric
Connections:
- net +5V: now also U3.20 (VCC)
- net GND: now also U3.10 (GND)
- net OPROM_D08: now reaches U9.13 (D0)
- net OPROM_D09: now reaches U9.14 (D1)
- net OPROM_D10: now reaches U9.15 (D2)
- net OPROM_D11: now reaches U9.17 (D3)
- net OPROM_D12: now reaches U9.18 (D4)
- net OPROM_D13: now reaches U9.19 (D5)
- net OPROM_D14: now reaches U9.20 (D6)
- net OPROM_D15: now reaches U9.21 (D7)
- net PROM_D08: now reaches U6.13 (D0)
- net PROM_D09: now reaches U6.14 (D1)
- net PROM_D10: now reaches U6.15 (D2)
- net PROM_D11: now reaches U6.17 (D3)
- net PROM_D12: now reaches U6.18 (D4)
- net PROM_D13: now reaches U6.19 (D5)
- net PROM_D14: now reaches U6.20 (D6)
- net PROM_D15: now reaches U6.21 (D7)
- net PROM_D16: now reaches U8.13 (D0)
- net PROM_D17: now reaches U8.14 (D1)
- net PROM_D18: now reaches U8.15 (D2)
- net PROM_D19: now reaches U8.17 (D3)
- net PROM_D20: now reaches U8.18 (D4)
- net PROM_D21: now reaches U8.19 (D5)
- net PROM_D22: now reaches U8.20 (D6)
- net PROM_D23: now reaches U8.21 (D7)
- net PROM_D00: now reaches U2.13 (D0)
- net PROM_D01: now reaches U2.14 (D1)
- net PROM_D02: now reaches U2.15 (D2)
- net PROM_D03: now reaches U2.17 (D3)
- net PROM_D04: now reaches U2.18 (D4)
- net PROM_D05: now reaches U2.19 (D5)
- net PROM_D06: now reaches U2.20 (D6)
- net PROM_D07: now reaches U2.21 (D7)
- net OPROM_D00: now reaches U10.13 (D0)
- net OPROM_D01: now reaches U10.14 (D1)
- net OPROM_D02: now reaches U10.15 (D2)
- net OPROM_D03: now reaches U10.17 (D3)
- net OPROM_D04: now reaches U10.18 (D4)
- net OPROM_D05: now reaches U10.19 (D5)
- net OPROM_D06: now reaches U10.20 (D6)
- net OPROM_D07: now reaches U10.21 (D7)
- net PROM_D24: now reaches U7.13 (D0)
- net PROM_D25: now reaches U7.14 (D1)
- net PROM_D26: now reaches U7.15 (D2)
- net PROM_D27: now reaches U7.17 (D3)
- net PROM_D28: now reaches U7.18 (D4)
- net PROM_D29: now reaches U7.19 (D5)
- net PROM_D30: now reaches U7.20 (D6)
- net PROM_D31: now reaches U7.21 (D7)
- net RAM_D00: now reaches U1.13 (DQ0)
- net RAM_D01: now reaches U1.14 (DQ1)
- net RAM_D02: now reaches U1.15 (DQ2)
- net RAM_D03: now reaches U1.17 (DQ3)
- net RAM_D04: now reaches U1.18 (DQ4)
- net RAM_D05: now reaches U1.19 (DQ5)
- net RAM_D06: now reaches U1.20 (DQ6)
- net RAM_D07: now reaches U1.21 (DQ7)
Other:
- moved on the sheet: U3

Commit message: did a good chunk of IO PCB schematic
Parts:
- added C10: 330nF, Capacitor_SMD:C_0402_1005Metric, symbol Device:C
- added C11, C3, C4, C5, C6, C7, C8, C9: 100nF, Capacitor_SMD:C_0402_1005Metric, symbol Device:C
- added D1: RX, LED_SMD:LED_0402_1005Metric, symbol Device:LED
- added D2: TX, LED_SMD:LED_0402_1005Metric, symbol Device:LED
- added D30, D31, D32, D33, D34, D35, D36, D37, D38, D39, D40, D41, D42, D43, D44, D45, D46, D47, D48, D49, D50, D51, D52, D53, D54, D55, D56, D57, D58, D59, D60, D61, D62, D63, D64, D65, D66, D67, D68, D69, D70, D71, D72, D73, D74, D75: LED, LED_SMD:LED_0402_1005Metric, symbol Device:LED
- added J1: USB_B, symbol Connector:USB_B
- added J2: Conn_02x03_Odd_Even, Connector_PinHeader_2.54mm:PinHeader_2x03_P2.54mm_Vertical, symbol Connector_Generic:Conn_02x03_Odd_Even
- added J3: Conn_02x08_Odd_Even, Connector_PinHeader_2.54mm:PinHeader_2x08_P2.54mm_Vertical, symbol Connector_Generic:Conn_02x08_Odd_Even
- added J4: Conn_02x40_Odd_Even, Connector_PinSocket_2.54mm:PinSocket_2x40_P2.54mm_Horizontal, symbol Connector_Generic:Conn_02x40_Odd_Even
- added J5, J6: Conn_02x16_Odd_Even, Connector_PinHeader_2.54mm:PinHeader_2x16_P2.54mm_Horizontal, symbol Connector_Generic:Conn_02x16_Odd_Even
- added J8: Conn_02x24_Odd_Even, Connector_PinHeader_2.54mm:PinHeader_2x24_P2.54mm_Horizontal, symbol Connector_Generic:Conn_02x24_Odd_Even
- added Q129, Q131, Q133, Q135, Q137, Q139, Q141, Q143, Q145, Q147, Q149, Q151, Q153, Q155, Q157, Q159, Q161, Q163, Q165, Q167, Q169, Q171, Q173, Q175, Q177, Q179, Q181, Q183, Q185, Q187, Q189, Q191, Q193, Q195, Q197, Q199, Q201, Q203, Q205, Q207, Q209, Q211, Q213, Q215, Q217, Q219: IRLML6244, Package_TO_SOT_SMD:SOT-23, symbol Transistor_FET:IRLML6244
- added Q130, Q132, Q134, Q136, Q138, Q140, Q142, Q144, Q146, Q148, Q150, Q152, Q154, Q156, Q158, Q160, Q162, Q164, Q166, Q168, Q170, Q172, Q174, Q176, Q178, Q180, Q182, Q184, Q186, Q188, Q190, Q192, Q194, Q196, Q198, Q200, Q202, Q204, Q206, Q208, Q210, Q212, Q214, Q216, Q218, Q220: IRLML6402, Package_TO_SOT_SMD:SOT-23, symbol Transistor_FET:IRLML6402
- added R1, R10, R11, R14, R16, R18, R2, R20, R22, R23, R24, R25, R26, R3, R33, R34, R35, R4, R5, R6, R7, R8, R9: 1K, Resistor_SMD:R_0402_1005Metric, symbol Device:R
- added R12, R13, R15, R17, R19, R21, R27, R28, R29, R30, R31, R32, R36, R42, R43, R44, R45, R46, R47, R48, R49, R50, R51, R52, R53: 10K, Resistor_SMD:R_0402_1005Metric, symbol Device:R
- added R142, R143, R144, R145, R146, R147, R148, R149, R150, R151, R152, R153, R154, R155, R156, R157, R158, R159, R160, R161, R162, R163, R164, R165, R166, R167, R168, R169, R170, R171, R172, R173, R174, R175, R176, R177, R178, R179, R180, R181, R182, R183, R184, R185, R186, R187, R188, R189, R190, R191, R192, R193, R194, R195, R196, R197, R198, R199, R200, R201, R202, R203, R204, R205, R206, R207, R208, R209, R210, R211, R212, R213, R214, R215, R216, R217, R218, R219, R220, R221, R222, R223, R224, R225, R226, R227, R228, R229, R230, R231, R232, R233: 1000, Resistor_SMD:R_0402_1005Metric, symbol Device:R
- added R37, R38, R39, R40, R41, R54, R55, R56, R57, R58, R59, R60, R61, R62, R63, R64, R65, R66, R67, R68, R69, R70, R71, R72, R73, R74, R75, R76, R77, R78, R79, R80, R81, R82, R83, R84, R85, R86, R87, R88, R89, R90, R91, R92, R93, R94: 100K, Resistor_SMD:R_0402_1005Metric, symbol Device:R
- added SW1, SW2, SW3, SW4, SW5, SW6, SW7: SW_Push, symbol Switch:SW_Push
- added SW8, SW9: SW_DIP_x03, symbol Switch:SW_DIP_x03
- added U11, U26: 74HC138, Package_SO:SOIC-16_3.9x9.9mm_P1.27mm, symbol 74xx:74HC138
- added U12, U13, U14, U15, U16, U17, U19, U20, U21, U22, U23, U24, U29, U30, U31, U32, U33, U34, U35, U36, U37, U38, U39, U40, U41: 74HC245, symbol 74xx:74HC245
- added U18: 74HC14, Package_SO:SOIC-14_3.9x8.7mm_P1.27mm, symbol 74xx:74HC14
- added U42, U43: 74HCT238, symbol 74xx:74HCT238
- added U50, U51, U52, U53, U54, U55, U56, U57: 74LS157, Package_SO:SOIC-16_3.9x9.9mm_P1.27mm, symbol 74xx:74LS157
- C1, C2: value C -> 22pF
Connections:
- net RAM_A17 is gone; now on an unnamed net: U1.30 (A17)
- net RAM_A18 is gone; now on an unnamed net: U1.1 (A18)
- net +5V: now also U4.10 (VCC), U4.100 (AVCC), U4.31 (VCC), U4.61 (VCC), U4.80 (VCC), C10.2, D1.2 (A), D2.2 (A), J2.2 (Pin_2), J4.71 (Pin_71), J4.73 (Pin_73), J4.75 (Pin_75)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
- net GND: now also U4.11 (GND), U4.32 (GND), U4.62 (GND), U4.81 (GND), U4.99 (GND), U5.18 (GND), U5.21 (GND), U5.25 (AGND), U5.26 (TEST), U5.7 (GND), C10.1, C11.1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
- net OPROM_A0: now also U13.18 (B0), U32.18 (B0)
- net OPROM_A1: now also U13.17 (B1), U32.17 (B1)
- net OPROM_A10: now also U14.16 (B2), U33.16 (B2)
- net OPROM_A11: now also U14.15 (B3), U33.15 (B3)
- net OPROM_A12: now also U14.14 (B4), U33.14 (B4)
- net OPROM_A13: now also U14.13 (B5), U33.13 (B5)
- net OPROM_A14: now also U14.12 (B6), U33.12 (B6)
- net OPROM_A15: now also U14.11 (B7), U33.11 (B7)
- net OPROM_A16: now also R30.2, R33.2
- net OPROM_A17: now also R31.2, R34.2
- net OPROM_A18: now also R32.2, R35.2
- net OPROM_A2: now also U13.16 (B2), U32.16 (B2)
- net OPROM_A3: now also U13.15 (B3), U32.15 (B3)
- net OPROM_A4: now also U13.14 (B4), U32.14 (B4)
- net OPROM_A5: now also U13.13 (B5), U32.13 (B5)
- net OPROM_A6: now also U13.12 (B6), U32.12 (B6)
- net OPROM_A7: now also U13.11 (B7), U32.11 (B7)
- net OPROM_A8: now also U14.18 (B0), U33.18 (B0)
- net OPROM_A9: now also U14.17 (B1), U33.17 (B1)
- net OPROM_D00: now also U23.18 (B0), U40.18 (B0)
- net OPROM_D01: now also U23.17 (B1), U40.17 (B1)
- net OPROM_D02: now also U23.16 (B2), U40.16 (B2)
- net OPROM_D03: now also U23.15 (B3), U40.15 (B3)
- net OPROM_D04: now also U23.14 (B4), U40.14 (B4)
- net OPROM_D05: now also U23.13 (B5), U40.13 (B5)
- net OPROM_D06: now also U23.12 (B6), U40.12 (B6)
- net OPROM_D07: now also U23.11 (B7), U40.11 (B7)
- net OPROM_D08: now also U24.18 (B0), U41.18 (B0)
- net OPROM_D09: now also U24.17 (B1), U41.17 (B1)
- net OPROM_D10: now also U24.16 (B2), U41.16 (B2)
- net OPROM_D11: now also U24.15 (B3), U41.15 (B3)
- net OPROM_D12: now also U24.14 (B4), U41.14 (B4)
- net OPROM_D13: now also U24.13 (B5), U41.13 (B5)
- net OPROM_D14: now also U24.12 (B6), U41.12 (B6)
- net OPROM_D15: now also U24.11 (B7), U41.11 (B7)
- net PROM_A0: now also U3.18 (B0), U29.18 (B0)
- net PROM_A1: now also U3.17 (B1), U29.17 (B1)
- net PROM_A10: now also U12.16 (B2), U30.16 (B2)
- net PROM_A11: now also U12.15 (B3), U30.15 (B3)
- net PROM_A12: now also U12.14 (B4), U30.14 (B4)
- net PROM_A13: now also U12.13 (B5), U30.13 (B5)
- net PROM_A14: now also U12.12 (B6), U30.12 (B6)
- net PROM_A15: now also U12.11 (B7), U30.11 (B7)
- net PROM_A16: now also R24.2, R27.2
- net PROM_A17: now also R25.2, R28.2
- net PROM_A18: now also R26.2, R29.2
- net PROM_A2: now also U3.16 (B2), U29.16 (B2)
- net PROM_A3: now also U3.15 (B3), U29.15 (B3)
- net PROM_A4: now also U3.14 (B4), U29.14 (B4)
- net PROM_A5: now also U3.13 (B5), U29.13 (B5)
- net PROM_A6: now also U3.12 (B6), U29.12 (B6)
- new net: D32.1 (K), R147.2
- new net: Q205.3 (D), Q206.1 (G), R218.1
- new net: Q187.3 (D), Q188.1 (G), R200.1
- new net: U15.19 (CE), U16.19 (CE), U26.12 (~{Y3})
- new net: U13.19 (CE), U14.19 (CE), U26.13 (~{Y2})
- new net: Q129.3 (D), Q130.1 (G), R142.1
- new net: Q185.3 (D), Q186.1 (G), R198.1
- new net: Q183.3 (D), Q184.1 (G), R196.1
- new net: Q199.3 (D), Q200.1 (G), R212.1
- new net: Q201.3 (D), Q202.1 (G), R214.1
- new net: R11.2, R12.2, SW1.2
- new net: U11.9 (~{Y6}), U23.19 (CE)
- new net: J3.12 (Pin_12), R8.2
- new net: D30.1 (K), R143.2
- new net: D67.1 (K), R217.2
- new net: Q153.3 (D), Q154.1 (G), R166.1
- new net: Q217.3 (D), Q218.1 (G), R230.1
- new net: C8.2, R20.1, U18.11
- new net: D33.1 (K), R149.2
- new net: D59.1 (K), R201.2
- new net: Q167.3 (D), Q168.1 (G), R180.1
- new net: Q197.3 (D), Q198.1 (G), R210.1
- new net: D2.1 (K), R2.2
- new net: U11.12 (~{Y3}), U20.19 (CE)
- new net: R50.1, U32.1 (A->B)
- new net: D36.1 (K), R155.2
- new net: Q179.3 (D), Q180.1 (G), R192.1
- new net: Q131.3 (D), Q132.1 (G), R144.1
- new net: D57.1 (K), R197.2
- new net: D56.1 (K), R195.2
- new net: Q133.3 (D), Q134.1 (G), R146.1
- new net: Q135.3 (D), Q136.1 (G), R148.1
- new net: C6.2, R16.1, U18.5
- new net: Q145.3 (D), Q146.1 (G), R158.1
- new net: R15.2, R16.2, SW3.2
- new net: Q175.3 (D), Q176.1 (G), R188.1
- new net: D47.1 (K), R177.2
- new net: D35.1 (K), R153.2
- new net: D65.1 (K), R213.2
- new net: R51.1, U33.1 (A->B)
- new net: R43.1, U13.1 (A->B)
- new net: R19.2, R20.2, SW5.2
- new net: Q213.3 (D), Q214.1 (G), R226.1
- new net: D43.1 (K), R169.2
- new net: D51.1 (K), R185.2
- new net: U32.19 (CE), U33.19 (CE), U42.13 (Y2)
- new net: D41.1 (K), R165.2
- new net: Q139.3 (D), Q140.1 (G), R152.1
- new net: R49.1, U30.1 (A->B)
- new net: Q173.3 (D), Q174.1 (G), R186.1
- new net: Q169.3 (D), Q170.1 (G), R182.1
- new net: Q151.3 (D), Q152.1 (G), R164.1
- new net: Q147.3 (D), Q148.1 (G), R160.1
- new net: D73.1 (K), R229.2
- new net: Q143.3 (D), Q144.1 (G), R156.1
- new net: Q163.3 (D), Q164.1 (G), R176.1
- new net: Q137.3 (D), Q138.1 (G), R150.1
- new net: D48.1 (K), R179.2
- new net: D53.1 (K), R189.2
- new net: Q171.3 (D), Q172.1 (G), R184.1
- new net: Q177.3 (D), Q178.1 (G), R190.1
- new net: D31.1 (K), R145.2
- new net: D50.1 (K), R183.2
- new net: R46.1, U14.1 (A->B)
- new net: R44.1, U15.1 (A->B)
- new net: D49.1 (K), R181.2
- new net: Q191.3 (D), Q192.1 (G), R204.1
- new net: Q141.3 (D), Q142.1 (G), R154.1
- new net: C4.2, R11.1, U18.1
- new net: D60.1 (K), R203.2
- new net: Q195.3 (D), Q196.1 (G), R208.1
- new net: D62.1 (K), R207.2
- new net: D38.1 (K), R159.2
- new net: Q159.3 (D), Q160.1 (G), R172.1
- new net: J3.10 (Pin_10), R7.2
- new net: J3.14 (Pin_14), R9.2
- new net: J3.16 (Pin_16), R10.2
- new net: J3.2 (Pin_2), R3.2
- new net: J3.4 (Pin_4), R4.2
- new net: J3.6 (Pin_6), R5.2
- new net: J3.8 (Pin_8), R6.2
- new net: Q181.3 (D), Q182.1 (G), R194.1
- new net: U11.13 (~{Y2}), U19.19 (CE)
- new net: R48.1, U29.1 (A->B)
- new net: U29.19 (CE), U30.19 (CE), U42.14 (Y1)
- new net: U40.19 (CE), U43.9 (Y6)
- new net: Q207.3 (D), Q208.1 (G), R220.1
- new net: D34.1 (K), R151.2
- new net: Q189.3 (D), Q190.1 (G), R202.1
- new net: D72.1 (K), R227.2
- new net: C7.2, R18.1, U18.9
- new net: D61.1 (K), R205.2
- new net: D63.1 (K), R209.2
- new net: U11.10 (~{Y5}), U22.19 (CE)
- new net: R52.1, U36.1 (A->B)
- new net: Q203.3 (D), Q204.1 (G), R216.1
- new net: D74.1 (K), R231.2
- new net: U39.19 (CE), U43.10 (Y5)
- new net: U38.19 (CE), U43.11 (Y4)
- new net: U35.19 (CE), U43.12 (Y3)
- new net: U34.19 (CE), U43.13 (Y2)
- new net: U31.19 (CE), U43.14 (Y1)
- new net: U41.19 (CE), U43.7 (Y7)
- new net: R45.1, U16.1 (A->B)
- new net: D68.1 (K), R219.2
- new net: U36.19 (CE), U37.19 (CE), U42.12 (Y3)
- new net: Q211.3 (D), Q212.1 (G), R224.1
- new net: D64.1 (K), R211.2
- new net: D75.1 (K), R233.2
- new net: R33.1, SW9.1
- new net: D69.1 (K), R221.2
- new net: D71.1 (K), R225.2
- new net: Q157.3 (D), Q158.1 (G), R170.1
- new net: Q149.3 (D), Q150.1 (G), R162.1
- new net: R53.1, U37.1 (A->B)
- new net: Q193.3 (D), Q194.1 (G), R206.1
- new net: Q161.3 (D), Q162.1 (G), R174.1
- new net: U11.7 (~{Y7}), U24.19 (CE)
- new net: R24.1, SW8.1
- new net: D54.1 (K), R191.2
- new net: D42.1 (K), R167.2
- new net: R47.1, U12.1 (A->B)
- new net: D55.1 (K), R193.2
- new net: R17.2, R18.2, SW4.2
- new net: D44.1 (K), R171.2
- new net: Q219.3 (D), Q220.1 (G), R232.1
- new net: R26.1, SW8.3
- new net: D45.1 (K), R173.2
- new net: D37.1 (K), R157.2
- new net: D1.1 (K), R1.2
- new net: C5.2, R14.1, U18.3
- new net: Q215.3 (D), Q216.1 (G), R228.1
- new net: Q165.3 (D), Q166.1 (G), R178.1
- new net: D66.1 (K), R215.2
- new net: R21.2, R22.2, SW6.2
- new net: D46.1 (K), R175.2
- new net: D58.1 (K), R199.2
- new net: D40.1 (K), R163.2
- new net: R35.1, SW9.3
- new net: Q209.3 (D), Q210.1 (G), R222.1
- new net: U11.11 (~{Y4}), U21.19 (CE)
- new net: U11.14 (~{Y1}), U17.19 (CE)
- new net: D52.1 (K), R187.2
- new net: Q155.3 (D), Q156.1 (G), R168.1
- new net: D39.1 (K), R161.2
- new net: R34.1, SW9.2
- new net: D70.1 (K), R223.2
- new net: C9.2, R22.1, U18.13
- new net: R13.2, R14.2, SW2.2
- new net: R25.1, SW8.2
- new net ALU_A0: J4.21 (Pin_21), J8.3 (Pin_3)
- new net ALU_A1: J4.23 (Pin_23), J8.5 (Pin_5)
- new net ALU_A2: J4.25 (Pin_25), J8.7 (Pin_7)
- new net ALU_A3: J4.27 (Pin_27), J8.9 (Pin_9)
- new net ALU_A4: J4.29 (Pin_29), J8.13 (Pin_13)
- new net ALU_A5: J4.31 (Pin_31), J8.15 (Pin_15)
- new net ALU_A6: J4.33 (Pin_33), J8.17 (Pin_17)
- new net ALU_A7: J4.35 (Pin_35), J8.19 (Pin_19)
- new net ALU_B0: J8.4 (Pin_4), U50.4 (Za)
- new net ALU_B1: J8.6 (Pin_6), U50.7 (Zb)
- new net ALU_B2: J8.8 (Pin_8), U50.9 (Zc)
- new net ALU_B3: J8.10 (Pin_10), U50.12 (Zd)
- new net ALU_B4: J8.14 (Pin_14), U51.4 (Za)
- new net ALU_B5: J8.16 (Pin_16), U51.7 (Zb)
- new net ALU_B6: J8.18 (Pin_18), U51.9 (Zc)
- new net ALU_B7: J8.20 (Pin_20), U51.12 (Zd)
- new net ALU_CEN: J8.35 (Pin_35)
- new net ALU_CIN: J8.33 (Pin_33)
- new net ALU_COUT: J4.8 (Pin_8), J8.27 (Pin_27)
- new net ALU_NEG: J4.6 (Pin_6), J8.25 (Pin_25)
- new net ALU_OP0: D72.2 (A), J8.39 (Pin_39), Q214.3 (D)
- new net ALU_OP1: D73.2 (A), D74.2 (A), J8.41 (Pin_41), Q216.3 (D), Q218.3 (D)
- new net ALU_OP2: J8.43 (Pin_43)
- new net ALU_OVF: J4.10 (Pin_10), J8.29 (Pin_29)
- new net ALU_RES0: J8.24 (Pin_24), U56.2 (I0a)
- new net ALU_RES1: J8.26 (Pin_26), U56.5 (I0b)
- new net ALU_RES2: J8.28 (Pin_28), U56.11 (I0c)
- new net ALU_RES3: J8.30 (Pin_30), U56.14 (I0d)
- new net ALU_RES4: J8.34 (Pin_34), U57.2 (I0a)
- new net ALU_RES5: J8.36 (Pin_36), U57.5 (I0b)
- new net ALU_RES6: J8.38 (Pin_38), U57.11 (I0c)
- new net ALU_RES7: J8.40 (Pin_40), U57.14 (I0d)
- new net ALU_ZERO: J4.4 (Pin_4), J8.23 (Pin_23)
- new net ARBIT_ASRC_SEL0: U26.1 (A0), U42.1 (A0)
- new net ARBIT_ASRC_SEL1: U26.2 (A1), U42.2 (A1)
- new net ARBIT_DDIR_SEL: U17.1 (A->B), U19.1 (A->B), U20.1 (A->B), U21.1 (A->B), U22.1 (A->B), U23.1 (A->B), U24.1 (A->B)
- new net ARBIT_DSRC_SEL0: U11.1 (A0), U43.1 (A0)
- new net ARBIT_DSRC_SEL1: U11.2 (A1), U43.2 (A1)
- new net ARBIT_DSRC_SEL2: U11.3 (A2), U43.3 (A2)
- new net CTRL_ADRSEL: Q207.1 (G), R88.1, U40.9 (A7)
- new net CTRL_ALUOP0: Q213.1 (G), R91.1, U41.4 (A2)
- new net CTRL_ALUOP1: Q215.1 (G), Q217.1 (G), R92.1, R93.1, U41.5 (A3)
- new net CTRL_ALUOP2: U41.6 (A4)
- new net CTRL_CRYEN: Q219.1 (G), R94.1, U41.7 (A5)
- new net CTRL_FWEN: Q205.1 (G), R87.1, U40.8 (A6)
- new net CTRL_HALT: Q201.1 (G), R85.1, U40.6 (A4)
- new net CTRL_IOREN: Q195.1 (G), R82.1, U40.3 (A1)
- new net CTRL_IOWEN: Q197.1 (G), R83.1, U40.4 (A2)
- new net CTRL_OPSEL: Q203.1 (G), R86.1, U40.7 (A5)
- new net CTRL_PCSSEL: Q199.1 (G), R84.1, U40.5 (A3)
- new net CTRL_REGWEN: Q193.1 (G), R81.1, U40.2 (A0)
- new net CTRL_RESSEL: Q209.1 (G), R89.1, U41.2 (A0)
- new net CTRL_ZINV: Q211.1 (G), R90.1, U41.3 (A1)
- new net INS_IMM0: Q129.1 (G), R37.1, U34.2 (A0)
- new net INS_IMM1: Q131.1 (G), R38.1, U34.3 (A1)
- new net INS_IMM10: Q149.1 (G), R59.1, U35.4 (A2)
- new net INS_IMM11: Q151.1 (G), R60.1, U35.5 (A3)
- new net INS_IMM12: Q153.1 (G), R61.1, U35.6 (A4)
- new net INS_IMM13: Q155.1 (G), R62.1, U35.7 (A5)
- new net INS_IMM14: Q157.1 (G), R63.1, U35.8 (A6)
- new net INS_IMM15: Q159.1 (G), R64.1, U35.9 (A7)
- new net INS_IMM2: Q133.1 (G), R39.1, U34.4 (A2)
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Other:
- note added: "Output from Muxer"
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
Commit message: IO PCB schematic REV A done?
Parts:
- removed C10: 330nF, Capacitor_SMD:C_0402_1005Metric, symbol Device:C
- removed U17, U31: 74HC245, symbol 74xx:74HC245
- added C12, C13, C14, C15, C16, C17, C18, C19, C20, C21, C22, C23, C24, C25, C27, C28, C29, C30, C31, C32, C33, C34, C35, C36, C37, C38, C39, C40, C42, C43, C44, C45, C46, C47, C48, C49, C50, C51, C52, C53, C54, C55, C56, C57, C58, C59, C60, C61, C62, C63, C64, C65, C66, C67, C68, C69, C70, C71, C72, C73, C74, C75, C76, C77, C78, C79, C80, C81, C82, C83, C84, C85, C86, C87, C88, C89, C90, C91, C92, C93, C94, C95, C96: 100nF, Capacitor_SMD:C_0402_1005Metric, symbol Device:C
- added D100, D101, D102, D103, D104, D105, D106, D107, D108, D109, D110, D111, D112, D113, D76, D77, D78, D79, D80, D81, D82, D83, D84, D85, D86, D87, D88, D89, D90, D91, D92, D93, D94, D95, D96, D98, D99: LED, LED_SMD:LED_0402_1005Metric, symbol Device:LED
- added D3, D4, D5: RX, LED_SMD:LED_0402_1005Metric, symbol Device:LED
- added D6: D_Zener, Diode_SMD:D_SOD-123, symbol Device:D_Zener
- added F1: Fuse, Fuse:Fuseholder_Clip-5x20mm_Littelfuse_520_Inline_P20.50x5.80mm_D1.30mm_Horizontal, symbol Device:Fuse
- added J10: Conn_02x18_Odd_Even, Connector_PinSocket_2.54mm:PinSocket_2x18_P2.54mm_Horizontal, symbol Connector_Generic:Conn_02x18_Odd_Even
- added J7: Conn_02x12_Odd_Even, Connector_PinHeader_2.54mm:PinHeader_2x12_P2.54mm_Vertical, symbol Connector_Generic:Conn_02x12_Odd_Even
- added J9: Barrel_Jack_MountingPin, Connector_BarrelJack:BarrelJack_Horizontal, symbol Connector:Barrel_Jack_MountingPin
- added Q2: IRF4905, Package_TO_SOT_THT:TO-220-3_Vertical, symbol Transistor_FET:IRF4905
- added Q221, Q223, Q225, Q227, Q229, Q231, Q233, Q235, Q237, Q239, Q241, Q243, Q245, Q247, Q249, Q251, Q253, Q254, Q256, Q258, Q260, Q264, Q266, Q268, Q270, Q272, Q274, Q276, Q278, Q280, Q282, Q284, Q286, Q288, Q290, Q292, Q294: IRLML6244, Package_TO_SOT_SMD:SOT-23, symbol Transistor_FET:IRLML6244
- added Q222, Q224, Q226, Q228, Q230, Q232, Q234, Q236, Q238, Q240, Q242, Q244, Q246, Q248, Q250, Q252, Q255, Q257, Q259, Q261, Q265, Q267, Q269, Q271, Q273, Q275, Q277, Q279, Q281, Q283, Q285, Q287, Q289, Q291, Q293, Q295: IRLML6402, Package_TO_SOT_SMD:SOT-23, symbol Transistor_FET:IRLML6402
- added R100, R101, R102, R103, R104, R105, R106, R107, R108, R109, R110, R111, R112, R113, R114, R119, R120, R121, R122, R123, R124, R125, R126, R127, R128, R129, R130, R131, R132, R133, R134, R135, R136, R137, R138, R139, R140, R141, R307, R95, R96, R97, R98, R99: 100K, Resistor_SMD:R_0402_1005Metric, symbol Device:R
- added R115: 10K, Resistor_THT:R_Axial_DIN0207_L6.3mm_D2.5mm_P10.16mm_Horizontal, symbol Device:R
- added R116, R117, R118: 10K, Resistor_SMD:R_0402_1005Metric, symbol Device:R
- added R234, R235, R236, R237, R238, R239, R240, R241, R242, R243, R244, R245, R246, R247, R248, R249, R250, R251, R252, R253, R254, R255, R256, R257, R258, R259, R260, R261, R262, R263, R264, R265, R266, R267, R268, R269, R270, R271, R272, R273, R274, R277, R278, R279, R280, R281, R282, R283, R284, R285, R286, R287, R288, R289, R290, R291, R292, R293, R294, R295, R296, R297, R298, R299, R300, R301, R302, R303, R304, R305, R306, R308, R309: 1000, Resistor_SMD:R_0402_1005Metric, symbol Device:R
- added R310, R311, R312: 1K, Resistor_SMD:R_0402_1005Metric, symbol Device:R
- added U17, U25, U27, U28, U31, U44, U45, U46, U47, U48, U49, U58, U59, U60, U61, U62, U63, U64, U65, U66, U67, U68, U69, U70, U71, U72, U73, U74, U75, U76, U77, U78, U79, U80, U85, U86, U91, U92: 74HC00, Package_SO:SOIC-14_3.9x8.7mm_P1.27mm, symbol 74xx:74HC00
- added U81, U82, U83, U84: 74LS157, Package_SO:SOIC-16_3.9x9.9mm_P1.27mm, symbol 74xx:74LS157
- added U87, U89, U90: 74HC245, Package_SO:TSSOP-20_4.4x6.5mm_P0.65mm, symbol 74xx:74HC245
- added U88: 74HCT238, Package_SO:SOIC-16_3.9x9.9mm_P1.27mm, symbol 74xx:74HCT238
- C1, C2: footprint (none) -> Capacitor_SMD:C_0402_1005Metric
- J1: footprint (none) -> Connector_USB:USB_B_OST_USB-B1HSxx_Horizontal; now not fitted; now left out of the parts list
- J2, J3, J4: now not fitted; now left out of the parts list
- J5, J6: now not fitted
- SW1, SW2, SW3, SW4, SW5, SW6, SW7: footprint (none) -> Button_Switch_THT:SW_PUSH_6mm_H5mm; now not fitted; now left out of the parts list
- SW8, SW9: footprint (none) -> Package_DIP:DIP-6_W7.62mm; now not fitted; now left out of the parts list
- U12, U13, U14, U15, U16, U19, U20, U21, U22, U23, U24, U29, U3, U30, U32, U33, U34, U35, U36, U37, U38, U39, U40, U41: footprint (none) -> Package_SO:TSSOP-20_4.4x6.5mm_P0.65mm
- U42, U43: footprint (none) -> Package_SO:SOIC-16_3.9x9.9mm_P1.27mm
Connections:
- net ALU_CEN is gone; now on net S_CTRL_CRYEN: J8.35 (Pin_35)
- net ALU_CIN is gone; now on net RFAB_COUT: J8.33 (Pin_33)
- net ARBIT_D0 is gone; now on net IOBUS_DATA0: U19.2 (A0), U20.2 (A0), U21.2 (A0), U22.2 (A0), U23.2 (A0), U24.2 (A0), U4.97 (PF0)
- net ARBIT_D1 is gone; now on net IOBUS_DATA1: U19.3 (A1), U20.3 (A1), U21.3 (A1), U22.3 (A1), U23.3 (A1), U24.3 (A1), U4.96 (PF1)
- net ARBIT_D2 is gone; now on net IOBUS_DATA2: U19.4 (A2), U20.4 (A2), U21.4 (A2), U22.4 (A2), U23.4 (A2), U24.4 (A2), U4.95 (PF2)
- net ARBIT_D3 is gone; now on net IOBUS_DATA3: U19.5 (A3), U20.5 (A3), U21.5 (A3), U22.5 (A3), U23.5 (A3), U24.5 (A3), U4.94 (PF3)
- net ARBIT_D4 is gone; now on net IOBUS_DATA4: U19.6 (A4), U20.6 (A4), U21.6 (A4), U22.6 (A4), U23.6 (A4), U24.6 (A4), U4.93 (PF4)
- net ARBIT_D5 is gone; now on net IOBUS_DATA5: U19.7 (A5), U20.7 (A5), U21.7 (A5), U22.7 (A5), U23.7 (A5), U24.7 (A5), U4.92 (PF5)
- net ARBIT_D6 is gone; now on net IOBUS_DATA6: U19.8 (A6), U20.8 (A6), U21.8 (A6), U22.8 (A6), U23.8 (A6), U24.8 (A6), U4.91 (PF6)
- net ARBIT_D7 is gone; now on net IOBUS_DATA7: U19.9 (A7), U20.9 (A7), U21.9 (A7), U22.9 (A7), U23.9 (A7), U24.9 (A7), U4.90 (PF7)
- net PC0_WEN is gone; now on net +5V: J5.27 (Pin_27)
- net PC1_!CLR is gone; now on net S_NRST_CPU: J6.29 (Pin_29)
- net PC1_CLK is gone; now on net CLK2: J6.25 (Pin_25)
- net PC1_WEN is gone; now on net +5V: J6.27 (Pin_27)
- net RAM_D00 is gone; now on net IOBUS_DATA0: U1.13 (DQ0)
- net RAM_D01 is gone; now on net IOBUS_DATA1: U1.14 (DQ1)
- net RAM_D02 is gone; now on net IOBUS_DATA2: U1.15 (DQ2)
- net RAM_D03 is gone; now on net IOBUS_DATA3: U1.17 (DQ3)
- net RAM_D04 is gone; now on net IOBUS_DATA4: U1.18 (DQ4)
- net RAM_D05 is gone; now on net IOBUS_DATA5: U1.19 (DQ5)
- net RAM_D06 is gone; now on net IOBUS_DATA6: U1.20 (DQ6)
- net RAM_D07 is gone; now on net IOBUS_DATA7: U1.21 (DQ7)
- net RFAB_!CLR is gone; now on net S_NRST_CPU: J4.65 (Pin_65)
- net RFAB_FWEN is gone; now on net S_CTRL_FWEN: J4.78 (Pin_78)
- net RFAB_RSEL00 is gone; now on net S_INS_REG_OP00: J4.58 (Pin_58)
- net RFAB_RSEL01 is gone; now on net S_INS_REG_OP01: J4.60 (Pin_60)
- net RFAB_RSEL02 is gone; now on net S_INS_REG_OP02: J4.62 (Pin_62)
- net RFAB_RSEL10 is gone; now on net S_INS_REG_OP10: J4.57 (Pin_57)
- net RFAB_RSEL11 is gone; now on net S_INS_REG_OP11: J4.59 (Pin_59)
- net RFAB_RSEL12 is gone; now on net S_INS_REG_OP12: J4.61 (Pin_61)
- net RFAB_RWEN is gone; now on net S_CTRL_REGWEN: J4.76 (Pin_76)
- net RFAB_WSEL0 is gone; now on net S_INS_REG_DEST0: J4.66 (Pin_66)
- net RFAB_WSEL1 is gone; now on net S_INS_REG_DEST1: J4.68 (Pin_68)
- net RFAB_WSEL2 is gone; now on net S_INS_REG_DEST2: J4.70 (Pin_70)
- net +5V: now also C12.2, C13.2, C14.2, C15.2, C16.2, C17.2, C18.2, C19.2, C20.2, C21.2, C22.2, C23.2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
- net ALU_ZERO: now also U85.1, U85.4
- net ARBIT_ASRC_SEL0: now also U4.35 (PL0)
- net ARBIT_ASRC_SEL1: now also U4.36 (PL1)
- net ARBIT_CLK0: now also Q254.1 (G), R111.1
- net ARBIT_CLK1: now also Q256.1 (G), R112.1
- net ALU_A0 renamed RFAB_R00
- net ALU_A1 renamed RFAB_R01
- net ALU_A2 renamed RFAB_R02
- net ALU_A3 renamed RFAB_R03
- net ALU_A4 renamed RFAB_R04
- net ALU_A5 renamed RFAB_R05
- net ALU_A6 renamed RFAB_R06
- net ALU_A7 renamed RFAB_R07
- net ALU_OP0 renamed S_CTRL_ALUOP0
- net ALU_OP1 renamed S_CTRL_ALUOP1
- net ALU_OP2 renamed S_CTRL_ALUOP2
- net ARBIT_HALTED renamed PCINCR_OVF
- net PC0_!CLR renamed S_NRST_CPU
- net PC0_CLK renamed CLK2
- net RFAB_CLK renamed CLK1
- new net: Q264.3 (D), Q265.1 (G), R277.1
- new net: Q256.3 (D), Q257.1 (G), R269.1
- new net: D87.1 (K), R257.2
- new net: U59.13, U59.8
- new net: U59.3, U59.5, U59.9, U60.1, U60.2
- new net: Q237.3 (D), Q238.1 (G), R250.1
- new net: Q270.3 (D), Q271.1 (G), R283.1
- new net: D104.1 (K), R290.2
- new net: U75.3, U75.5, U75.9, U76.1, U76.2
- new net: U76.3, U77.1, U77.4
- new net: D3.2 (A), R310.2
- new net: D98.1 (K), R278.2
- new net: D92.1 (K), Q253.3 (D)
- new net: D96.1 (K), R274.2
- new net: Q239.3 (D), Q240.1 (G), R252.1
- new net: Q229.3 (D), Q230.1 (G), R242.1
- new net: U64.3, U65.1, U65.4
- new net: U65.3, U65.5, U65.9, U66.1, U66.2
- new net: Q280.3 (D), Q281.1 (G), R293.1
- new net: D6.2 (A), Q2.1 (G), R115.1
- new net: F1.2, Q2.2 (D)
- new net: Q278.3 (D), Q279.1 (G), R291.1
- new net: Q247.3 (D), Q248.1 (G), R260.1
- new net: U65.12, U65.6
- new net: U65.13, U65.8
- new net: Q251.3 (D), Q252.1 (G), R264.1
- new net: U48.3, U49.1, U49.4
- new net: U49.3, U49.5, U49.9, U58.1, U58.2
- new net: U49.12, U49.6
- new net: U46.3, U47.1, U47.4
- new net: U47.3, U47.5, U47.9, U48.1, U48.2
- new net: U47.12, U47.6
- new net: D78.1 (K), R239.2
- new net: U77.3, U77.5, U77.9, U78.1, U78.2
- new net: D79.1 (K), R241.2
- new net: U67.3, U67.5, U67.9, U68.1, U68.2
- new net: U68.3, U69.1, U69.4
- new net: U73.13, U73.8
- new net: U73.3, U73.5, U73.9, U74.1, U74.2
- new net: D83.1 (K), R249.2
- new net: Q223.3 (D), Q224.1 (G), R236.1
- new net: U85.11, U86.1
- new net: U86.3, U86.4, U86.5
- new net: Q258.3 (D), Q259.1 (G), R271.1
- new net: D99.1 (K), R280.2
- new net: D92.2 (A), R266.1
- new net: U28.3, U28.5, U28.9, U44.1, U44.2
- new net: U44.3, U45.1, U45.4
- new net: U31.3, U31.4, U31.5
- new net: D91.1 (K), R265.2
- new net: D111.1 (K), R304.2
- new net: Q292.3 (D), Q293.1 (G), R305.1
- new net: U58.3, U59.1, U59.4
- new net: Q294.3 (D), Q295.1 (G), R308.1
- new net: D93.1 (K), R268.2
- new net: Q274.3 (D), Q275.1 (G), R287.1
- new net: U25.3, U25.5, U25.9, U27.1, U27.2
- new net: U27.3, U28.1, U28.4
- new net: U28.12, U28.6
- new net: U28.13, U28.8
- new net: U49.13, U49.8
- new net: U77.13, U77.8
- new net: Q225.3 (D), Q226.1 (G), R238.1
- new net: Q245.3 (D), Q246.1 (G), R258.1
- new net: U74.3, U75.1, U75.4
- new net: U60.3, U61.1, U61.4
- new net: U61.3, U61.5, U61.9, U62.1, U62.2
- new net: U61.12, U61.6
- new net: D101.1 (K), R284.2
- new net: U73.12, U73.6
- new net: Q254.3 (D), Q255.1 (G), R267.1
- new net: D82.1 (K), R247.2
- new net: U25.13, U25.8
- new net: Q260.3 (D), Q261.1 (G), R273.1
- new net: Q231.3 (D), Q232.1 (G), R244.1
- new net: Q227.3 (D), Q228.1 (G), R240.1
- new net: U72.3, U73.1, U73.4
- new net: D88.1 (K), R259.2
- new net: D86.1 (K), R255.2
- new net: D90.1 (K), R263.2
- new net: Q241.3 (D), Q242.1 (G), R254.1
- new net: Q243.3 (D), Q244.1 (G), R256.1
- new net: D110.1 (K), R302.2
- new net: D106.1 (K), R294.2
- new net: Q268.3 (D), Q269.1 (G), R281.1
- new net: Q221.3 (D), Q222.1 (G), R234.1
- new net: D84.1 (K), R251.2
- new net: Q276.3 (D), Q277.1 (G), R289.1
- new net: U45.3, U45.5, U45.9, U46.1, U46.2
- new net: Q235.3 (D), Q236.1 (G), R248.1
- new net: U61.13, U61.8
- new net: U91.3, U91.4, U91.5
- new net: D94.1 (K), R270.2
- new net: U78.3, U79.1, U79.4
- new net: U79.3, U79.5, U79.9, U80.1, U80.2
- new net: F1.1, J9.1
- new net: Q290.3 (D), Q291.1 (G), R303.1
- new net: D113.1 (K), R309.2
- new net: U85.12, U85.6
- new net: U85.13, U85.8
- new net: Q266.3 (D), Q267.1 (G), R279.1
- new net: D102.1 (K), R286.2
- new net: D100.1 (K), R282.2
- new net: Q288.3 (D), Q289.1 (G), R301.1
- new net: Q282.3 (D), Q283.1 (G), R295.1
- new net: U17.3, U17.4, U17.5
- new net: R116.1, U87.1 (A->B)
- new net: U91.11, U91.9, U92.2
- new net: Q284.3 (D), Q285.1 (G), R297.1
- new net: R118.1, U89.1 (A->B)
- new net: U88.15 (Y0), U89.19 (CE)
- new net: U91.10, U91.6
- new net: D85.1 (K), R253.2
- new net: D103.1 (K), R288.2
- new net: U70.3, U71.1, U71.4
- new net: U71.3, U71.5, U71.9, U72.1, U72.2
- new net: U71.12, U71.6
- new net: U63.12, U63.6
- new net: U63.13, U63.8
- new net: U71.13, U71.8
- new net: D5.2 (A), R312.2
- new net: U79.13, U79.8
- new net: U45.12, U45.6
- new net: U45.13, U45.8
- new net: D95.1 (K), R272.2
- new net: Q272.3 (D), Q273.1 (G), R285.1
- new net: U66.3, U67.1, U67.4
- new net: U67.12, U67.6
- new net: D108.1 (K), R298.2
- new net: D4.2 (A), R311.2
- new net: U63.3, U63.5, U63.9, U64.1, U64.2
- new net: U25.12, U25.6
- new net: Q233.3 (D), Q234.1 (G), R246.1
- new net: Q249.3 (D), Q250.1 (G), R262.1
- new net: D109.1 (K), R300.2
- new net: Q286.3 (D), Q287.1 (G), R299.1
- new net: U88.14 (Y1), U90.19 (CE)
- new net: R117.1, U90.1 (A->B), U90.5 (A3), U90.7 (A5)
- new net: U69.3, U69.5, U69.9, U70.1, U70.2
- new net: U69.12, U69.6
- new net: D89.1 (K), R261.2
- new net: U47.13, U47.8
- new net: D112.1 (K), R306.2
- new net: U59.12, U59.6
- new net: D107.1 (K), R296.2
- new net: D77.1 (K), R237.2
- new net: U77.12, U77.6
- new net: D105.1 (K), R292.2
- new net: U79.12, U79.6
- new net: U67.13, U67.8
- new net: U85.3, U85.5, U85.9
- new net: D81.1 (K), R245.2
- new net: U62.3, U63.1, U63.4
- new net: U17.12, U17.13, U17.8
- new net: U75.12, U75.6
- new net: U69.13, U69.8
- new net: U75.13, U75.8
- new net: D76.1 (K), R235.2
- new net: D80.1 (K), R243.2
- new net BRANCH: Q253.1 (G), U81.1 (S), U82.1 (S), U83.1 (S), U84.1 (S), U86.6
- new net CLK0: D93.2 (A), Q255.3 (D)
- new net IOBUS_ADDR0: D98.2 (A), J10.13 (Pin_13), Q265.3 (D), U36.2 (A0), U81.3 (I1a)
- new net IOBUS_ADDR1: D99.2 (A), J10.14 (Pin_14), Q267.3 (D), U36.3 (A1), U81.6 (I1b)
- new net IOBUS_ADDR10: D108.2 (A), J10.25 (Pin_25), Q285.3 (D), U37.4 (A2), U83.10 (I1c)
- new net IOBUS_ADDR11: D109.2 (A), J10.26 (Pin_26), Q287.3 (D), U37.5 (A3), U83.13 (I1d)
- new net IOBUS_ADDR12: D110.2 (A), J10.27 (Pin_27), Q289.3 (D), U37.6 (A4), U84.3 (I1a)
- new net IOBUS_ADDR13: D111.2 (A), J10.28 (Pin_28), Q291.3 (D), U37.7 (A5), U84.6 (I1b)
- new net IOBUS_ADDR14: D112.2 (A), J10.29 (Pin_29), Q293.3 (D), U37.8 (A6), U84.10 (I1c)
- new net IOBUS_ADDR15: D113.2 (A), Q295.3 (D), U17.1, U17.9, U31.1, U37.9 (A7), U84.13 (I1d), U91.12, U91.13
- new net IOBUS_ADDR2: D100.2 (A), J10.15 (Pin_15), Q269.3 (D), U36.4 (A2), U81.10 (I1c)
- new net IOBUS_ADDR3: D101.2 (A), J10.16 (Pin_16), Q271.3 (D), U36.5 (A3), U81.13 (I1d)
- new net IOBUS_ADDR4: D102.2 (A), J10.17 (Pin_17), Q273.3 (D), U36.6 (A4), U82.3 (I1a)
- new net IOBUS_ADDR5: D103.2 (A), J10.18 (Pin_18), Q275.3 (D), U36.7 (A5), U82.6 (I1b)
- new net IOBUS_ADDR6: D104.2 (A), J10.19 (Pin_19), Q277.3 (D), U36.8 (A6), U82.10 (I1c)
- new net IOBUS_ADDR7: D105.2 (A), J10.20 (Pin_20), Q279.3 (D), U36.9 (A7), U82.13 (I1d)
- new net IOBUS_ADDR8: D106.2 (A), J10.23 (Pin_23), Q281.3 (D), U37.2 (A0), U83.3 (I1a)
- new net IOBUS_ADDR9: D107.2 (A), J10.24 (Pin_24), Q283.3 (D), U37.3 (A1), U83.6 (I1b)
- new net IOBUS_CLK: J10.33 (Pin_33), U31.6
- new net IOBUS_READ: J10.32 (Pin_32), U17.11
- new net IOBUS_WRITE: J10.34 (Pin_34), U17.6
- new net PCINCR_OUT0: U25.11, U81.2 (I0a)
- new net PCINCR_OUT1: U28.11, U81.5 (I0b)
- new net PCINCR_OUT10: U69.11, U83.11 (I0c)
- new net PCINCR_OUT11: U71.11, U83.14 (I0d)
- new net PCINCR_OUT12: U73.11, U84.2 (I0a)
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
Commit message: almost done with placement for IO board
Parts:
- removed R48, R49, R50, R51, R52, R53: 10K, Resistor_SMD:R_0402_1005Metric, symbol Device:R
- added C100, C101, C102, C103, C104, C105, C106, C107, C108, C109, C110, C111, C99: 100nF, Capacitor_SMD:C_0402_1005Metric, symbol Device:C
- added C26, C41, C97, C98: 22uF, Capacitor_THT:C_Radial_D5.0mm_H11.0mm_P2.00mm, symbol Device:C
- added D7: PWR_USB, LED_SMD:LED_0402_1005Metric, symbol Device:LED
- added R313: 1K, Resistor_SMD:R_0402_1005Metric, symbol Device:R
- D3: value RX -> IND1
- D4: value RX -> PWR
- D5: value RX -> IND0
- J4: footprint Connector_PinSocket_2.54mm:PinSocket_2x40_P2.54mm_Horizontal -> Connector_PinHeader_2.54mm:PinHeader_2x40_P2.54mm_Horizontal
- J5, J6: footprint Connector_PinHeader_2.54mm:PinHeader_2x16_P2.54mm_Horizontal -> Connector_PinSocket_2.54mm:PinSocket_2x16_P2.54mm_Horizontal
- J7: footprint Connector_PinHeader_2.54mm:PinHeader_2x12_P2.54mm_Vertical -> Connector_PinSocket_2.54mm:PinSocket_2x12_P2.54mm_Vertical
- J8: footprint Connector_PinHeader_2.54mm:PinHeader_2x24_P2.54mm_Horizontal -> Connector_PinSocket_2.54mm:PinSocket_2x24_P2.54mm_Horizontal
- SW1: value SW_Push -> BTN_RESET
- SW2: value SW_Push -> BTN_HALT
- SW3: value SW_Push -> BTN_STEP
- SW4: value SW_Push -> BTN_CLKEN
- SW5: value SW_Push -> BTN_CLKUP
- SW6: value SW_Push -> BTN_CLKDOWN
- SW7: value SW_Push -> BTN_RESET_ATMEGA
Connections:
- net +5V: now also C100.2, C101.2, C102.2, C103.2, C104.2, C105.2, C106.2, C107.2, C108.2, C109.2, C110.2, C111.2, C26.1, C41.1, C97.1, C98.1, C99.2; no longer C50.2, D1.2 (A), D2.2 (A), U18.14 (VCC)
- net ARBIT_BTN_CLKDOWN: no longer U18.12
- net ARBIT_BTN_CLKEN: no longer U18.8
- net ARBIT_BTN_CLKUP: no longer U18.10
- net ARBIT_BTN_RESET: no longer U18.2
- net ARBIT_BTN_STEP: no longer U18.6
- net ARBIT_BTN_TOGGLEHALT: no longer U18.4
- net GND: now also U29.1 (A->B), U30.1 (A->B), U32.1 (A->B), U32.11 (B7), U33.1 (A->B), U33.11 (B7), U33.12 (B6), U33.13 (B5), U33.14 (B4), U33.15 (B3), U33.16 (B2), U33.17 (B1), U33.18 (B0), U36.1 (A->B), U37.1 (A->B), C100.1, C101.1, C102.1, C103.1, C104.1, C105.1, C106.1, C107.1, C108.1, C109.1, C110.1, C111.1, C26.2, C41.2, C97.2, C98.2, C99.1, D7.1 (K); no longer C50.1, U18.7 (GND), U32.9 (A7), U33.2 (A0), U33.3 (A1), U33.4 (A2), U33.5 (A3), U33.6 (A4), U33.7 (A5), U33.8 (A6), U33.9 (A7)
- net INS_OPCODE0: now also U32.18 (B0); no longer U32.2 (A0)
- net INS_OPCODE1: now also U32.17 (B1); no longer U32.3 (A1)
- net INS_OPCODE2: now also U32.16 (B2); no longer U32.4 (A2)
- net INS_OPCODE3: now also U32.15 (B3); no longer U32.5 (A3)
- net INS_OPCODE4: now also U32.14 (B4); no longer U32.6 (A4)
- net INS_OPCODE5: now also U32.13 (B5); no longer U32.7 (A5)
- net INS_OPCODE6: now also U32.12 (B6); no longer U32.8 (A6)
- net IOBUS_ADDR0: now also U36.18 (B0); no longer U36.2 (A0)
- net IOBUS_ADDR1: now also U36.17 (B1); no longer U36.3 (A1)
- net IOBUS_ADDR10: now also U37.16 (B2); no longer U37.4 (A2)
- net IOBUS_ADDR11: now also U37.15 (B3); no longer U37.5 (A3)
- net IOBUS_ADDR12: now also U37.14 (B4); no longer U37.6 (A4)
- net IOBUS_ADDR13: now also U37.13 (B5); no longer U37.7 (A5)
- net IOBUS_ADDR14: now also U37.12 (B6); no longer U37.8 (A6)
- net IOBUS_ADDR15: now also U37.11 (B7); no longer U37.9 (A7)
- net IOBUS_ADDR2: now also U36.16 (B2); no longer U36.4 (A2)
- net IOBUS_ADDR3: now also U36.15 (B3); no longer U36.5 (A3)
- net IOBUS_ADDR4: now also U36.14 (B4); no longer U36.6 (A4)
- net IOBUS_ADDR5: now also U36.13 (B5); no longer U36.7 (A5)
- net IOBUS_ADDR6: now also U36.12 (B6); no longer U36.8 (A6)
- net IOBUS_ADDR7: now also U36.11 (B7); no longer U36.9 (A7)
- net IOBUS_ADDR8: now also U37.18 (B0); no longer U37.2 (A0)
- net IOBUS_ADDR9: now also U37.17 (B1); no longer U37.3 (A1)
- net OPROM_A0: now also U32.2 (A0); no longer U32.18 (B0)
- net OPROM_A1: now also U32.3 (A1); no longer U32.17 (B1)
- net OPROM_A10: now also U33.4 (A2); no longer U33.16 (B2)
- net OPROM_A11: now also U33.5 (A3); no longer U33.15 (B3)
- net OPROM_A12: now also U33.6 (A4); no longer U33.14 (B4)
- net OPROM_A13: now also U33.7 (A5); no longer U33.13 (B5)
- net OPROM_A14: now also U33.8 (A6); no longer U33.12 (B6)
- net OPROM_A15: now also U33.9 (A7); no longer U33.11 (B7)
- net OPROM_A2: now also U32.4 (A2); no longer U32.16 (B2)
- net OPROM_A3: now also U32.5 (A3); no longer U32.15 (B3)
- net OPROM_A4: now also U32.6 (A4); no longer U32.14 (B4)
- net OPROM_A5: now also U32.7 (A5); no longer U32.13 (B5)
- net OPROM_A6: now also U32.8 (A6); no longer U32.12 (B6)
- net OPROM_A7: now also U32.9 (A7); no longer U32.11 (B7)
- net OPROM_A8: now also U33.2 (A0); no longer U33.18 (B0)
- net OPROM_A9: now also U33.3 (A1); no longer U33.17 (B1)
- net PROM_A0: now also U29.2 (A0); no longer U29.18 (B0)
- net PROM_A1: now also U29.3 (A1); no longer U29.17 (B1)
- net PROM_A10: now also U30.4 (A2); no longer U30.16 (B2)
- net PROM_A11: now also U30.5 (A3); no longer U30.15 (B3)
- net PROM_A12: now also U30.6 (A4); no longer U30.14 (B4)
- net PROM_A13: now also U30.7 (A5); no longer U30.13 (B5)
- net PROM_A14: now also U30.8 (A6); no longer U30.12 (B6)
- net PROM_A15: now also U30.9 (A7); no longer U30.11 (B7)
- net PROM_A2: now also U29.4 (A2); no longer U29.16 (B2)
- net PROM_A3: now also U29.5 (A3); no longer U29.15 (B3)
- net PROM_A4: now also U29.6 (A4); no longer U29.14 (B4)
- net PROM_A5: now also U29.7 (A5); no longer U29.13 (B5)
- net PROM_A6: now also U29.8 (A6); no longer U29.12 (B6)
- net PROM_A7: now also U29.9 (A7); no longer U29.11 (B7)
- net PROM_A8: now also U30.2 (A0); no longer U30.18 (B0)
- net PROM_A9: now also U30.3 (A1); no longer U30.17 (B1)
- net RAM_A0: now also U36.2 (A0); no longer U36.18 (B0)
- net RAM_A1: now also U36.3 (A1); no longer U36.17 (B1)
- net RAM_A10: now also U37.4 (A2); no longer U37.16 (B2)
- net RAM_A11: now also U37.5 (A3); no longer U37.15 (B3)
- net RAM_A12: now also U37.6 (A4); no longer U37.14 (B4)
- net RAM_A13: now also U37.7 (A5); no longer U37.13 (B5)
- net RAM_A14: now also U37.8 (A6); no longer U37.12 (B6)
- net RAM_A15: now also U37.9 (A7); no longer U37.11 (B7)
- net RAM_A2: now also U36.4 (A2); no longer U36.16 (B2)
- net RAM_A3: now also U36.5 (A3); no longer U36.15 (B3)
- net RAM_A4: now also U36.6 (A4); no longer U36.14 (B4)
- net RAM_A5: now also U36.7 (A5); no longer U36.13 (B5)
- net RAM_A6: now also U36.8 (A6); no longer U36.12 (B6)
- net RAM_A7: now also U36.9 (A7); no longer U36.11 (B7)
- net RAM_A8: now also U37.2 (A0); no longer U37.18 (B0)
- net RAM_A9: now also U37.3 (A1); no longer U37.17 (B1)
- net S_PC0: now also U29.18 (B0); no longer U29.2 (A0)
- net S_PC1: now also U29.17 (B1); no longer U29.3 (A1)
- net S_PC10: now also U30.16 (B2); no longer U30.4 (A2)
- net S_PC11: now also U30.15 (B3); no longer U30.5 (A3)
- net S_PC12: now also U30.14 (B4); no longer U30.6 (A4)
- net S_PC13: now also U30.13 (B5); no longer U30.7 (A5)
- net S_PC14: now also U30.12 (B6); no longer U30.8 (A6)
- net S_PC15: now also U30.11 (B7); no longer U30.9 (A7)
- net S_PC2: now also U29.16 (B2); no longer U29.4 (A2)
- net S_PC3: now also U29.15 (B3); no longer U29.5 (A3)
- net S_PC4: now also U29.14 (B4); no longer U29.6 (A4)
- net S_PC5: now also U29.13 (B5); no longer U29.7 (A5)
- net S_PC6: now also U29.12 (B6); no longer U29.8 (A6)
- net S_PC7: now also U29.11 (B7); no longer U29.9 (A7)
- net S_PC8: now also U30.18 (B0); no longer U30.2 (A0)
- net S_PC9: now also U30.17 (B1); no longer U30.3 (A1)
- net VUSB: now also D1.2 (A), D2.2 (A), R313.1
- net at C8.2, R20.1: no longer U18.11
- net at C6.2, R16.1: no longer U18.5
- net at C4.2, R11.1: no longer U18.1
- net at C7.2, R18.1: no longer U18.9
- net at C5.2, R14.1: no longer U18.3
- net at C9.2, R22.1: no longer U18.13
- new net: D7.2 (A), R313.2
Other:
- moved on the sheet: C50, J2, U18A, U18B, U18C, U18D, U18E, U18F, U18G
