File: hardware/io/io.kicad_sch (KiCad schematic)
At the start: 793 parts, among them J1 USB_B, J10 Conn_02x18_Odd_Even, J11 Barrel_Jack_Switch_Pin3Ring, J2 Conn_02x03_Odd_Even, J3 Conn_02x08_Odd_Even, J4 Conn_02x40_Odd_Even, J5 Conn_02x16_Odd_Even, J6 Conn_02x16_Odd_Even, J7 Conn_02x12_Odd_Even, J8 Conn_02x24_Odd_Even, Q129 IRLML6244, Q130 IRLML6402, Q131 IRLML6244, Q132 IRLML6402, Q133 IRLML6244, Q134 IRLML6402, Q135 IRLML6244, Q136 IRLML6402, Q137 IRLML6244, Q138 IRLML6402, Q139 IRLML6244, Q140 IRLML6402, Q141 IRLML6244, Q142 IRLML6402, Q143 IRLML6244, Q144 IRLML6402, Q145 IRLML6244, Q146 IRLML6402, Q147 IRLML6244, Q148 IRLML6402, Q149 IRLML6244, Q150 IRLML6402, Q151 IRLML6244, Q152 IRLML6402, Q153 IRLML6244, Q154 IRLML6402, Q155 IRLML6244, Q156 IRLML6402, Q157 IRLML6244, Q158 IRLML6402, Q159 IRLML6244, Q160 IRLML6402, Q161 IRLML6244, Q162 IRLML6402, Q163 IRLML6244, Q164 IRLML6402, Q165 IRLML6244, Q166 IRLML6402, Q167 IRLML6244, Q168 IRLML6402, Q169 IRLML6244, Q170 IRLML6402, Q171 IRLML6244, Q172 IRLML6402, Q173 IRLML6244, Q174 IRLML6402, Q175 IRLML6244, Q176 IRLML6402, Q177 IRLML6244, Q178 IRLML6402, Q179 IRLML6244, Q180 IRLML6402, Q181 IRLML6244, Q182 IRLML6402, Q183 IRLML6244, Q184 IRLML6402, Q185 IRLML6244, Q186 IRLML6402, Q187 IRLML6244, Q188 IRLML6402, Q189 IRLML6244, Q190 IRLML6402, Q191 IRLML6244, Q192 IRLML6402, Q193 IRLML6244, Q194 IRLML6402, Q195 IRLML6244, Q196 IRLML6402, Q197 IRLML6244, Q198 IRLML6402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

Commit message: as ordered
Parts:
- C1, C2: LCSC (none) -> C541460
- C100, C101, C102, C103, C104, C105, C106, C107, C108, C109, C11, C110, C111, C12, C13, C14, C15, C16, C17, C18, C19, C20, C21, C22, C23, C24, C25, C27, C28, C29, C3, C30, C31, C32, C33, C34, C35, C36, C37, C38, C39, C4, C40, C42, C43, C44, C45, C46, C47, C48, C49, C5, C50, C51, C52, C53, C54, C55, C56, C57, C58, C59, C6, C60, C61, C62, C63, C64, C65, C66, C67, C68, C69, C7, C70, C71, C72, C73, C74, C75, C76, C77, C78, C79, C8, C80, C81, C82, C83, C84, C85, C86, C87, C88, C89, C9, C90, C91, C92, C93, C94, C95, C96, C99: LCSC (none) -> C77020
- D1, D2, D3, D4, D5, D7: LCSC (none) -> C965793
- D6: LCSC (none) -> C444414
- R1, R10, R11, R14, R16, R18, R2, R20, R22, R23, R24, R25, R26, R3, R310, R311, R312, R313, R33, R34, R35, R4, R5, R6, R7, R8, R9: LCSC (none) -> C106235
- R100, R101, R102, R103, R104, R105, R106, R107, R108, R109, R110, R111, R112, R113, R114, R119, R120, R121, R122, R123, R124, R125, R126, R127, R128, R129, R130, R131, R132, R133, R134, R135, R136, R137, R138, R139, R140, R141, R307, R37, R38, R39, R40, R41, R54, R55, R56, R57, R58, R59, R60, R61, R62, R63, R64, R65, R66, R67, R68, R69, R70, R71, R72, R73, R74, R75, R76, R77, R78, R79, R80, R81, R82, R83, R84, R85, R86, R87, R88, R89, R90, R91, R92, R93, R94, R95, R96, R97, R98, R99: LCSC C60490 -> C60491
- R116, R117, R118, R12, R13, R15, R17, R19, R21, R27, R28, R29, R30, R31, R32, R36, R42, R43, R44, R45, R46, R47: LCSC (none) -> C60490
- U11, U26: LCSC (none) -> C5602
- U12, U13, U14, U15, U16, U19, U20, U21, U22, U23, U24, U29, U3, U30, U32, U33, U34, U35, U36, U37, U38, U39, U40, U41, U87, U89, U90: LCSC (none) -> C5626
- U17, U25, U27, U28, U31, U44, U45, U46, U47, U48, U49, U58, U59, U60, U61, U62, U63, U64, U65, U66, U67, U68, U69, U70, U71, U72, U73, U74, U75, U76, U77, U78, U79, U80, U85, U86, U91, U92: LCSC (none) -> C5586
- U18: LCSC (none) -> C5605
- U4: LCSC (none) -> C22460
- U42, U43, U88: LCSC (none) -> C5620
- U5: LCSC (none) -> C8690
- Y1: LCSC (none) -> C5261144
